File: Befehle.sch (KiCad schematic (older format))
At the start: 55 parts, among them P2 CONN_02X10, U1 4069, U2 74LS04, U3 7400, U4 74HCT02, U5 74LS541, U6 74LS373, U7 74LS139, U8 74LS540

Commit message: Footprints added
Parts:
- added U9: 74LS540, symbol 74LS540
- U1: symbol 4069 -> 74LS14
- U3, U4: footprint (none) -> Housings_DIP:DIP-14_W7.62mm_Socket_LongPads
- U5, U6: footprint Housings_DIP:DIP-18_W7.62mm_Socket_LongPads -> Housings_DIP:DIP-20_W7.62mm_Socket_LongPads
- U8: footprint Housings_DIP:DIP-20_W7.62mm_SMDSocket_SmallPads -> Housings_DIP:DIP-20_W7.62mm_Socket_LongPads
- renumbered P2 to P1
Changed lines of the file:
@@
 F 0 "U6" H -6400 3234 50  0000 C CNN
 F 1 "74LS373" H -6400 3325 50  0000 C CNN
-F 2 "Housings_DIP:DIP-18_W7.62mm_Socket_LongPads" H -6400 4000 50  0000 C CNN
+F 2 "Housings_DIP:DIP-20_W7.62mm_Socket_LongPads" H -6400 4000 50  0000 C CNN
 F 3 "" H -6400 4000 50  0000 C CNN
 	1    -6400 4000
@@
 F 0 "U5" H -6400 434 50  0000 C CNN
 F 1 "74LS541" H -6400 525 50  0000 C CNN
-F 2 "Housings_DIP:DIP-18_W7.62mm_Socket_LongPads" H -6400 1200 50  0000 C CNN
+F 2 "Housings_DIP:DIP-20_W7.62mm_Socket_LongPads" H -6400 1200 50  0000 C CNN
 F 3 "" H -6400 1200 50  0000 C CNN
 	1    -6400 1200
@@
 F 0 "U4" H -7700 4550 50  0000 C CNN
 F 1 "74HCT02" H -7650 4450 50  0000 C CNN
-F 2 "" H -7700 4500 50  0000 C CNN
+F 2 "Housings_DIP:DIP-14_W7.62mm_Socket_LongPads" H -7700 4500 50  0000 C CNN
 F 3 "" H -7700 4500 50  0000 C CNN
 	1    -7700 4500
@@
 F 0 "U4" H -7700 5100 50  0000 C CNN
 F 1 "74HCT02" H -7650 5000 50  0000 C CNN
-F 2 "" H -7700 5050 50  0000 C CNN
+F 2 "Housings_DIP:DIP-14_W7.62mm_Socket_LongPads" H -7700 5050 50  0000 C CNN
 F 3 "" H -7700 5050 50  0000 C CNN
 	2    -7700 5050
@@
 F 0 "U4" H -7700 5650 50  0000 C CNN
 F 1 "74HCT02" H -7650 5550 50  0000 C CNN
-F 2 "" H -7700 5600 50  0000 C CNN
+F 2 "Housings_DIP:DIP-14_W7.62mm_Socket_LongPads" H -7700 5600 50  0000 C CNN
 F 3 "" H -7700 5600 50  0000 C CNN
 	3    -7700 5600
@@
 F 0 "U4" H -7700 6200 50  0000 C CNN
 F 1 "74HCT02" H -7650 6100 50  0000 C CNN
-F 2 "" H -7700 6150 50  0000 C CNN
+F 2 "Housings_DIP:DIP-14_W7.62mm_Socket_LongPads" H -7700 6150 50  0000 C CNN
 F 3 "" H -7700 6150 50  0000 C CNN
 	4    -7700 6150
@@
 F 0 "U8" H -4050 284 50  0000 C CNN
 F 1 "74LS540" H -4050 375 50  0000 C CNN
-F 2 "Housings_DIP:DIP-20_W7.62mm_SMDSocket_SmallPads" H -4050 1050 50  0000 C CNN
+F 2 "Housings_DIP:DIP-20_W7.62mm_Socket_LongPads" H -4050 1050 50  0000 C CNN
 F 3 "" H -4050 1050 50  0000 C CNN
 	1    -4050 1050
@@
 F 0 "U3" H -8400 7300 50  0000 C CNN
 F 1 "7400" H -8400 7150 50  0000 C CNN
-F 2 "" H -8400 7250 50  0000 C CNN
+F 2 "Housings_DIP:DIP-14_W7.62mm_Socket_LongPads" H -8400 7250 50  0000 C CNN
 F 3 "" H -8400 7250 50  0000 C CNN
 	2    -8400 7250
@@
 F 0 "U3" H -8300 8500 50  0000 C CNN
 F 1 "7400" H -8300 8350 50  0000 C CNN
-F 2 "" H -8300 8450 50  0000 C CNN
+F 2 "Housings_DIP:DIP-14_W7.62mm_Socket_LongPads" H -8300 8450 50  0000 C CNN
 F 3 "" H -8300 8450 50  0000 C CNN
 	3    -8300 8450
@@
 F 0 "U3" H -7650 8900 50  0000 C CNN
 F 1 "7400" H -7650 8750 50  0000 C CNN
-F 2 "" H -7650 8850 50  0000 C CNN
+F 2 "Housings_DIP:DIP-14_W7.62mm_Socket_LongPads" H -7650 8850 50  0000 C CNN
 F 3 "" H -7650 8850 50  0000 C CNN
 	4    -7650 8850
@@
 F 0 "U3" H -8650 6100 50  0000 C CNN
 F 1 "7400" H -8650 5950 50  0000 C CNN
-F 2 "" H -8650 6050 50  0000 C CNN
+F 2 "Housings_DIP:DIP-14_W7.62mm_Socket_LongPads" H -8650 6050 50  0000 C CNN
 F 3 "" H -8650 6050 50  0000 C CNN
 	1    -8650 6050
@@
 $EndComp
 $Comp
-L 4069 U1
+L 74LS14 U1
 U 1 1 57FBE09D
 P -9250 950
@@
 $EndComp
 $Comp
-L VCC #PWR01
+L VCC #PWR5
 U 1 1 57FBF211
 P -8800 2450
-F 0 "#PWR01" H -8800 2300 50  0001 C CNN
+F 0 "#PWR5" H -8800 2300 50  0001 C CNN
 F 1 "VCC" H -8800 2600 50  0000 C CNN
 F 2 "" H -8800 2450 50  0000 C CNN
@@
 $EndComp
 $Comp
-L VCC #PWR02
+L VCC #PWR1
 U 1 1 57FBF424
 P -9700 1250
-F 0 "#PWR02" H -9700 1100 50  0001 C CNN
+F 0 "#PWR1" H -9700 1100 50  0001 C CNN
 F 1 "VCC" H -9700 1400 50  0000 C CNN
 F 2 "" H -9700 1250 50  0000 C CNN
@@
 enableR
 $Comp
-L GND #PWR03
+L GND #PWR10
 U 1 1 57FC32E9
 P -6200 1900
-F 0 "#PWR03" H -6200 1650 50  0001 C CNN
+F 0 "#PWR10" H -6200 1650 50  0001 C CNN
 F 1 "GND" H -6200 1750 50  0000 C CNN
 F 2 "" H -6200 1900 50  0000 C CNN
@@
 $EndComp
 $Comp
-L GND #PWR04
+L GND #PWR9
 U 1 1 57FC33C9
 P -6300 1900
-F 0 "#PWR04" H -6300 1650 50  0001 C CNN
+F 0 "#PWR9" H -6300 1650 50  0001 C CNN
 F 1 "GND" H -6300 1750 50  0000 C CNN
 F 2 "" H -6300 1900 50  0000 C CNN
@@
 $EndComp
 $Comp
-L GND #PWR05
+L GND #PWR13
 U 1 1 57FC4CCE
 P -3600 1750
-F 0 "#PWR05" H -3600 1500 50  0001 C CNN
+F 0 "#PWR13" H -3600 1500 50  0001 C CNN
 F 1 "GND" H -3600 1600 50  0000 C CNN
 F 2 "" H -3600 1750 50  0000 C CNN
@@
 $EndComp
 $Comp
-L VCC #PWR06
+L VCC #PWR14
 U 1 1 57FC686E
 P -3450 5100
-F 0 "#PWR06" H -3450 4950 50  0001 C CNN
+F 0 "#PWR14" H -3450 4950 50  0001 C CNN
 F 1 "VCC" H -3450 5250 50  0000 C CNN
 F 2 "" H -3450 5100 50  0000 C CNN
@@
 $EndComp
 $Comp
-L VCC #PWR07
+L VCC #PWR15
 U 1 1 57FC839A
 P -3200 9450
-F 0 "#PWR07" H -3200 9300 50  0001 C CNN
+F 0 "#PWR15" H -3200 9300 50  0001 C CNN
 F 1 "VCC" H -3200 9600 50  0000 C CNN
 F 2 "" H -3200 9450 50  0000 C CNN
@@
 3
 $Comp
-L VCC #PWR08
+L VCC #PWR7
 U 1 1 57FCF846
 P -8300 3700
-F 0 "#PWR08" H -8300 3550 50  0001 C CNN
+F 0 "#PWR7" H -8300 3550 50  0001 C CNN
 F 1 "VCC" H -8300 3850 50  0000 C CNN
 F 2 "" H -8300 3700 50  0000 C CNN
@@
 $EndComp
 $Comp
-L GND #PWR09
+L GND #PWR12
 U 1 1 580EBD54
 P -5850 6350
-F 0 "#PWR09" H -5850 6100 50  0001 C CNN
+F 0 "#PWR12" H -5850 6100 50  0001 C CNN
 F 1 "GND" H -5850 6200 50  0000 C CNN
 F 2 "" H -5850 6350 50  0000 C CNN
@@
 $EndComp
 $Comp
-L VCC #PWR010
+L VCC #PWR11
 U 1 1 580EC580
 P -5900 4700
-F 0 "#PWR010" H -5900 4550 50  0001 C CNN
+F 0 "#PWR11" H -5900 4550 50  0001 C CNN
 F 1 "VCC" H -5900 4850 50  0000 C CNN
 F 2 "" H -5900 4700 50  0000 C CNN
@@
 $EndComp
 $Comp
-L VCC #PWR011
+L VCC #PWR6
 U 1 1 580F57E4
 P -8700 8400
-F 0 "#PWR011" H -8700 8250 50  0001 C CNN
+F 0 "#PWR6" H -8700 8250 50  0001 C CNN
 F 1 "VCC" H -8700 8550 50  0000 C CNN
 F 2 "" H -8700 8400 50  0000 C CNN
@@
 $EndComp
 $Comp
-L VCC #PWR012
+L VCC #PWR3
 U 1 1 582A32CB
 P -9150 5900
-F 0 "#PWR012" H -9150 5750 50  0001 C CNN
+F 0 "#PWR3" H -9150 5750 50  0001 C CNN
 F 1 "VCC" H -9150 6050 50  0000 C CNN
 F 2 "" H -9150 5900 50  0000 C CNN
@@
 $EndComp
 $Comp
-L VCC #PWR013
+L VCC #PWR2
 U 1 1 582B09F9
 P -9500 5000
-F 0 "#PWR013" H -9500 4850 50  0001 C CNN
+F 0 "#PWR2" H -9500 4850 50  0001 C CNN
 F 1 "VCC" H -9500 5150 50  0000 C CNN
 F 2 "" H -9500 5000 50  0000 C CNN
@@
 $EndComp
 $Comp
-L VCC #PWR014
+L VCC #PWR4
 U 1 1 582B5718
 P -8850 3600
-F 0 "#PWR014" H -8850 3450 50  0001 C CNN
+F 0 "#PWR4" H -8850 3450 50  0001 C CNN
 F 1 "VCC" H -8850 3750 50  0000 C CNN
 F 2 "" H -8850 3600 50  0000 C CNN
@@
 $EndComp
 $Comp
-L GND #PWR015
+L GND #PWR8
 U 1 1 582B6B6B
 P -7750 2350
-F 0 "#PWR015" H -7750 2100 50  0001 C CNN
+F 0 "#PWR8" H -7750 2100 50  0001 C CNN
 F 1 "GND" H -7750 2200 50  0000 C CNN
 F 2 "" H -7750 2350 50  0000 C CNN
@@
 $EndComp
 $Comp
-L CONN_02X10 P2
+L CONN_02X10 P1
 U 1 1 5A1624C1
 P -6350 7300
-F 0 "P2" V -6304 6762 50  0000 R CNN
+F 0 "P1" V -6304 6762 50  0000 R CNN
 F 1 "CONN_02X10" V -6395 6762 50  0000 R CNN
 F 2 "Connect:IDC_Header_Straight_20pins" H -6350 6100 50  0000 C CNN
@@
 	-6900 2650 -3950 2650
 Wire Bus Line
-	-3950 2650 -3950 1950
+	-3950 1950 -3950 2650
 Wire Bus Line
-	-3950 1950 -4650 1950
+	-4650 1950 -3950 1950
 Wire Wire Line
 	-3300 -150 -4550 -150
@@
 	-6200 4700 -6200 4750
 Wire Wire Line
-	-42900 25500 -42900 40500
-Wire Wire Line
-	-42900 40500 -58500 40500
+	-42900 40500 -42900 25500
+Wire Wire Line
+	-58500 40500 -42900 40500
 Wire Wire Line
 	-58500 40500 -58500 25400
@@
 	-53650 48450 -56350 48450
 Connection ~ -53650 40500
+$Comp
+L 74LS540 U9
+U 1 1 5A1F49EC
+P -2250 7100
+F 0 "U9" H -2250 6900 50  0000 C CNN
+F 1 "74LS540" H -2250 6800 50  0000 C CNN
+F 2 "" H -2250 7100 50  0000 C CNN
+F 3 "" H -2250 7100 50  0000 C CNN
+	1    -2250 7100
+	1    0    0    -1
+$EndComp
 $EndSCHEMATC
