File: Befehle.sch (KiCad schematic (older format))
At the start: 56 parts, among them J1 691213710003, P1 CONN_02X10, P2 CONN_02X10, P3 CONN_01X01, P4 CONN_01X01, U1 74LS14, U2 74540, U3 7400, U4 74HCT02, U5 74LS541, U6 74LS373, U7 74LS139, U8 74LS540

Commit message: used libraries added
Parts:
- removed J1: 691213710003, 691213710003, symbol PCB~Terminal~Blocks:691213710003
Changed lines of the file:
@@
 	1550 6700 1550 6650
 Connection ~ 1550 6350
-$Comp
-L PCB~Terminal~Blocks:691213710003 J1
-U 1 1 5AC4CF5E
-P 1300 4650
-F 0 "J1" H 1265 4690 50  0000 L CNN
-F 1 "691213710003" H 1265 4599 50  0000 L CNN
-F 2 "691213710003" H 1300 4650 50  0001 L BNN
-F 3 "1.12 USD" H 1300 4650 50  0001 L BNN
-F 4 "Warning" H 1300 4650 50  0001 L BNN "Field4"
-F 5 "Wurth Electronics" H 1300 4650 50  0001 L BNN "Field5"
-F 6 "TERM BLK 5MM HORZ ENTRY MOD 3P" H 1300 4650 50  0001 L BNN "Field6"
-F 7 "None" H 1300 4650 50  0001 L BNN "Field7"
-F 8 "691213710003" H 1300 4650 50  0001 L BNN "Field8"
-	1    1300 4650
-	1    0    0    -1
-$EndComp
 Text GLabel 900  4900 0    60   Input ~ 0
 upPC
@@
 Wire Wire Line
 	-3100 8550 -3000 8550
-Wire Bus Line
-	-6500 6800 -6300 6800
 Wire Wire Line
 	-2900 8500 -2900 8750
 Wire Bus Line
+	-6500 6800 -6300 6800
+Wire Bus Line
 	-6300 6800 -5900 6800

Commit message: Befehle: Header ausgetauscht
Parts:
- P1, P2: footprint Connect:IDC_Header_Straight_20pins -> tg_foodprint:Pin_Header_Straight_2x10_Pitch2.00mmBonsai.pretty
Connections:
- wire segments 258 -> 278
Changed lines of the file:
@@
 EESchema Schematic File Version 4
+LIBS:Befehle-cache
 EELAYER 26 0
 EELAYER END
@@
 F 0 "P2" V -6004 -1288 50  0000 R CNN
 F 1 "CONN_02X10" V -6095 -1288 50  0000 R CNN
-F 2 "Connect:IDC_Header_Straight_20pins" H -6050 -1950 50  0000 C CNN
+F 2 "tg_foodprint:Pin_Header_Straight_2x10_Pitch2.00mmBonsai.pretty" H -6050 -1950 50  0000 C CNN
 F 3 "" H -6050 -1950 50  0000 C CNN
 	1    -6050 -750
@@
 F 0 "P1" V -6254 6662 50  0000 R CNN
 F 1 "CONN_02X10" V -6345 6662 50  0000 R CNN
-F 2 "Connect:IDC_Header_Straight_20pins" H -6300 6000 50  0000 C CNN
+F 2 "tg_foodprint:Pin_Header_Straight_2x10_Pitch2.00mmBonsai.pretty" H -6300 6000 50  0000 C CNN
 F 3 "" H -6300 6000 50  0000 C CNN
 	1    -6300 7200
@@
 Wire Wire Line
 	-5900 6900 -5650 6900
-Wire Wire Line
-	-6850 7400 -5650 7400
-Wire Wire Line
-	-6550 -1050 -5450 -1050
 Connection ~ -3100 8550
 Wire Wire Line
@@
 Wire Wire Line
 	-2900 8500 -2900 8750
+Wire Wire Line
+	-6550 -1050 -6450 -1050
+Connection ~ -5550 -1050
+Wire Wire Line
+	-5550 -1050 -5450 -1050
+Connection ~ -6450 -1050
+Wire Wire Line
+	-6450 -1050 -6350 -1050
+Connection ~ -6350 -1050
+Wire Wire Line
+	-6350 -1050 -6250 -1050
+Connection ~ -6250 -1050
+Wire Wire Line
+	-6250 -1050 -6150 -1050
+Connection ~ -6150 -1050
+Wire Wire Line
+	-6150 -1050 -6050 -1050
+Connection ~ -6050 -1050
+Wire Wire Line
+	-6050 -1050 -5950 -1050
+Connection ~ -5950 -1050
+Wire Wire Line
+	-5950 -1050 -5850 -1050
+Connection ~ -5850 -1050
+Wire Wire Line
+	-5850 -1050 -5750 -1050
+Connection ~ -5750 -1050
+Wire Wire Line
+	-5750 -1050 -5650 -1050
+Connection ~ -5650 -1050
+Wire Wire Line
+	-5650 -1050 -5550 -1050
+Wire Wire Line
+	-6850 7400 -6700 7400
 Wire Bus Line
 	-6500 6800 -6300 6800
@@
 Wire Bus Line
 	-7050 4850 -6300 4850
+Connection ~ -6700 7400
+Wire Wire Line
+	-6700 7400 -6600 7400
+Connection ~ -5800 7400
+Wire Wire Line
+	-5800 7400 -5650 7400
+Connection ~ -6600 7400
+Wire Wire Line
+	-6600 7400 -6500 7400
+Connection ~ -6500 7400
+Wire Wire Line
+	-6500 7400 -6400 7400
+Connection ~ -6400 7400
+Wire Wire Line
+	-6400 7400 -6300 7400
+Connection ~ -6300 7400
+Wire Wire Line
+	-6300 7400 -6200 7400
+Connection ~ -6200 7400
+Wire Wire Line
+	-6200 7400 -6100 7400
+Connection ~ -6100 7400
+Wire Wire Line
+	-6100 7400 -6000 7400
+Connection ~ -6000 7400
+Wire Wire Line
+	-6000 7400 -5900 7400
+Connection ~ -5900 7400
+Wire Wire Line
+	-5900 7400 -5800 7400
 $EndSCHEMATC
