File: Steuerwerk.sch (KiCad schematic (older format))
At the start: 95 parts

Commit message: Steuerwerk aktualisiert
Connections:
- wire segments 206 -> 297

Commit message: Steuerwerk aktualisiert
Connections:
- wire segments 297 -> 300
Changed lines of the file:
@@
 	850  6300 1900 6300
 Wire Wire Line
-	1900 6300 6850 3600
+	1900 6300 4300 4500
 $Comp
 L 74LS374 U?
@@
 	0    -1   1    0
 $EndComp
+Wire Wire Line
+	4300 4500 4300 3700
+Wire Wire Line
+	4300 3700 4650 3700
+Wire Wire Line
+	4650 3700 6550 3750
 $EndSCHEMATC

Commit message: Steuerwerk aktualisiert
Parts:
- added D?: LED, symbol LED
- added P? (x14): CONN_01X01, symbol CONN_01X01
- added R?: R, symbol R
- added U?: 74LS04, symbol 74LS04
Connections:
- net labels added: 1, 10, 11, 12, 13, 14, 15, 16, 2, 3, 4, 5, 6, 7, 8, 9, Takt, clrMPC, enAkku, enDEC, enSTW, loadIR, vom_Befehle-decoder
- wire segments 300 -> 303

Commit message: Annotierung und Footprints
Parts:
- removed R? (x15): R, symbol R
- added D23, D24, D25, D26, D27, D28, D29, D30, D31, D32, D33, D34, D35, D36, D37, D38, D39, D40, D41, D42, D43, D44, D45, D46, D47, D48, D49, D50, D51, D52, D53, D54, D55, D56, D57, D58, D59, D60, D61: Led_Small, symbol Led_Small
- added R20, R21, R23, R25, R26, R28, R30, R32, R33, R34, R35, R36, R37, R38, R39: R, symbol R
- D10, D11, D12, D14, D15, D16, D17, D18, D19, D2, D20, D21, D22, D3, D4, D5, D6, D7, D8, D9: renamed from D?; footprint (none) -> LEDs:LED-3MM
- R10, R11, R13, R14, R15, R17, R19, R2, R22, R24, R27, R29, R3, R31, R4, R5, R6, R7, R8, R9: renamed from R?; footprint (none) -> Resistors_ThroughHole:Resistor_Horizontal_RM10mm
- gave numbers to parts that had none: 40
Connections:
- wire segments 303 -> 269
- no-connect marks 0 -> 3
Other:
- note removed: "138"
- note removed: "161"
- note removed: "374"

Commit message: Steuerwerk: Footprints
Parts:
- D13, D23, D24, D25, D26, D27, D28, D31, D32, D33, D34, D35, D36, D37, D38, D39, D40, D41, D42, D43, D44, D45, D46, D47, D48, D49, D50, D51, D52, D53, D54, D55, D56, D57, D58, D59, D60, D61: footprint (none) -> LEDs:LED-3MM
- R1, R12, R18, R20, R21, R23, R25, R26, R28, R30, R32, R33, R34, R35, R36, R37, R38, R39: footprint (none) -> Resistors_ThroughHole:Resistor_Horizontal_RM10mm

Commit message: Footprints Steuerwerk
Parts:
- P10: footprint (none) -> Connect:1pin
Changed lines of the file:
@@
 F 0 "P10" H 700 2250 50  0000 C CNN
 F 1 "CONN_01X01" V 800 2150 50  0000 C CNN
-F 2 "" H 700 2150 50  0001 C CNN
+F 2 "Connect:1pin" H 700 2150 50  0001 C CNN
 F 3 "" H 700 2150 50  0000 C CNN
 	1    700  2150

Commit message: neue Steuerwerk Resistoren mit dateien
Parts:
- R1, R10, R11, R12, R13, R14, R15, R17, R18, R19, R2, R20, R21, R22, R23, R24, R25, R26, R27, R28, R29, R3, R30, R31, R32, R33, R34, R35, R36, R37, R38, R39, R4, R5, R6, R7, R8, R9: footprint Resistors_ThroughHole:Resistor_Horizontal_RM10mm -> Resistors_ThroughHole:R_Axial_DIN0207_L6.3mm_D2.5mm_P10.16mm_Horizontal

Commit message: Dioden und Anschlüsse
Parts:
- D1, D30: footprint (none) -> LEDs:LED_D1.8mm_W1.8mm_H2.4mm_Horizontal_O1.27mm_Z4.9mm
- D10, D11, D12, D13, D14, D15, D16, D17, D18, D19, D2, D20, D21, D22, D23, D24, D25, D26, D27, D28, D3, D31, D32, D33, D34, D35, D36, D37, D38, D39, D4, D40, D41, D42, D43, D44, D45, D46, D47, D48, D49, D5, D50, D51, D52, D53, D54, D55, D56, D57, D58, D59, D6, D60, D61, D7, D8, D9: footprint LEDs:LED-3MM -> LEDs:LED_D1.8mm_W1.8mm_H2.4mm_Horizontal_O1.27mm_Z4.9mm
- P1, P11, P12, P13, P14, P15, P16, P17, P18, P19, P2, P20, P21, P22, P23, P24, P3, P4, P5, P6, P7, P8, P9: footprint (none) -> Connect:1pin
