File: Steuerwerk.sch (KiCad schematic (older format))
At the start: 134 parts, among them P1 CONN_01X01, P10 CONN_01X01, P11 CONN_01X01, P12 CONN_01X01, P13 CONN_01X01, P14 CONN_01X01, P15 CONN_01X01, P16 CONN_01X01, P17 CONN_01X01, P18 CONN_01X01, P19 CONN_01X01, P2 CONN_01X01, P20 CONN_01X01, P21 CONN_01X01, P22 CONN_01X01, P23 CONN_01X01, P24 CONN_01X01, P3 CONN_01X01, P4 CONN_01X01, P5 CONN_01X01, P6 CONN_01X01, P7 CONN_01X01, P8 CONN_01X01, P9 CONN_01X01, Q1 Q_PNP_BCE, U1 74LS04, U2 74LS161, U3 74LS04, U4 74LS138, U5 74LS138, U6 74LS04, U7 74LS374, U8 74LS04, U9 74LS374

Commit message: fehlende Chips und Komponenten hinzugefügt
Parts:
- D29: footprint (none) -> LEDs:LED_D1.8mm_W1.8mm_H2.4mm_Horizontal_O1.27mm_Z4.9mm
- R16: footprint (none) -> Resistors_ThroughHole:R_Axial_DIN0207_L6.3mm_D2.5mm_P10.16mm_Horizontal
- U1, U3, U7, U9: footprint (none) -> Housings_DIP:DIP-20_W7.62mm_Socket_LongPads
- U2, U4, U5: footprint (none) -> Housings_DIP:DIP-16_W7.62mm_Socket_LongPads
- U6, U8: footprint (none) -> Housings_DIP:DIP-18_W7.62mm_Socket_LongPads
Changed lines of the file:
@@
 F 0 "U4" H 4150 2116 50  0000 C CNN
 F 1 "74LS138" H 4150 2025 50  0000 C CNN
-F 2 "" H 4150 1450 50  0001 C CNN
+F 2 "Housings_DIP:DIP-16_W7.62mm_Socket_LongPads" H 4150 1450 50  0001 C CNN
 F 3 "" H 4150 1450 50  0000 C CNN
 	1    4150 1450
@@
 F 0 "U5" H 4150 3466 50  0000 C CNN
 F 1 "74LS138" H 4150 3375 50  0000 C CNN
-F 2 "" H 4150 2800 50  0001 C CNN
+F 2 "Housings_DIP:DIP-16_W7.62mm_Socket_LongPads" H 4150 2800 50  0001 C CNN
 F 3 "" H 4150 2800 50  0000 C CNN
 	1    4150 2800
@@
 F 0 "U2" H 2500 1925 50  0000 C CNN
 F 1 "74LS161" H 2500 1834 50  0000 C CNN
-F 2 "" H 2500 1200 50  0001 C CNN
+F 2 "Housings_DIP:DIP-16_W7.62mm_Socket_LongPads" H 2500 1200 50  0001 C CNN
 F 3 "" H 2500 1200 50  0000 C CNN
 	1    2500 1200
@@
 F 0 "R16" H 4720 696 50  0000 L CNN
 F 1 "R" H 4720 605 50  0000 L CNN
-F 2 "" V 4580 650 50  0001 C CNN
+F 2 "Resistors_ThroughHole:R_Axial_DIN0207_L6.3mm_D2.5mm_P10.16mm_Horizontal" V 4580 650 50  0001 C CNN
 F 3 "" H 4650 650 50  0000 C CNN
 	1    4650 650
@@
 F 0 "U7" V 5904 3672 50  0000 R CNN
 F 1 "74LS374" V 5995 3672 50  0000 R CNN
-F 2 "" H 5950 4300 50  0001 C CNN
+F 2 "Housings_DIP:DIP-20_W7.62mm_Socket_LongPads" H 5950 4300 50  0001 C CNN
 F 3 "" H 5950 4300 50  0000 C CNN
 	1    5950 4300
@@
 F 0 "U1" V 2454 3778 50  0000 L CNN
 F 1 "74LS04" V 2545 3778 50  0000 L CNN
-F 2 "" H 2500 3600 50  0001 C CNN
+F 2 "Housings_DIP:DIP-20_W7.62mm_Socket_LongPads" H 2500 3600 50  0001 C CNN
 F 3 "" H 2500 3600 50  0000 C CNN
 	4    2500 3600
@@
 F 0 "U1" V 2754 3778 50  0000 L CNN
 F 1 "74LS04" V 2845 3778 50  0000 L CNN
-F 2 "" H 2800 3600 50  0001 C CNN
+F 2 "Housings_DIP:DIP-20_W7.62mm_Socket_LongPads" H 2800 3600 50  0001 C CNN
 F 3 "" H 2800 3600 50  0000 C CNN
 	6    2800 3600
@@
 F 0 "U3" V 3054 3778 50  0000 L CNN
 F 1 "74LS04" V 3145 3778 50  0000 L CNN
-F 2 "" H 3100 3600 50  0001 C CNN
+F 2 "Housings_DIP:DIP-20_W7.62mm_Socket_LongPads" H 3100 3600 50  0001 C CNN
 F 3 "" H 3100 3600 50  0000 C CNN
 	2    3100 3600
@@
 F 0 "U3" V 3354 3778 50  0000 L CNN
 F 1 "74LS04" V 3445 3778 50  0000 L CNN
-F 2 "" H 3400 3600 50  0001 C CNN
+F 2 "Housings_DIP:DIP-20_W7.62mm_Socket_LongPads" H 3400 3600 50  0001 C CNN
 F 3 "" H 3400 3600 50  0000 C CNN
 	4    3400 3600
@@
 F 0 "U1" V 2054 6178 50  0000 L CNN
 F 1 "74LS04" V 2145 6178 50  0000 L CNN
-F 2 "" H 2100 6000 50  0001 C CNN
+F 2 "Housings_DIP:DIP-20_W7.62mm_Socket_LongPads" H 2100 6000 50  0001 C CNN
 F 3 "" H 2100 6000 50  0000 C CNN
 	2    2100 6000
@@
 F 0 "U1" V 2354 6178 50  0000 L CNN
 F 1 "74LS04" V 2445 6178 50  0000 L CNN
-F 2 "" H 2400 6000 50  0001 C CNN
+F 2 "Housings_DIP:DIP-20_W7.62mm_Socket_LongPads" H 2400 6000 50  0001 C CNN
 F 3 "" H 2400 6000 50  0000 C CNN
 	3    2400 6000
@@
 F 0 "U1" V 2654 6178 50  0000 L CNN
 F 1 "74LS04" V 2745 6178 50  0000 L CNN
-F 2 "" H 2700 6000 50  0001 C CNN
+F 2 "Housings_DIP:DIP-20_W7.62mm_Socket_LongPads" H 2700 6000 50  0001 C CNN
 F 3 "" H 2700 6000 50  0000 C CNN
 	5    2700 6000
@@
 F 0 "U3" V 2954 6178 50  0000 L CNN
 F 1 "74LS04" V 3045 6178 50  0000 L CNN
-F 2 "" H 3000 6000 50  0001 C CNN
+F 2 "Housings_DIP:DIP-20_W7.62mm_Socket_LongPads" H 3000 6000 50  0001 C CNN
 F 3 "" H 3000 6000 50  0000 C CNN
 	1    3000 6000
@@
 F 0 "U3" V 3254 6178 50  0000 L CNN
 F 1 "74LS04" V 3345 6178 50  0000 L CNN
-F 2 "" H 3300 6000 50  0001 C CNN
+F 2 "Housings_DIP:DIP-20_W7.62mm_Socket_LongPads" H 3300 6000 50  0001 C CNN
 F 3 "" H 3300 6000 50  0000 C CNN
 	3    3300 6000
@@
 F 0 "U3" V 3554 6178 50  0000 L CNN
 F 1 "74LS04" V 3645 6178 50  0000 L CNN
-F 2 "" H 3600 6000 50  0001 C CNN
+F 2 "Housings_DIP:DIP-20_W7.62mm_Socket_LongPads" H 3600 6000 50  0001 C CNN
 F 3 "" H 3600 6000 50  0000 C CNN
 	5    3600 6000
@@
 F 0 "U3" V 3854 6178 50  0000 L CNN
 F 1 "74LS04" V 3945 6178 50  0000 L CNN
-F 2 "" H 3900 6000 50  0001 C CNN
+F 2 "Housings_DIP:DIP-20_W7.62mm_Socket_LongPads" H 3900 6000 50  0001 C CNN
 F 3 "" H 3900 6000 50  0000 C CNN
 	6    3900 6000
@@
 F 0 "U6" V 4154 6178 50  0000 L CNN
 F 1 "74LS04" V 4245 6178 50  0000 L CNN
-F 2 "" H 4200 6000 50  0001 C CNN
+F 2 "Housings_DIP:DIP-18_W7.62mm_Socket_LongPads" H 4200 6000 50  0001 C CNN
 F 3 "" H 4200 6000 50  0000 C CNN
 	1    4200 6000
@@
 F 0 "U6" V 4454 6178 50  0000 L CNN
 F 1 "74LS04" V 4545 6178 50  0000 L CNN
-F 2 "" H 4500 6000 50  0001 C CNN
+F 2 "Housings_DIP:DIP-18_W7.62mm_Socket_LongPads" H 4500 6000 50  0001 C CNN
 F 3 "" H 4500 6000 50  0000 C CNN
 	2    4500 6000
@@
 F 0 "U6" V 4754 6178 50  0000 L CNN
 F 1 "74LS04" V 4845 6178 50  0000 L CNN
-F 2 "" H 4800 6000 50  0001 C CNN
+F 2 "Housings_DIP:DIP-18_W7.62mm_Socket_LongPads" H 4800 6000 50  0001 C CNN
 F 3 "" H 4800 6000 50  0000 C CNN
 	3    4800 6000
@@
 F 0 "U6" V 5054 6178 50  0000 L CNN
 F 1 "74LS04" V 5145 6178 50  0000 L CNN
-F 2 "" H 5100 6000 50  0001 C CNN
+F 2 "Housings_DIP:DIP-18_W7.62mm_Socket_LongPads" H 5100 6000 50  0001 C CNN
 F 3 "" H 5100 6000 50  0000 C CNN
 	4    5100 6000
@@
 F 0 "U6" V 5354 6178 50  0000 L CNN
 F 1 "74LS04" V 5445 6178 50  0000 L CNN
-F 2 "" H 5400 6000 50  0001 C CNN
+F 2 "Housings_DIP:DIP-18_W7.62mm_Socket_LongPads" H 5400 6000 50  0001 C CNN
 F 3 "" H 5400 6000 50  0000 C CNN
 	5    5400 6000
@@
 F 0 "U6" V 5654 6178 50  0000 L CNN
 F 1 "74LS04" V 5745 6178 50  0000 L CNN
-F 2 "" H 5700 6000 50  0001 C CNN
+F 2 "Housings_DIP:DIP-18_W7.62mm_Socket_LongPads" H 5700 6000 50  0001 C CNN
 F 3 "" H 5700 6000 50  0000 C CNN
 	6    5700 6000
@@
 F 0 "U8" V 5954 6178 50  0000 L CNN
 F 1 "74LS04" V 6045 6178 50  0000 L CNN
-F 2 "" H 6000 6000 50  0001 C CNN
+F 2 "Housings_DIP:DIP-18_W7.62mm_Socket_LongPads" H 6000 6000 50  0001 C CNN
 F 3 "" H 6000 6000 50  0000 C CNN
 	1    6000 6000
@@
 F 0 "U8" V 6254 6178 50  0000 L CNN
 F 1 "74LS04" V 6345 6178 50  0000 L CNN
-F 2 "" H 6300 6000 50  0001 C CNN
+F 2 "Housings_DIP:DIP-18_W7.62mm_Socket_LongPads" H 6300 6000 50  0001 C CNN
 F 3 "" H 6300 6000 50  0000 C CNN
 	2    6300 6000
@@
 F 0 "U8" V 6554 6178 50  0000 L CNN
 F 1 "74LS04" V 6645 6178 50  0000 L CNN
-F 2 "" H 6600 6000 50  0001 C CNN
+F 2 "Housings_DIP:DIP-18_W7.62mm_Socket_LongPads" H 6600 6000 50  0001 C CNN
 F 3 "" H 6600 6000 50  0000 C CNN
 	3    6600 6000
@@
 F 0 "U1" V 1254 6328 50  0000 L CNN
 F 1 "74LS04" V 1345 6328 50  0000 L CNN
-F 2 "" H 1300 6150 50  0001 C CNN
+F 2 "Housings_DIP:DIP-20_W7.62mm_Socket_LongPads" H 1300 6150 50  0001 C CNN
 F 3 "" H 1300 6150 50  0000 C CNN
 	1    1300 6150
@@
 F 0 "D29" H 5300 1375 50  0000 L CNN
 F 1 "Led_Small" H 5175 1150 50  0000 L CNN
-F 2 "" V 5350 1250 50  0001 C CNN
+F 2 "LEDs:LED_D1.8mm_W1.8mm_H2.4mm_Horizontal_O1.27mm_Z4.9mm" V 5350 1250 50  0001 C CNN
 F 3 "" V 5350 1250 50  0000 C CNN
 	1    5350 1250
@@
 F 0 "U9" V 7704 3622 50  0000 R CNN
 F 1 "74LS374" V 7795 3622 50  0000 R CNN
-F 2 "" H 7750 4250 50  0001 C CNN
+F 2 "Housings_DIP:DIP-20_W7.62mm_Socket_LongPads" H 7750 4250 50  0001 C CNN
 F 3 "" H 7750 4250 50  0000 C CNN
 	1    7750 4250

Commit message: speichermodul to new version
Parts:
- added P? (x2): CONN_01X01, Connect:1pin, symbol conn:Conn_01x01
- D1, D11, D12, D14, D15, D16, D17, D18, D19, D2, D20, D21, D22, D3, D5, D7, D9: symbol LED -> device:LED_Small
- D10, D13, D4, D6, D8: symbol LED -> device:LED
- D23, D24, D25, D26, D27, D28, D29, D30, D31, D32, D33, D34, D35, D36, D37, D38, D39, D40, D41, D42, D43, D44, D45, D46, D47, D48, D49, D50, D51, D52, D53, D54, D55, D56, D57, D58, D59, D60, D61: symbol Led_Small -> device:LED_Small
- P1, P10, P11, P12, P13, P14, P15, P16, P17, P18, P19, P2, P20, P21, P22, P23, P24, P3, P4, P5, P6, P7, P8, P9: symbol CONN_01X01 -> conn:Conn_01x01
- Q1: symbol Q_PNP_BCE -> device:Q_PNP_BCE
- R1, R10, R11, R12, R13, R14, R15, R16, R17, R18, R19, R2, R20, R21, R22, R23, R24, R25, R26, R27, R28, R29, R3, R30, R31, R32, R33, R34, R35, R36, R37, R38, R39, R4, R5, R6, R7, R8, R9: symbol R -> device:R
- U1, U3, U6, U8: symbol 74LS04 -> 74xx:74LS04
- U2: symbol 74LS161 -> 74xx:74LS161
- U4, U5: symbol 74LS138 -> 74xx:74LS138
- U7, U9: symbol 74LS374 -> 74xx:74LS374
Connections:
- wire segments 269 -> 466

Commit message: Steuerwerk to pcb
Parts:
- gave numbers to parts that had none: 2
Changed lines of the file:
@@
 $EndComp
 $Comp
-L conn:Conn_01x01 P?
+L conn:Conn_01x01 P25
 U 1 1 5B01D923
 P 8600 6100
-F 0 "P?" H 8600 6200 50  0000 C CNN
+F 0 "P25" H 8600 6200 50  0000 C CNN
 F 1 "CONN_01X01" V 8700 6100 50  0000 C CNN
 F 2 "Connect:1pin" H 8600 6100 50  0001 C CNN
@@
 $EndComp
 $Comp
-L conn:Conn_01x01 P?
+L conn:Conn_01x01 P26
 U 1 1 5B01DA8F
 P 8900 5650
-F 0 "P?" H 8900 5750 50  0000 C CNN
+F 0 "P26" H 8900 5750 50  0000 C CNN
 F 1 "CONN_01X01" V 9000 5650 50  0000 C CNN
 F 2 "Connect:1pin" H 8900 5650 50  0001 C CNN

Commit message: part changed 240 in lib added
Parts:
- removed unit 4 of U1
- removed unit 6 of U1
- removed unit 2 of U3
- removed unit 4 of U3
- added U?: 74ls240, Housings_DIP:DIP-20_W7.62mm_Socket_LongPads, symbol bonsai:74ls240
- added U? (x3): 74ls240, symbol bonsai:74ls240
- Q1: footprint (none) -> TO_SOT_Packages_THT:TO-92_Molded_Narrow
Connections:
- wire segments 466 -> 474
Changed lines of the file:
@@
 $EndComp
 $Comp
-L 74xx:74LS04 U1
-U 4 1 57EA11E0
-P 2500 3600
-F 0 "U1" V 2454 3778 50  0000 L CNN
-F 1 "74LS04" V 2545 3778 50  0000 L CNN
-F 2 "Housings_DIP:DIP-20_W7.62mm_Socket_LongPads" H 2500 3600 50  0001 C CNN
-F 3 "" H 2500 3600 50  0000 C CNN
-	4    2500 3600
-	0    1    1    0
-$EndComp
-$Comp
-L 74xx:74LS04 U1
-U 6 1 57EA12A6
-P 2800 3600
-F 0 "U1" V 2754 3778 50  0000 L CNN
-F 1 "74LS04" V 2845 3778 50  0000 L CNN
-F 2 "Housings_DIP:DIP-20_W7.62mm_Socket_LongPads" H 2800 3600 50  0001 C CNN
-F 3 "" H 2800 3600 50  0000 C CNN
-	6    2800 3600
-	0    1    1    0
-$EndComp
-$Comp
-L 74xx:74LS04 U3
-U 2 1 57EA130A
-P 3100 3600
-F 0 "U3" V 3054 3778 50  0000 L CNN
-F 1 "74LS04" V 3145 3778 50  0000 L CNN
-F 2 "Housings_DIP:DIP-20_W7.62mm_Socket_LongPads" H 3100 3600 50  0001 C CNN
-F 3 "" H 3100 3600 50  0000 C CNN
-	2    3100 3600
-	0    1    1    0
-$EndComp
-$Comp
-L 74xx:74LS04 U3
-U 4 1 57EA137D
-P 3400 3600
-F 0 "U3" V 3354 3778 50  0000 L CNN
-F 1 "74LS04" V 3445 3778 50  0000 L CNN
-F 2 "Housings_DIP:DIP-20_W7.62mm_Socket_LongPads" H 3400 3600 50  0001 C CNN
-F 3 "" H 3400 3600 50  0000 C CNN
-	4    3400 3600
-	0    1    1    0
-$EndComp
-$Comp
 L device:R R4
 U 1 1 57EA1677
@@
 $EndComp
 $Comp
-L power:VCC #PWR018
-U 1 1 57F362A5
-P 5700 7150
-F 0 "#PWR018" H 5700 7000 50  0001 C CNN
-F 1 "VCC" H 5718 7323 50  0000 C CNN
-F 2 "" H 5700 7150 50  0000 C CNN
-F 3 "" H 5700 7150 50  0000 C CNN
-	1    5700 7150
-	-1   0    0    1
-$EndComp
-$Comp
 L 74xx:74LS04 U8
 U 1 1 57F362AB
@@
 F 0 "Q1" H 4750 850 50  0000 R CNN
 F 1 "Q_PNP_BCE" H 5050 750 50  0000 R CNN
-F 2 "" H 4650 900 50  0001 C CNN
+F 2 "TO_SOT_Packages_THT:TO-92_Molded_Narrow" H 4650 900 50  0001 C CNN
 F 3 "" H 4450 800 50  0000 C CNN
 	1    4450 800
@@
 L power:GND #PWR022
 U 1 1 57FCDFA0
-P 4200 950
-F 0 "#PWR022" H 4200 700 50  0001 C CNN
-F 1 "GND" H 4200 800 50  0000 C CNN
-F 2 "" H 4200 950 50  0000 C CNN
-F 3 "" H 4200 950 50  0000 C CNN
-	1    4200 950
+P 4250 900
+F 0 "#PWR022" H 4250 650 50  0001 C CNN
+F 1 "GND" H 4250 750 50  0000 C CNN
+F 2 "" H 4250 900 50  0000 C CNN
+F 3 "" H 4250 900 50  0000 C CNN
+	1    4250 900
 	-1   0    0    1
 $EndComp
@@
 	900  800  900  1150
 Wire Wire Line
-	4200 1000 4350 1000
-Wire Wire Line
-	4200 950  4200 1000
-Wire Wire Line
 	1550 500  4500 500
 Connection ~ 4800 5350
@@
 	6000 7050 6000 7150
 Wire Wire Line
-	5700 7150 5700 7050
-Wire Wire Line
 	5400 7050 5400 7150
 Wire Wire Line
@@
 $EndComp
 Wire Wire Line
-	8900 5850 8900 5950
+	8900 5850 8900 5900
+Wire Wire Line
+	5700 7050 5700 7150
+$Comp
+L power:VCC #PWR018
+U 1 1 5A45F268
+P 5700 7150
+F 0 "#PWR018" H 5700 7000 50  0001 C CNN
+F 1 "VCC" H 5718 7323 50  0000 C CNN
+F 2 "" H 5700 7150 50  0000 C CNN
+F 3 "" H 5700 7150 50  0000 C CNN
+	1    5700 7150
+	-1   0    0    1
+$EndComp
+$Comp
+L power:VCC #PWR031
+U 1 1 5A49AF77
+P 2900 5950
+F 0 "#PWR031" H 2900 5800 50  0001 C CNN
+F 1 "VCC" H 2918 6123 50  0000 C CNN
+F 2 "" H 2900 5950 50  0001 C CNN
+F 3 "" H 2900 5950 50  0001 C CNN
+	1    2900 5950
+	-1   0    0    1
+$EndComp
+Wire Wire Line
+	4350 1000 4300 1000
+Wire Wire Line
+	4300 1000 4300 900
+Wire Wire Line
+	4300 900  4250 900
+$Comp
+L power:VCC #PWR032
+U 1 1 5A4D73FD
+P 4150 950
+F 0 "#PWR032" H 4150 800 50  0001 C CNN
+F 1 "VCC" H 4167 1123 50  0000 C CNN
+F 2 "" H 4150 950 50  0001 C CNN
+F 3 "" H 4150 950 50  0001 C CNN
+	1    4150 950
+	1    0    0    -1
+$EndComp
+Wire Wire Line
+	4150 950  4150 1000
+$Comp
+L power:VCC #PWR033
+U 1 1 5A514764
+P 5300 5950
+F 0 "#PWR033" H 5300 5800 50  0001 C CNN
+F 1 "VCC" H 5318 6123 50  0000 C CNN
+F 2 "" H 5300 5950 50  0001 C CNN
+F 3 "" H 5300 5950 50  0001 C CNN
+	1    5300 5950
+	-1   0    0    1
+$EndComp
+$Comp
+L power:PWR_FLAG #FLG01
+U 1 1 5A5164E7
+P 9000 5900
+F 0 "#FLG01" H 9000 5975 50  0001 C CNN
+F 1 "PWR_FLAG" V 9000 6028 50  0000 L CNN
+F 2 "" H 9000 5900 50  0001 C CNN
+F 3 "" H 9000 5900 50  0001 C CNN
+	1    9000 5900
+	0    1    1    0
+$EndComp
+Wire Wire Line
+	9000 5900 8900 5900
+Connection ~ 8900 5900
+Wire Wire Line
+	8900 5900 8900 5950
 Wire Wire Line
 	8600 5800 8600 5900
+$Comp
+L bonsai:74ls240 U?
+U 1 1 5A64E1D9
+P 2500 3550
+F 0 "U?" V 2454 3988 50  0000 L CNN
+F 1 "74ls240" V 2545 3988 50  0000 L CNN
+F 2 "Housings_DIP:DIP-20_W7.62mm_Socket_LongPads" H 2500 3550 50  0001 C CNN
+F 3 "" H 2500 3550 50  0001 C CNN
+	1    2500 3550
+	0    1    1    0
+$EndComp
+$Comp
+L bonsai:74ls240 U?
+U 2 1 5A73EF27
+P 2800 3550
+F 0 "U?" V 2754 3988 50  0000 L CNN
+F 1 "74ls240" V 2845 3988 50  0000 L CNN
+F 2 "" H 2800 3550 50  0001 C CNN
+F 3 "" H 2800 3550 50  0001 C CNN
+	2    2800 3550
+	0    1    1    0
+$EndComp
+$Comp
+L bonsai:74ls240 U?
+U 3 1 5A73F27C
+P 3100 3550
+F 0 "U?" V 3054 3988 50  0000 L CNN
+F 1 "74ls240" V 3145 3988 50  0000 L CNN
+F 2 "" H 3100 3550 50  0001 C CNN
+F 3 "" H 3100 3550 50  0001 C CNN
+	3    3100 3550
+	0    1    1    0
+$EndComp
+$Comp
+L bonsai:74ls240 U?
+U 4 1 5A73F5E4
+P 3400 3550
+F 0 "U?" V 3354 3988 50  0000 L CNN
+F 1 "74ls240" V 3445 3988 50  0000 L CNN
+F 2 "" H 3400 3550 50  0001 C CNN
+F 3 "" H 3400 3550 50  0001 C CNN
+	4    3400 3550
+	0    1    1    0
+$EndComp
+Wire Wire Line
+	3400 3950 3400 4050
+Wire Wire Line
+	3100 4050 3100 3950
+Wire Wire Line
+	2800 3950 2800 4050
+Wire Wire Line
+	2500 4050 2500 3950
 $EndSCHEMATC

Commit message: 74541 output series (south) corrected, tackt, enDec, enSTW, clrMPC, enAkku, laodIR checked
Parts:
- removed U1, U3: 74LS04, Housings_DIP:DIP-20_W7.62mm_Socket_LongPads, symbol 74xx:74LS04
- removed U6, U8: 74LS04, Housings_DIP:DIP-18_W7.62mm_Socket_LongPads, symbol 74xx:74LS04
- added unit 1 of U1
- added U3, U6: 74541, symbol 74540:74541
- gave numbers to parts that had none: 1
Connections:
- wire segments 474 -> 404

Commit message: Steuerwerk: some minor fixes
Connections:
- wire segments 404 -> 394

Commit message: Steuerwerk: 74ls161 (nort west) adapted labels and error corrections
Parts:
- removed U2: 74LS161, Housings_DIP:DIP-16_W7.62mm_Socket_LongPads, symbol 74xx:74LS161
- added U2: 74LS161, symbol 74ls161bonsai:74LS161
Connections:
- wire segments 394 -> 399
- no-connect marks 3 -> 2
Changed lines of the file:
@@
 $EndComp
 $Comp
-L 74xx:74LS161 U2
-U 1 1 57E937E4
-P 2500 1200
-F 0 "U2" H 2500 1925 50  0000 C CNN
-F 1 "74LS161" H 2500 1834 50  0000 C CNN
-F 2 "Housings_DIP:DIP-16_W7.62mm_Socket_LongPads" H 2500 1200 50  0001 C CNN
-F 3 "" H 2500 1200 50  0000 C CNN
-	1    2500 1200
-	1    0    0    -1
-$EndComp
-$Comp
 L device:R R16
 U 1 1 57E93BD4
@@
 Text Label 900  2150 0    60   ~ 0
 vom_Befehle-decoder
-NoConn ~ 3550 3050
-NoConn ~ 3200 1200
 $Comp
 L power:VCC #PWR025
@@
 	1400 4550 850  4550
 Wire Wire Line
-	1800 1000 900  2150
-Wire Wire Line
-	1450 900  1450 1000
-Wire Wire Line
-	1800 900  1450 900
-Wire Wire Line
-	1450 1000 900  1650
-Wire Wire Line
 	900  800  900  1150
 Wire Wire Line
@@
 	3250 900  3250 2650
 Wire Wire Line
-	3200 1000 3200 2950
+	3200 1000 3200 1800
 Wire Wire Line
 	4750 3150 11150 3150
@@
 	4950 3600 5450 3600
 Wire Wire Line
-	1600 1200 1550 500
-Wire Wire Line
-	1800 1200 1600 1200
-Wire Wire Line
 	4750 1800 7600 1800
 Wire Wire Line
@@
 	3400 900  3400 1300
 Wire Wire Line
-	3200 900  3250 900
-Wire Wire Line
 	3500 1200 3550 1200
 Wire Wire Line
 	3500 800  3500 1200
 Wire Wire Line
-	3200 800  3300 800
-Wire Wire Line
 	3550 700  3550 1100
 Wire Wire Line
-	3200 700  3350 700
-Wire Wire Line
 	7950 3350 8800 3350
 Wire Wire Line
@@
 Wire Wire Line
 	750  5650 750  5550
-Connection ~ 3350 1800
 Wire Wire Line
 	3350 1800 3350 2450
@@
 Connection ~ 4750 1700
 Wire Wire Line
-	1550 500  4650 500
-Wire Wire Line
 	3400 3500 3350 3500
 Wire Wire Line
@@
 	3350 2450 3350 3500
 Wire Wire Line
-	3550 3050 2950 3050
-Wire Wire Line
 	1800 3050 1800 4900
 Wire Wire Line
@@
 Wire Wire Line
 	2950 1700 2950 3050
-Connection ~ 2950 3050
 Wire Wire Line
 	2950 3050 1800 3050
@@
 	1    0    0    -1
 $EndComp
+$Comp
+L 74ls161bonsai:74LS161 U2
+U 1 1 5B42C8F2
+P 2500 1200
+F 0 "U2" H 2493 1925 50  0000 C CNN
+F 1 "74LS161" H 2493 1834 50  0000 C CNN
+F 2 "" H 2500 1200 50  0001 C CNN
+F 3 "" H 2500 1200 50  0001 C CNN
+	1    2500 1200
+	1    0    0    -1
+$EndComp
+Wire Wire Line
+	3100 700  3350 700
+Wire Wire Line
+	3100 800  3300 800
+Wire Wire Line
+	3100 900  3250 900
+Wire Wire Line
+	3100 1000 3200 1000
+Wire Wire Line
+	3350 1800 3200 1800
+Connection ~ 3200 1800
+Wire Wire Line
+	3200 1800 3200 2950
+Wire Wire Line
+	950  900  950  1650
+Wire Wire Line
+	950  1650 900  1650
+Wire Wire Line
+	950  900  1800 900
+Wire Wire Line
+	1800 1000 1000 1000
+Wire Wire Line
+	1000 1000 1000 2150
+Wire Wire Line
+	1000 2150 900  2150
+Wire Wire Line
+	1500 1200 1500 500
+Wire Wire Line
+	1500 1200 1800 1200
+Wire Wire Line
+	1500 500  4650 500
+Wire Wire Line
+	3550 3050 2950 3050
+Connection ~ 2950 3050
+NoConn ~ 3100 1200
 $EndSCHEMATC

Commit message: steuerwerk: .sch almost debuged
Parts:
- U2: renamed from U3; footprint (none) -> Housings_DIP:DIP-20_W7.62mm_Socket_LongPads
- U3: renamed from U2; footprint (none) -> Housings_DIP:DIP-16_W7.62mm_Socket_LongPads
- U6: footprint (none) -> Housings_DIP:DIP-20_W7.62mm_Socket_LongPads
- renumbered D23 to D17, D24 to D18, D25 to D19, D26 to D20, D27 to D21, D17 to D22, D28 to D23, D29 to D24, D30 to D25, D31 to D26, D32 to D27, D33 to D28, D18 to D29, D34 to D30, D35 to D31, D19 to D32, D36 to D33, D20 to D34, D37 to D35, D21 to D36, D38 to D37, D39 to D38, D40 to D39, D41 to D40, D22 to D41, R22 to R21, R21 to R22, R27 to R26, R26 to R27, R29 to R28, R28 to R29, R31 to R30, R30 to R31, U3 to U2, U9 to U8
