File: _saved_EinTaktReset.sch (KiCad schematic (older format))
At the start: 65 parts, among them IC1 74LS624, P1 CONN_02X10, P10 CONN_01X01, P11 CONN_01X01, P12 CONN_01X01, P13 CONN_01X01, P14 CONN_01X01, P15 CONN_01X01, P2 CONN_01X01, P3 CONN_01X01, P4 CONN_02X10, P5 CONN_01X01, P6 CONN_01X01, P7 CONN_01X01, P8 CONN_01X01, P9 CONN_01X01, SW1 SPST, SW10 SPST, SW11 SPST, SW12 SPST, SW13 SPST, SW2 SWITCH_INV, SW3 SPST, SW4 SPST, SW5 SPST, SW6 SWITCH_INV, SW7 SPST, SW8 SPST, SW9 SPST, U1 74LS132, U10 74LS00, U2 74540En, U3 74LS132, U4 74HCT541_PWR, U5 74LS32, U6 74LS00, U8 74LS32, U9 74LS32

Commit message: footprint library added
Parts:
- renumbered U3 to U1, U4 to U3, U8 to U4, U9 to U4, U5 to U4, U10 to U5, U6 to U5
Changed lines of the file:
@@
 $EndComp
 $Comp
-L 74xx:74LS32 U8
-U 1 1 57E94702
+L 74xx:74LS32 U4
+U 2 1 57E94702
 P 5550 3750
-F 0 "U8" V 5504 3979 50  0000 L CNN
+F 0 "U4" V 5504 3979 50  0000 L CNN
 F 1 "74LS32" V 5595 3979 50  0000 L CNN
 F 2 "Housings_DIP:DIP-14_W7.62mm_Socket_LongPads" H 5550 3750 50  0000 C CNN
 F 3 "" H 5550 3750 50  0000 C CNN
-	1    5550 3750
+	2    5550 3750
 	0    1    1    0
 $EndComp
@@
 $EndComp
 $Comp
-L 74xx:74LS00 U10
-U 1 1 57E954F3
+L 74xx:74LS00 U5
+U 3 1 57E954F3
 P 6250 2550
-F 0 "U10" V 6296 2301 50  0000 R CNN
+F 0 "U5" V 6296 2301 50  0000 R CNN
 F 1 "74LS00" V 6205 2301 50  0000 R CNN
 F 2 "Housings_DIP:DIP-14_W7.62mm_Socket_LongPads" H 6250 2550 60  0001 C CNN
 F 3 "" H 6250 2550 60  0001 C CNN
-	1    6250 2550
-	-1   0    0    1
-$EndComp
-$Comp
-L 74xx:74LS00 U10
-U 2 1 57E9566C
+	3    6250 2550
+	-1   0    0    1
+$EndComp
+$Comp
+L 74xx:74LS00 U5
+U 4 1 57E9566C
 P 7450 2550
-F 0 "U10" V 7496 2301 50  0000 R CNN
+F 0 "U5" V 7496 2301 50  0000 R CNN
 F 1 "74LS00" V 7405 2301 50  0000 R CNN
 F 2 "Housings_DIP:DIP-14_W7.62mm_Socket_LongPads" H 7450 2550 60  0001 C CNN
 F 3 "" H 7450 2550 60  0001 C CNN
-	2    7450 2550
+	4    7450 2550
 	-1   0    0    1
 $EndComp
@@
 $EndComp
 $Comp
-L 74xx:74LS00 U6
+L 74xx:74LS00 U5
 U 1 1 5845CB68
 P 5050 6100
-F 0 "U6" V 5096 5851 50  0000 R CNN
+F 0 "U5" V 5096 5851 50  0000 R CNN
 F 1 "74LS00" V 5005 5851 50  0000 R CNN
 F 2 "" H 5050 6100 60  0001 C CNN
@@
 $EndComp
 $Comp
-L 74xx:74LS00 U6
+L 74xx:74LS00 U5
 U 2 1 5845CDF7
 P 5850 6700
-F 0 "U6" V 5896 6451 50  0000 R CNN
+F 0 "U5" V 5896 6451 50  0000 R CNN
 F 1 "74LS00" V 5805 6451 50  0000 R CNN
 F 2 "" H 5850 6700 60  0001 C CNN
@@
 $EndComp
 $Comp
-L 74xx:74LS132 U3
+L 74xx:74LS132 U1
 U 3 1 5845E5BA
 P 2950 7000
-F 0 "U3" V 2996 6751 50  0000 R CNN
+F 0 "U1" V 2996 6751 50  0000 R CNN
 F 1 "74LS132" V 2905 6751 50  0000 R CNN
 F 2 "Housings_DIP:DIP-14_W7.62mm_Socket_LongPads" H 2950 7000 60  0001 C CNN
@@
 $EndComp
 $Comp
-L 74xx:74LS32 U9
-U 2 1 584605A7
+L 74xx:74LS32 U4
+U 3 1 584605A7
 P 5750 7900
-F 0 "U9" V 5796 7651 50  0000 R CNN
+F 0 "U4" V 5796 7651 50  0000 R CNN
 F 1 "74LS32" V 5705 7651 50  0000 R CNN
 F 2 "Housings_DIP:DIP-14_W7.62mm_Socket_LongPads" H 5750 7900 60  0000 C CNN
 F 3 "" H 5750 7900 60  0001 C CNN
-	2    5750 7900
-	0    1    1    0
-$EndComp
-$Comp
-L 74xx:74LS32 U5
+	3    5750 7900
+	0    1    1    0
+$EndComp
+$Comp
+L 74xx:74LS32 U4
 U 1 1 58460B85
 P 4800 8400
-F 0 "U5" V 4846 8151 50  0000 R CNN
+F 0 "U4" V 4846 8151 50  0000 R CNN
 F 1 "74LS32" V 4755 8151 50  0000 R CNN
 F 2 "" H 4800 8400 60  0001 C CNN
@@
 $EndComp
 $Comp
-L 74xx:74HCT541_PWR U4
+L 74xx:74HCT541_PWR U3
 U 1 1 57E935F2
 P 4750 2450
-F 0 "U4" H 4750 3378 50  0000 C CNN
+F 0 "U3" H 4750 3378 50  0000 C CNN
 F 1 "74HCT541_PWR" H 4750 3287 50  0000 C CNN
 F 2 "Housings_DIP:DIP-20_W7.62mm_Socket_LongPads" H 4750 2450 50  0000 C CNN
@@
 $Comp
 L 74xx:74LS32 U6
-U 3 1 5A32CD74
+U 1 1 5A32CD74
 P 5500 9700
 F 0 "U6" V 5546 9451 50  0000 R CNN
@@
 F 2 "Housings_DIP:DIP-14_W7.62mm_Socket_LongPads" H 5500 9700 60  0001 C CNN
 F 3 "" H 5500 9700 60  0001 C CNN
-	3    5500 9700
-	1    0    0    -1
-$EndComp
+	1    5500 9700
+	1    0    0    -1
+$EndComp
