File: EinTaktReset.sch (KiCad schematic (older format))
At the start: 64 parts

Commit message: resistors added,label and output pins added
Parts:
- removed 10k?: ., symbol R
- removed R?: 10 k, symbol R
- removed U? (x8): 74540, symbol 74540
- added P? (x11): CONN_01X01, Connect:1pin, symbol CONN_01X01
- added R?: 10k, symbol R
- added RP?: R_PACK8BUSSED, symbol R_PACK8BUSSED
- added U? (x8): 74540En, symbol 74540En
- R?: renamed from 10k?; value . -> 10k
Connections:
- net labels added: CLK, auto, clrAkku, clrMPC, clrPC, enAkku, enDEC, enSTW, loadIR
- wire segments 142 -> 165
Other:
- moved on the sheet: D?, DROT

Commit message: Eintakt.sch to new kicad version
Parts:
- added P14, P15: CONN_01X01, Connect:1pin, symbol conn:Conn_01x01
- 10k1: renamed from 10k; symbol R -> device:R
- 10k__poti1: renamed from 10k__poti; symbol R -> device:R
- 4,7k1, 4,7k2: renamed from 4,7k?; symbol R -> device:R
- 4,7k3: renamed from 4,7k; symbol R -> device:R
- C1, C2, C3, C4: renamed from C?; symbol CP -> bonsai:CP
- C5: renamed from C?; symbol C -> bonsai:C
- D1: renamed from D?; symbol D -> bonsai:D
- D2: renamed from D?; symbol LED-RESCUE-EinTaktReset -> bonsai:LED
- DROT1: renamed from DROT; symbol LED-RESCUE-EinTaktReset -> bonsai:Led_Small
- IC1: renamed from IC?; symbol 74LS624 -> 74ls624:74LS624
- P1, P2: renamed from P?; symbol CONN_02X10 -> conn:Conn_02x10_Counter_Clockwise
- P10, P11, P12, P13, P3, P4, P5, P6, P7, P8, P9: renamed from P?; symbol CONN_01X01 -> conn:Conn_01x01
- R1, R10, R11, R12, R2, R3, R4, R5, R6, R7, R8, R9: renamed from R?; symbol R -> device:R
- R150: symbol R -> device:R
- RP1: renamed from RP?; symbol R_PACK8BUSSED -> bonsai:R_PACK8BUSSED
- SW1, SW10, SW11, SW12, SW13, SW3, SW4, SW5, SW7, SW8, SW9: renamed from SW?; symbol SPST -> bonsai:SW_PUSH
- SW2, SW6: renamed from SW?; symbol SWITCH_INV -> bonsai:SWITCH_INV
- U1, U4, U5, U7: renamed from U?; symbol 4001 -> cmos4000:4001
- U2: renamed from U?; symbol 74540En -> 74540:74540En
- U3: renamed from U?; symbol 74HCT541_PWR -> 74xx:74HCT541_PWR
- U6: renamed from U?; symbol 74LS32 -> 74xx:74LS32
Connections:
- net labels added: OEB, VDD
- wire segments 165 -> 254

Commit message: Eintakt bugfixing ERC (more or less) done
Parts:
- removed 10k__poti1: ., symbol device:R
- added RV1: POT, symbol bonsai:POT
- U1: symbol cmos4000:4001 -> 74xx:74LS132
- U4: symbol cmos4000:4001 -> 74xx:74LS32
- U5, U7: symbol cmos4000:4001 -> 74xx:74LS00
Connections:
- net labels removed: OEB, VCC
- wire segments 254 -> 259

Commit message: names and footprints fixes
Parts:
- 10k1, 4,7k1, 4,7k2, 4,7k3, R1, R2, R3: footprint (none) -> Resistors_ThroughHole:R_Axial_DIN0207_L6.3mm_D2.5mm_P10.16mm_Horizontal
- P1: footprint (none) -> Connect:IDC_Header_Straight_20pins
- P4: renamed from P2; footprint (none) -> Connect:IDC_Header_Straight_20pins
- R10: renamed from R9; footprint (none) -> Resistors_ThroughHole:R_Axial_DIN0207_L6.3mm_D2.5mm_P10.16mm_Horizontal
- R11: renamed from R10; footprint (none) -> Resistors_ThroughHole:R_Axial_DIN0207_L6.3mm_D2.5mm_P10.16mm_Horizontal
- R12: renamed from R11; footprint (none) -> Resistors_ThroughHole:R_Axial_DIN0207_L6.3mm_D2.5mm_P10.16mm_Horizontal
- R13: renamed from R12; footprint (none) -> Resistors_ThroughHole:R_Axial_DIN0207_L6.3mm_D2.5mm_P10.16mm_Horizontal
- R4: renamed from R150; footprint (none) -> Resistors_ThroughHole:R_Axial_DIN0207_L6.3mm_D2.5mm_P10.16mm_Horizontal
- R5: renamed from R4; footprint (none) -> Resistors_ThroughHole:R_Axial_DIN0207_L6.3mm_D2.5mm_P10.16mm_Horizontal
- R6: renamed from R5; footprint (none) -> Resistors_ThroughHole:R_Axial_DIN0207_L6.3mm_D2.5mm_P10.16mm_Horizontal
- R7: renamed from R6; footprint (none) -> Resistors_ThroughHole:R_Axial_DIN0207_L6.3mm_D2.5mm_P10.16mm_Horizontal
- R8: renamed from R7; footprint (none) -> Resistors_ThroughHole:R_Axial_DIN0207_L6.3mm_D2.5mm_P10.16mm_Horizontal
- R9: renamed from R8; footprint (none) -> Resistors_ThroughHole:R_Axial_DIN0207_L6.3mm_D2.5mm_P10.16mm_Horizontal
- RP1: footprint (none) -> Housings_SIP:SIP9_Housing_BigPads
- U1: value AND -> 74LS132
- U2, U3: footprint (none) -> Housings_DIP:DIP-20_W7.62mm_Socket_LongPads
- U4: value >=1 -> 74LS32
- U5: value AND -> 74LS00
- U6: renamed from U4; value >=1 -> 74LS132
- U8: renamed from U7; value 4001 -> 74LS00
- renumbered P8 to P10, P9 to P11, P10 to P12, P11 to P13, P12 to P14, P13 to P15, P14 to P2, P15 to P3, P3 to P5, P4 to P6, P5 to P7, P6 to P8, P7 to P9, U6 to U7

Commit message: EinTaktReset checked, no ? found
Connections:
- wire segments 259 -> 258
Changed lines of the file:
@@
 	4850 7300 5650 7300
-Wire Wire Line
-	5850 7300 5650 7300
-Connection ~ 5850 7300
-Connection ~ 5650 7300
 Wire Wire Line
 	3250 5450 3400 5450

Commit message: foodprinting EintaktReset
Parts:
- C3, C4: footprint (none) -> Capacitors_ThroughHole:CP_Radial_D8.0mm_P3.50mm
- C5: footprint (none) -> Capacitors_ThroughHole:C_Disc_D3.0mm_W1.6mm_P2.50mm
- D2: footprint (none) -> LEDs:LED_D5.0mm
- DROT1: footprint LEDs:LED-3MM -> LEDs:LED_D3.0mm
- P1, P4: footprint Connect:IDC_Header_Straight_20pins -> Pin_Headers:Pin_Header_Straight_2x10_Pitch2.00mm
- RV1: footprint (none) -> Potentiometers:Potentiometer_Trimmer_Piher_PT-10v5_Horizontal_Px5.0mm_Py5.0mm
- SW6: footprint (none) -> Buttons_Switches_ThroughHole:SW_TH_Tactile_Omron_B3F-10xx
- U1: footprint (none) -> Housings_DIP:DIP-14_W7.62mm_Socket_LongPads
- U3: renamed from U1; footprint (none) -> Housings_DIP:DIP-14_W7.62mm_Socket_LongPads
- U6: renamed from U4; footprint (none) -> Housings_DIP:DIP-14_W7.62mm_Socket_LongPads
- U8: renamed from U7; footprint (none) -> Housings_DIP:DIP-14_W7.62mm_Socket_LongPads
- U9: renamed from U8; footprint (none) -> Housings_DIP:DIP-14_W7.62mm_Socket_LongPads
- renumbered U3 to U4, U4 to U5, U5 to U6, U6 to U7
Changed lines of the file:
@@
 $EndComp
 $Comp
-L 74xx:74LS32 U7
+L 74xx:74LS32 U8
 U 1 1 57E94702
 P 5550 3750
-F 0 "U7" V 5504 3979 50  0000 L CNN
+F 0 "U8" V 5504 3979 50  0000 L CNN
 F 1 "74LS32" V 5595 3979 50  0000 L CNN
-F 2 "" H 5550 3750 50  0000 C CNN
+F 2 "Housings_DIP:DIP-14_W7.62mm_Socket_LongPads" H 5550 3750 50  0000 C CNN
 F 3 "" H 5550 3750 50  0000 C CNN
 	1    5550 3750
@@
 F 0 "D2" V 5504 4928 50  0000 L CNN
 F 1 "LED" V 5595 4928 50  0000 L CNN
-F 2 "" H 5550 4850 50  0000 C CNN
+F 2 "LEDs:LED_D5.0mm" H 5550 4850 50  0000 C CNN
 F 3 "" H 5550 4850 50  0000 C CNN
 	1    5550 4850
@@
 $EndComp
 $Comp
-L 74xx:74LS00 U8
+L 74xx:74LS00 U9
 U 1 1 57E954F3
 P 6250 2550
-F 0 "U8" V 6296 2301 50  0000 R CNN
+F 0 "U9" V 6296 2301 50  0000 R CNN
 F 1 "74LS00" V 6205 2301 50  0000 R CNN
-F 2 "" H 6250 2550 60  0001 C CNN
+F 2 "Housings_DIP:DIP-14_W7.62mm_Socket_LongPads" H 6250 2550 60  0001 C CNN
 F 3 "" H 6250 2550 60  0001 C CNN
 	1    6250 2550
@@
 $EndComp
 $Comp
-L 74xx:74LS00 U8
+L 74xx:74LS00 U9
 U 2 1 57E9566C
 P 7450 2550
-F 0 "U8" V 7496 2301 50  0000 R CNN
+F 0 "U9" V 7496 2301 50  0000 R CNN
 F 1 "74LS00" V 7405 2301 50  0000 R CNN
-F 2 "" H 7450 2550 60  0001 C CNN
+F 2 "Housings_DIP:DIP-14_W7.62mm_Socket_LongPads" H 7450 2550 60  0001 C CNN
 F 3 "" H 7450 2550 60  0001 C CNN
 	2    7450 2550
@@
 F 0 "C4" H 3918 4696 50  0000 L CNN
 F 1 "220µ" H 3918 4605 50  0000 L CNN
-F 2 "" H 3838 4500 50  0000 C CNN
+F 2 "Capacitors_ThroughHole:CP_Radial_D8.0mm_P3.50mm" H 3838 4500 50  0000 C CNN
 F 3 "" H 3800 4650 50  0000 C CNN
 	1    3800 4650
@@
 F 0 "C3" H 3382 4604 50  0000 R CNN
 F 1 "220 µ" H 3382 4695 50  0000 R CNN
-F 2 "" H 3538 4500 50  0000 C CNN
+F 2 "Capacitors_ThroughHole:CP_Radial_D8.0mm_P3.50mm" H 3538 4500 50  0000 C CNN
 F 3 "" H 3500 4650 50  0000 C CNN
 	1    3500 4650
@@
 F 0 "C5" V 3548 4950 50  0000 C CNN
 F 1 "10n" V 3639 4950 50  0000 C CNN
-F 2 "" H 3838 4800 50  0000 C CNN
+F 2 "Capacitors_ThroughHole:C_Disc_D3.0mm_W1.6mm_P2.50mm" H 3838 4800 50  0000 C CNN
 F 3 "" H 3800 4950 50  0000 C CNN
 	1    3800 4950
@@
 $EndComp
 $Comp
-L 74xx:74LS00 U5
+L 74xx:74LS00 U6
 U 1 1 5845CB68
 P 5050 6100
-F 0 "U5" V 5096 5851 50  0000 R CNN
+F 0 "U6" V 5096 5851 50  0000 R CNN
 F 1 "74LS00" V 5005 5851 50  0000 R CNN
 F 2 "" H 5050 6100 60  0001 C CNN
@@
 $EndComp
 $Comp
-L 74xx:74LS00 U5
+L 74xx:74LS00 U6
 U 2 1 5845CDF7
 P 5850 6700
-F 0 "U5" V 5896 6451 50  0000 R CNN
+F 0 "U6" V 5896 6451 50  0000 R CNN
 F 1 "74LS00" V 5805 6451 50  0000 R CNN
 F 2 "" H 5850 6700 60  0001 C CNN
@@
 $EndComp
 $Comp
-L 74xx:74LS132 U1
+L 74xx:74LS132 U3
 U 3 1 5845E5BA
 P 2950 7000
-F 0 "U1" V 2996 6751 50  0000 R CNN
+F 0 "U3" V 2996 6751 50  0000 R CNN
 F 1 "74LS132" V 2905 6751 50  0000 R CNN
-F 2 "" H 2950 7000 60  0001 C CNN
+F 2 "Housings_DIP:DIP-14_W7.62mm_Socket_LongPads" H 2950 7000 60  0001 C CNN
 F 3 "" H 2950 7000 60  0001 C CNN
 	3    2950 7000
@@
 F 0 "U1" V 2996 7451 50  0000 R CNN
 F 1 "74LS132" V 2905 7451 50  0000 R CNN
-F 2 "" H 2950 7700 60  0001 C CNN
+F 2 "Housings_DIP:DIP-14_W7.62mm_Socket_LongPads" H 2950 7700 60  0001 C CNN
 F 3 "" H 2950 7700 60  0001 C CNN
 	4    2950 7700
@@
 $EndComp
 $Comp
-L 74xx:74LS32 U4
+L 74xx:74LS32 U6
 U 2 1 584605A7
 P 5750 7900
-F 0 "U4" V 5796 7651 50  0000 R CNN
+F 0 "U6" V 5796 7651 50  0000 R CNN
 F 1 "74LS32" V 5705 7651 50  0000 R CNN
-F 2 "" H 5750 7900 60  0001 C CNN
+F 2 "Housings_DIP:DIP-14_W7.62mm_Socket_LongPads" H 5750 7900 60  0000 C CNN
 F 3 "" H 5750 7900 60  0001 C CNN
 	2    5750 7900
@@
 $EndComp
 $Comp
-L 74xx:74LS32 U4
+L 74xx:74LS32 U5
 U 1 1 58460B85
 P 4800 8400
-F 0 "U4" V 4846 8151 50  0000 R CNN
+F 0 "U5" V 4846 8151 50  0000 R CNN
 F 1 "74LS32" V 4755 8151 50  0000 R CNN
 F 2 "" H 4800 8400 60  0001 C CNN
@@
 F 0 "DROT1" H 3700 8705 50  0000 C CNN
 F 1 "LED" H 3700 8614 50  0000 C CNN
-F 2 "LEDs:LED-3MM" H 3700 8523 50  0000 C CNN
+F 2 "LEDs:LED_D3.0mm" H 3700 8523 50  0000 C CNN
 F 3 "" H 3700 8400 50  0000 C CNN
 	1    3700 8400
@@
 $EndComp
 $Comp
-L 74xx:74HCT541_PWR U3
+L 74xx:74HCT541_PWR U4
 U 1 1 57E935F2
 P 4750 2450
-F 0 "U3" H 4750 3378 50  0000 C CNN
+F 0 "U4" H 4750 3378 50  0000 C CNN
 F 1 "74HCT541_PWR" H 4750 3287 50  0000 C CNN
 F 2 "Housings_DIP:DIP-20_W7.62mm_Socket_LongPads" H 4750 2450 50  0000 C CNN
@@
 F 0 "P4" H 7000 2100 50  0000 C CNN
 F 1 "CONN_02X10" V 7000 1550 50  0000 C CNN
-F 2 "Connect:IDC_Header_Straight_20pins" H 7000 350 50  0000 C CNN
+F 2 "Pin_Headers:Pin_Header_Straight_2x10_Pitch2.00mm" H 7000 350 50  0000 C CNN
 F 3 "" H 7000 350 50  0000 C CNN
 	1    7000 1550
@@
 F 0 "P1" H 2550 2100 50  0000 C CNN
 F 1 "CONN_02X10" V 2550 1550 50  0000 C CNN
-F 2 "Connect:IDC_Header_Straight_20pins" H 2550 350 50  0000 C CNN
+F 2 "Pin_Headers:Pin_Header_Straight_2x10_Pitch2.00mm" H 2550 350 50  0000 C CNN
 F 3 "" H 2550 350 50  0000 C CNN
 	1    2550 1550
@@
 $EndComp
 $Comp
-L 74xx:74LS32 U6
+L 74xx:74LS32 U7
 U 3 1 5A32CD74
 P 5500 9700
-F 0 "U6" V 5546 9451 50  0000 R CNN
+F 0 "U7" V 5546 9451 50  0000 R CNN
 F 1 "74LS132" V 5455 9451 50  0000 R CNN
 F 2 "" H 5500 9700 60  0001 C CNN
@@
 F 0 "SW6" H 4250 9925 50  0000 C CNN
 F 1 "SWITCH_INV" H 4250 9834 50  0000 C CNN
-F 2 "" H 4250 9600 50  0000 C CNN
+F 2 "Buttons_Switches_ThroughHole:SW_TH_Tactile_Omron_B3F-10xx" H 4250 9600 50  0000 C CNN
 F 3 "" H 4250 9600 50  0000 C CNN
 	1    4250 9600
@@
 F 0 "RV1" V 2554 6272 50  0000 R CNN
 F 1 "POT" V 2645 6272 50  0000 R CNN
-F 2 "" H 2600 6350 60  0000 C CNN
+F 2 "Potentiometers:Potentiometer_Trimmer_Piher_PT-10v5_Horizontal_Px5.0mm_Py5.0mm" H 2600 6350 60  0000 C CNN
 F 3 "" H 2600 6350 60  0000 C CNN
 	1    2600 6350

Commit message: foodprinting EintaktReset2
Parts:
- U6: renamed from U7; footprint (none) -> Housings_DIP:DIP-14_W7.62mm_Socket_LongPads
- renumbered U9 to U10, U6 to U9
Changed lines of the file:
@@
 $EndComp
 $Comp
-L 74xx:74LS00 U9
+L 74xx:74LS00 U10
 U 1 1 57E954F3
 P 6250 2550
-F 0 "U9" V 6296 2301 50  0000 R CNN
+F 0 "U10" V 6296 2301 50  0000 R CNN
 F 1 "74LS00" V 6205 2301 50  0000 R CNN
 F 2 "Housings_DIP:DIP-14_W7.62mm_Socket_LongPads" H 6250 2550 60  0001 C CNN
@@
 $EndComp
 $Comp
-L 74xx:74LS00 U9
+L 74xx:74LS00 U10
 U 2 1 57E9566C
 P 7450 2550
-F 0 "U9" V 7496 2301 50  0000 R CNN
+F 0 "U10" V 7496 2301 50  0000 R CNN
 F 1 "74LS00" V 7405 2301 50  0000 R CNN
 F 2 "Housings_DIP:DIP-14_W7.62mm_Socket_LongPads" H 7450 2550 60  0001 C CNN
@@
 $EndComp
 $Comp
-L 74xx:74LS32 U6
+L 74xx:74LS32 U9
 U 2 1 584605A7
 P 5750 7900
-F 0 "U6" V 5796 7651 50  0000 R CNN
+F 0 "U9" V 5796 7651 50  0000 R CNN
 F 1 "74LS32" V 5705 7651 50  0000 R CNN
 F 2 "Housings_DIP:DIP-14_W7.62mm_Socket_LongPads" H 5750 7900 60  0000 C CNN
@@
 $EndComp
 $Comp
-L 74xx:74LS32 U7
+L 74xx:74LS32 U6
 U 3 1 5A32CD74
 P 5500 9700
-F 0 "U7" V 5546 9451 50  0000 R CNN
+F 0 "U6" V 5546 9451 50  0000 R CNN
 F 1 "74LS132" V 5455 9451 50  0000 R CNN
-F 2 "" H 5500 9700 60  0001 C CNN
+F 2 "Housings_DIP:DIP-14_W7.62mm_Socket_LongPads" H 5500 9700 60  0001 C CNN
 F 3 "" H 5500 9700 60  0001 C CNN
 	3    5500 9700

Commit message: footprinting EintaktReset3
Parts:
- SW10, SW11, SW12, SW13, SW5, SW7, SW8, SW9: footprint (none) -> tg_foodprint:eintakt_tg_SW_CuK_JS202011CQN_DPDT_Straight
- renumbered U3 to U1, U4 to U3, U8 to U4, U9 to U4, U5 to U4, U10 to U5, U6 to U5
Changed lines of the file:
@@
 F 0 "SW5" H 4250 4465 50  0000 C CNN
 F 1 "SPST" H 4250 4374 50  0000 C CNN
-F 2 "" H 4250 4200 50  0000 C CNN
+F 2 "tg_foodprint:eintakt_tg_SW_CuK_JS202011CQN_DPDT_Straight" H 4250 4200 50  0000 C CNN
 F 3 "" H 4250 4200 50  0000 C CNN
 	1    4250 4200
@@
 F 0 "SW7" H 4350 4465 50  0000 C CNN
 F 1 "SPST" H 4350 4374 50  0000 C CNN
-F 2 "" H 4350 4200 50  0000 C CNN
+F 2 "tg_foodprint:eintakt_tg_SW_CuK_JS202011CQN_DPDT_Straight" H 4350 4200 50  0000 C CNN
 F 3 "" H 4350 4200 50  0000 C CNN
 	1    4350 4200
@@
 F 0 "SW8" H 4450 4465 50  0000 C CNN
 F 1 "SPST" H 4450 4374 50  0000 C CNN
-F 2 "" H 4450 4200 50  0000 C CNN
+F 2 "tg_foodprint:eintakt_tg_SW_CuK_JS202011CQN_DPDT_Straight" H 4450 4200 50  0000 C CNN
 F 3 "" H 4450 4200 50  0000 C CNN
 	1    4450 4200
@@
 F 0 "SW9" H 4550 4465 50  0000 C CNN
 F 1 "SPST" H 4550 4374 50  0000 C CNN
-F 2 "" H 4550 4200 50  0000 C CNN
+F 2 "tg_foodprint:eintakt_tg_SW_CuK_JS202011CQN_DPDT_Straight" H 4550 4200 50  0000 C CNN
 F 3 "" H 4550 4200 50  0000 C CNN
 	1    4550 4200
@@
 F 0 "SW10" H 4650 4465 50  0000 C CNN
 F 1 "SPST" H 4650 4374 50  0000 C CNN
-F 2 "" H 4650 4200 50  0000 C CNN
+F 2 "tg_foodprint:eintakt_tg_SW_CuK_JS202011CQN_DPDT_Straight" H 4650 4200 50  0000 C CNN
 F 3 "" H 4650 4200 50  0000 C CNN
 	1    4650 4200
@@
 F 0 "SW11" H 4750 4465 50  0000 C CNN
 F 1 "SPST" H 4750 4374 50  0000 C CNN
-F 2 "" H 4750 4200 50  0000 C CNN
+F 2 "tg_foodprint:eintakt_tg_SW_CuK_JS202011CQN_DPDT_Straight" H 4750 4200 50  0000 C CNN
 F 3 "" H 4750 4200 50  0000 C CNN
 	1    4750 4200
@@
 F 0 "SW12" H 4850 4465 50  0000 C CNN
 F 1 "SPST" H 4850 4374 50  0000 C CNN
-F 2 "" H 4850 4200 50  0000 C CNN
+F 2 "tg_foodprint:eintakt_tg_SW_CuK_JS202011CQN_DPDT_Straight" H 4850 4200 50  0000 C CNN
 F 3 "" H 4850 4200 50  0000 C CNN
 	1    4850 4200
@@
 F 0 "SW13" H 4950 4465 50  0000 C CNN
 F 1 "SPST" H 4950 4374 50  0000 C CNN
-F 2 "" H 4950 4200 50  0000 C CNN
+F 2 "tg_foodprint:eintakt_tg_SW_CuK_JS202011CQN_DPDT_Straight" H 4950 4200 50  0000 C CNN
 F 3 "" H 4950 4200 50  0000 C CNN
 	1    4950 4200
@@
 $EndComp
 $Comp
-L 74xx:74LS32 U8
-U 1 1 57E94702
+L 74xx:74LS32 U4
+U 2 1 57E94702
 P 5550 3750
-F 0 "U8" V 5504 3979 50  0000 L CNN
+F 0 "U4" V 5504 3979 50  0000 L CNN
 F 1 "74LS32" V 5595 3979 50  0000 L CNN
 F 2 "Housings_DIP:DIP-14_W7.62mm_Socket_LongPads" H 5550 3750 50  0000 C CNN
 F 3 "" H 5550 3750 50  0000 C CNN
-	1    5550 3750
+	2    5550 3750
 	0    1    1    0
 $EndComp
@@
 $EndComp
 $Comp
-L 74xx:74LS00 U10
-U 1 1 57E954F3
+L 74xx:74LS00 U5
+U 3 1 57E954F3
 P 6250 2550
-F 0 "U10" V 6296 2301 50  0000 R CNN
+F 0 "U5" V 6296 2301 50  0000 R CNN
 F 1 "74LS00" V 6205 2301 50  0000 R CNN
 F 2 "Housings_DIP:DIP-14_W7.62mm_Socket_LongPads" H 6250 2550 60  0001 C CNN
 F 3 "" H 6250 2550 60  0001 C CNN
-	1    6250 2550
+	3    6250 2550
 	-1   0    0    1
 $EndComp
 $Comp
-L 74xx:74LS00 U10
-U 2 1 57E9566C
+L 74xx:74LS00 U5
+U 4 1 57E9566C
 P 7450 2550
-F 0 "U10" V 7496 2301 50  0000 R CNN
+F 0 "U5" V 7496 2301 50  0000 R CNN
 F 1 "74LS00" V 7405 2301 50  0000 R CNN
 F 2 "Housings_DIP:DIP-14_W7.62mm_Socket_LongPads" H 7450 2550 60  0001 C CNN
 F 3 "" H 7450 2550 60  0001 C CNN
-	2    7450 2550
+	4    7450 2550
 	-1   0    0    1
 $EndComp
@@
 $EndComp
 $Comp
-L 74xx:74LS00 U6
+L 74xx:74LS00 U5
 U 1 1 5845CB68
 P 5050 6100
-F 0 "U6" V 5096 5851 50  0000 R CNN
+F 0 "U5" V 5096 5851 50  0000 R CNN
 F 1 "74LS00" V 5005 5851 50  0000 R CNN
 F 2 "" H 5050 6100 60  0001 C CNN
@@
 $EndComp
 $Comp
-L 74xx:74LS00 U6
+L 74xx:74LS00 U5
 U 2 1 5845CDF7
 P 5850 6700
-F 0 "U6" V 5896 6451 50  0000 R CNN
+F 0 "U5" V 5896 6451 50  0000 R CNN
 F 1 "74LS00" V 5805 6451 50  0000 R CNN
 F 2 "" H 5850 6700 60  0001 C CNN
@@
 $EndComp
 $Comp
-L 74xx:74LS132 U3
+L 74xx:74LS132 U1
 U 3 1 5845E5BA
 P 2950 7000
-F 0 "U3" V 2996 6751 50  0000 R CNN
+F 0 "U1" V 2996 6751 50  0000 R CNN
 F 1 "74LS132" V 2905 6751 50  0000 R CNN
 F 2 "Housings_DIP:DIP-14_W7.62mm_Socket_LongPads" H 2950 7000 60  0001 C CNN
@@
 $EndComp
 $Comp
-L 74xx:74LS32 U9
-U 2 1 584605A7
+L 74xx:74LS32 U4
+U 3 1 584605A7
 P 5750 7900
-F 0 "U9" V 5796 7651 50  0000 R CNN
+F 0 "U4" V 5796 7651 50  0000 R CNN
 F 1 "74LS32" V 5705 7651 50  0000 R CNN
 F 2 "Housings_DIP:DIP-14_W7.62mm_Socket_LongPads" H 5750 7900 60  0000 C CNN
 F 3 "" H 5750 7900 60  0001 C CNN
-	2    5750 7900
+	3    5750 7900
 	0    1    1    0
 $EndComp
 $Comp
-L 74xx:74LS32 U5
+L 74xx:74LS32 U4
 U 1 1 58460B85
 P 4800 8400
-F 0 "U5" V 4846 8151 50  0000 R CNN
+F 0 "U4" V 4846 8151 50  0000 R CNN
 F 1 "74LS32" V 4755 8151 50  0000 R CNN
 F 2 "" H 4800 8400 60  0001 C CNN
@@
 $EndComp
 $Comp
-L 74xx:74HCT541_PWR U4
+L 74xx:74HCT541_PWR U3
 U 1 1 57E935F2
 P 4750 2450
-F 0 "U4" H 4750 3378 50  0000 C CNN
+F 0 "U3" H 4750 3378 50  0000 C CNN
 F 1 "74HCT541_PWR" H 4750 3287 50  0000 C CNN
 F 2 "Housings_DIP:DIP-20_W7.62mm_Socket_LongPads" H 4750 2450 50  0000 C CNN
@@
 $Comp
 L 74xx:74LS32 U6
-U 3 1 5A32CD74
+U 1 1 5A32CD74
 P 5500 9700
 F 0 "U6" V 5546 9451 50  0000 R CNN
@@
 F 2 "Housings_DIP:DIP-14_W7.62mm_Socket_LongPads" H 5500 9700 60  0001 C CNN
 F 3 "" H 5500 9700 60  0001 C CNN
-	3    5500 9700
-	1    0    0    -1
-$EndComp
+	1    5500 9700
+	1    0    0    -1
+$EndComp
