File: speichermodul.kicad_pcb (KiCad board)
At the start: 2 copper layers, 100 x 160 mm, 53 parts, among them IC1 6116, P7 CONN_01X01, P8 CONN_02X10, P9 CONN_02X10, U1 7400, U2 74LS08, U3 74LS08, U4 74LS14, U5 74LS540, U6 74LS540

Commit message: einige Footprints geändert
Parts:
- added R7: R, Resistors_ThroughHole:R_Axial_DIN0207_L6.3mm_D2.5mm_P10.16mm_Horizontal, F.Cu at (64.8, 101.6)
- added R8: R, Resistors_ThroughHole:R_Axial_DIN0207_L6.3mm_D2.5mm_P10.16mm_Horizontal, F.Cu at (80.0, 101.6)
- R10, R11, R12, R13, R14, R15, R16, R17, R18, R19, R20, R21, R22, R23, R4, R9: footprint Resistors_ThroughHole:R_Axial_DIN0411_L9.9mm_D3.6mm_P15.24mm_Horizontal -> Resistors_ThroughHole:R_Axial_DIN0207_L6.3mm_D2.5mm_P10.16mm_Horizontal
- moved R21 260.4 mm to (298.3, 30.8), turned to 0 degrees
- moved R17 239.2 mm to (272.8, 37.5), turned to 0 degrees
- moved R23 235.8 mm to (298.3, 37.5), turned to 0 degrees
- moved R20 233.5 mm to (285.5, 37.5), turned to 0 degrees
- moved R18 232.2 mm to (285.5, 30.8), turned to 0 degrees
- moved R16 229.9 mm to (272.8, 30.8), turned to 0 degrees
- moved R19 227.1 mm to (272.8, 44.2), turned to 0 degrees
- moved R22 216.9 mm to (285.5, 44.2), turned to 0 degrees
- moved R10 26.8 mm to (64.8, 58.4)
- moved R12 21.7 mm to (54.6, 58.4)
- moved R11 10.5 mm to (81.3, 58.4)
- moved R9 10.5 mm to (76.2, 58.4)
- moved R14 9.92 mm to (87.6, 48.3), turned to 270 degrees
- moved R15 4.58 mm to (92.7, 58.4)
- moved R13 4.58 mm to (69.8, 58.4)
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Routing:
- net Net-(D9-Pad2): track 0.00 -> 19.9 mm
Other:
- board size 100 x 160 mm -> 160 x 100 mm

Commit message: Version changegit status! footprints, pcb speichermodul
Parts:
- added C1: 0, Capacitors_ThroughHole:C_Disc_D10.0mm_W2.5mm_P5.00mm, F.Cu at (30.7, 32.1)
- added P1: CONN_3X2, Connectors_Samtec:SDL-106-X-XX_2x03, F.Cu at (151.0, 114.6)
- added P2: CONN_01X01, Pin_Headers:Pin_Header_Straight_1x01_Pitch1.27mm, F.Cu at (-23.1, 156.5)
- added P3: CONN_01X01, Pin_Headers:Pin_Header_Straight_1x01_Pitch1.27mm, F.Cu at (4.64, 142.0)
- added P4: CONN_01X01, Pin_Headers:Pin_Header_Straight_1x01_Pitch1.27mm, F.Cu at (-2.01, 152.7)
- added P5: CONN_01X01, Pin_Headers:Pin_Header_Straight_1x01_Pitch1.27mm, F.Cu at (-2.01, 158.2)
- added P6: CONN_01X01, Pin_Headers:Pin_Header_Straight_1x01_Pitch1.27mm, F.Cu at (8.20, 147.4)
- added R5: 0, Resistors_ThroughHole:R_Axial_DIN0309_L9.0mm_D3.2mm_P15.24mm_Horizontal, F.Cu at (24.1, 40.6)
- added SW1: SW_PUSH, Buttons_Switches_ThroughHole:SW_PUSH_6mm_h5mm, F.Cu at (29.4, 127.0)
- added SW2: SW_PUSH, Buttons_Switches_ThroughHole:SW_PUSH_6mm_h5mm, F.Cu at (25.3, 141.6)
- P7: footprint Housings_DIP:DIP-16_W7.62mm -> Pin_Headers:Pin_Header_Straight_1x01_Pitch1.27mm
- moved R23 254.6 mm to (61.0, 129.5), turned to 270 degrees
- moved R16 238.3 mm to (55.9, 129.5), turned to 270 degrees
- moved R22 235.5 mm to (66.0, 129.5), turned to 270 degrees
- moved R21 230.3 mm to (90.2, 129.5), turned to 270 degrees
- moved R18 230.3 mm to (77.5, 129.5), turned to 270 degrees
- moved R17 221.7 mm to (71.1, 129.5), turned to 270 degrees
- moved R20 220.6 mm to (85.1, 129.5), turned to 270 degrees
- moved R19 209.7 mm to (81.3, 129.5), turned to 270 degrees
- moved P9 142.7 mm to (120.7, 35.6), turned to 270 degrees
- moved P8 121.9 mm to (77.5, 179.1), turned to 0 degrees
- moved R7 66.3 mm to (118.1, 141.0)
- moved P7 60.2 mm to (28.5, 171.2), turned to 0 degrees
- moved R8 39.6 mm to (109.2, 128.3)
- moved IC1 2.84 mm to (102.9, 78.7)
- turned RP2 to 90 degrees
Connections:
- P8 pad 1: GND -> Net-(P8-Pad1)
- P8 pad 10: GND -> Net-(P8-Pad10)
- P8 pad 12: GND -> Net-(P8-Pad12)
- P8 pad 14: GND -> Net-(P8-Pad14)
- P8 pad 16: GND -> Net-(P8-Pad16)
- P8 pad 18: GND -> Net-(P8-Pad18)
- P8 pad 19: GND -> Net-(P8-Pad1)
- P8 pad 2: GND -> Net-(P8-Pad2)
- P8 pad 20: GND -> Net-(P8-Pad20)
- P8 pad 4: GND -> Net-(P8-Pad4)
- P8 pad 6: GND -> Net-(P8-Pad6)
- P8 pad 8: GND -> Net-(P8-Pad8)
- P9 pad 1: GND -> Net-(P9-Pad1)
- P9 pad 10: GND -> Net-(P9-Pad10)
- P9 pad 12: GND -> Net-(P9-Pad12)
- P9 pad 14: GND -> Net-(P9-Pad14)
- P9 pad 16: GND -> Net-(P9-Pad16)
- P9 pad 18: GND -> Net-(P9-Pad18)
- P9 pad 19: GND -> Net-(P9-Pad1)
- P9 pad 2: GND -> Net-(P9-Pad2)
- P9 pad 20: GND -> Net-(P9-Pad20)
- P9 pad 4: GND -> Net-(P9-Pad4)
- P9 pad 6: GND -> Net-(P9-Pad6)
- P9 pad 8: GND -> Net-(P9-Pad8)
- U1 pad 1: Net-(R1-Pad2) -> Net-(U1-Pad1)
- U1 pad 13: Net-(R2-Pad1) -> Net-(U1-Pad13)
- U5 pad 19: GND -> Net-(U5-Pad19)
- U6 pad 19: GND -> Net-(U6-Pad19)

Commit message: PCB voll überaqrbeitet
Parts:
- added RP1: R_PACK4BUSSED, Resistors_ThroughHole:R_Array_SIP5, F.Cu at (118.1, 78.7)
- moved REF** 193.9 mm to (28.0, 22.0), turned to 270 degrees
- moved P5 138.2 mm to (40.6, 26.7)
- moved P3 122.4 mm to (45.7, 26.7)
- moved R7 69.1 mm to (77.5, 85.1), turned to 270 degrees
- moved R1 63.1 mm to (53.3, 85.1), turned to 270 degrees
- moved R8 58.4 mm to (69.8, 85.1), turned to 270 degrees
- moved P2 57.9 mm to (34.0, 166.0)
- moved P1 46.2 mm to (121.9, 78.7)
- moved P4 36.2 mm to (34.0, 156.0)
- moved P6 35.0 mm to (34.0, 171.0)
- moved RP2 33.6 mm to (92.7, 88.9)
- moved R2 31.9 mm to (54.6, 100.3), turned to 90 degrees
- moved R23 31.7 mm to (92.7, 129.5)
- moved D18 30.5 mm to (90.2, 118.1)
- moved R25 26.5 mm to (64.0, 166.0), turned to 270 degrees
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Connections:
- P8 pad 1: Net-(P8-Pad1) -> GND
- P8 pad 10: Net-(P8-Pad10) -> GND
- P8 pad 12: Net-(P8-Pad12) -> GND
- P8 pad 14: Net-(P8-Pad14) -> GND
- P8 pad 16: Net-(P8-Pad16) -> GND
- P8 pad 18: Net-(P8-Pad18) -> GND
- P8 pad 19: Net-(P8-Pad1) -> GND
- P8 pad 2: Net-(P8-Pad2) -> GND
- P8 pad 20: Net-(P8-Pad20) -> GND
- P8 pad 4: Net-(P8-Pad4) -> GND
- P8 pad 6: Net-(P8-Pad6) -> GND
- P8 pad 8: Net-(P8-Pad8) -> GND
- P9 pad 1: Net-(P9-Pad1) -> GND
- P9 pad 10: Net-(P9-Pad10) -> GND
- P9 pad 12: Net-(P9-Pad12) -> GND
- P9 pad 14: Net-(P9-Pad14) -> GND
- P9 pad 16: Net-(P9-Pad16) -> GND
- P9 pad 18: Net-(P9-Pad18) -> GND
- P9 pad 19: Net-(P9-Pad1) -> GND
- P9 pad 2: Net-(P9-Pad2) -> GND
- P9 pad 20: Net-(P9-Pad20) -> GND
- P9 pad 4: Net-(P9-Pad4) -> GND
- P9 pad 6: Net-(P9-Pad6) -> GND
- P9 pad 8: Net-(P9-Pad8) -> GND
- U1 pad 1: Net-(U1-Pad1) -> Net-(R1-Pad2)
- U1 pad 13: Net-(U1-Pad13) -> Net-(R2-Pad1)
- U5 pad 19: Net-(U5-Pad19) -> GND
- U6 pad 19: Net-(U6-Pad19) -> GND
Routing:
- net GND: track 0.00 -> 4.00 mm
Other:
- board size 160 x 100 mm -> 100 x 160 mm

Commit message: Pcb layout
Parts:
- R24, R25, R3: footprint Resistors_ThroughHole:R_Axial_DIN0309_L9.0mm_D3.2mm_P15.24mm_Horizontal -> Resistors_ThroughHole:R_Axial_DIN0207_L6.3mm_D2.5mm_P10.16mm_Horizontal
- moved R25 23.5 mm to (41.0, 171.0), turned to 0 degrees
- moved R24 13.9 mm to (51.0, 161.0)
- moved R3 13.9 mm to (51.0, 166.0)
- moved P8 1.00 mm to (89.0, 175.0)
