File: Akku.sch (KiCad schematic (older format))
At the start: 51 parts, among them P1 CONN_02X10, P2 CONN_02X10, P3 CONN_02X10, SW1 SWITCH_INV, SW2 SWITCH_INV, SW3 SWITCH_INV, U1 7400, U2 7408, U3 4069, U4 74LS193, U5 74LS541, U6 74LS193, U7 74LS540

Commit message: Akku.sch fertiggestellt, Footprintfehler behoben, PCB Grundauslegung begonnen
Parts:
- added P4, P5, P6: CONN_01X01, Connect:1pin, symbol CONN_01X01
- D1, D2, D3, D7: footprint (none) -> LEDs:LED_D5.0mm_FlatTop
- R1: footprint Resistors_ThroughHole:R_Axial_DIN0207_L6.3mm_D2.5mm_P10.16mm_Horizontal -> Resistors_ThroughHole:Resistor_Horizontal_RM10mm
- R2, R22, R3, R4, R7, R8: footprint (none) -> Resistors_ThroughHole:Resistor_Horizontal_RM10mm
- U3: footprint (none) -> Housings_DIP:DIP-14_W7.62mm_LongPads
- U8: renamed from U?; footprint (none) -> Housings_DIP:DIP-14_W7.62mm_LongPads
Connections:
- net labels added: down/up/enable/load/CLR
- wire segments 148 -> 151
Other:
- note added: "Dezember 2017"
- note removed: "November 2017\n"
Changed lines of the file:
@@
 Akku/PC - Modul
 Text Notes 8150 7650 0    60   ~ 0
-November 2017\n
+Dezember 2017
 Text Notes 7050 6850 0    197  ~ 0
 Akkumulator
@@
 F 0 "R22" H 9570 4996 50  0000 L CNN
 F 1 "R" H 9570 4905 50  0000 L CNN
-F 2 "" V 9430 4950 50  0000 C CNN
+F 2 "Resistors_ThroughHole:Resistor_Horizontal_RM10mm" V 9430 4950 50  0000 C CNN
 F 3 "" H 9500 4950 50  0000 C CNN
 	1    9500 4950
@@
 F 0 "D7" H 8850 6100 50  0000 C CNN
 F 1 "LED" H 8850 5900 50  0000 C CNN
-F 2 "" H 8850 6000 50  0000 C CNN
+F 2 "LEDs:LED_D5.0mm_FlatTop" H 8850 6000 50  0000 C CNN
 F 3 "" H 8850 6000 50  0000 C CNN
 	1    8850 6000
@@
 F 0 "D3" H 5700 2100 50  0000 C CNN
 F 1 "LED" H 5700 1900 50  0000 C CNN
-F 2 "" H 5700 2000 50  0000 C CNN
+F 2 "LEDs:LED_D5.0mm_FlatTop" H 5700 2000 50  0000 C CNN
 F 3 "" H 5700 2000 50  0000 C CNN
 	1    5700 2000
@@
 F 0 "U3" V 5004 3278 50  0000 L CNN
 F 1 "4069" V 5095 3278 50  0000 L CNN
-F 2 "" H 5050 3100 60  0000 C CNN
+F 2 "Housings_DIP:DIP-14_W7.62mm_LongPads" H 5050 3100 60  0000 C CNN
 F 3 "" H 5050 3100 60  0001 C CNN
 	2    5050 3100
@@
 F 0 "R7" H 3820 2596 50  0000 L CNN
 F 1 "R" H 3820 2505 50  0000 L CNN
-F 2 "" V 3680 2550 50  0000 C CNN
+F 2 "Resistors_ThroughHole:Resistor_Horizontal_RM10mm" V 3680 2550 50  0000 C CNN
 F 3 "" H 3750 2550 50  0000 C CNN
 	1    3750 2550
@@
 F 0 "R8" H 3820 2796 50  0000 L CNN
 F 1 "R" H 3820 2705 50  0000 L CNN
-F 2 "" V 3680 2750 50  0000 C CNN
+F 2 "Resistors_ThroughHole:Resistor_Horizontal_RM10mm" V 3680 2750 50  0000 C CNN
 F 3 "" H 3750 2750 50  0000 C CNN
 	1    3750 2750
@@
 F 0 "R1" V 2080 3850 50  0000 C CNN
 F 1 "R" V 2000 3850 50  0000 C CNN
-F 2 "Resistors_ThroughHole:R_Axial_DIN0207_L6.3mm_D2.5mm_P10.16mm_Horizontal" V 1930 3850 50  0000 C CNN
+F 2 "Resistors_ThroughHole:Resistor_Horizontal_RM10mm" V 1930 3850 50  0000 C CNN
 F 3 "" H 2000 3850 50  0000 C CNN
 	1    2000 3850
@@
 F 0 "U3" V 5154 4278 50  0000 L CNN
 F 1 "4069" V 5245 4278 50  0000 L CNN
-F 2 "" H 5200 4100 60  0000 C CNN
+F 2 "Housings_DIP:DIP-14_W7.62mm_LongPads" H 5200 4100 60  0000 C CNN
 F 3 "" H 5200 4100 60  0001 C CNN
 	3    5200 4100
@@
 F 0 "D1" H 5650 3700 50  0000 C CNN
 F 1 "LED" H 5650 3500 50  0000 C CNN
-F 2 "" H 5650 3600 50  0000 C CNN
+F 2 "LEDs:LED_D5.0mm_FlatTop" H 5650 3600 50  0000 C CNN
 F 3 "" H 5650 3600 50  0000 C CNN
 	1    5650 3600
@@
 F 0 "R2" V 2080 5250 50  0000 C CNN
 F 1 "R" V 2000 5250 50  0000 C CNN
-F 2 "" V 1930 5250 50  0000 C CNN
+F 2 "Resistors_ThroughHole:Resistor_Horizontal_RM10mm" V 1930 5250 50  0000 C CNN
 F 3 "" H 2000 5250 50  0000 C CNN
 	1    2000 5250
@@
 F 0 "R3" V 2080 5700 50  0000 C CNN
 F 1 "R" V 2000 5700 50  0000 C CNN
-F 2 "" V 1930 5700 50  0000 C CNN
+F 2 "Resistors_ThroughHole:Resistor_Horizontal_RM10mm" V 1930 5700 50  0000 C CNN
 F 3 "" H 2000 5700 50  0000 C CNN
 	1    2000 5700
@@
 F 0 "R4" V 2080 7100 50  0000 C CNN
 F 1 "R" V 2000 7100 50  0000 C CNN
-F 2 "" V 1930 7100 50  0000 C CNN
+F 2 "Resistors_ThroughHole:Resistor_Horizontal_RM10mm" V 1930 7100 50  0000 C CNN
 F 3 "" H 2000 7100 50  0000 C CNN
 	1    2000 7100
@@
 F 0 "D2" H 5650 6650 50  0000 C CNN
 F 1 "LED" H 5650 6450 50  0000 C CNN
-F 2 "" H 5650 6550 50  0000 C CNN
+F 2 "LEDs:LED_D5.0mm_FlatTop" H 5650 6550 50  0000 C CNN
 F 3 "" H 5650 6550 50  0000 C CNN
 	1    5650 6550
@@
 NoConn ~ 9700 4450
 $Comp
-L 74HC14 U?
+L 74HC14 U8
 U 1 1 5A159C74
 P 4150 3100
-F 0 "U?" H 4300 3200 50  0000 C CNN
+F 0 "U8" H 4300 3200 50  0000 C CNN
 F 1 "74HC14" H 4350 3000 50  0000 C CNN
-F 2 "" H 4150 3100 50  0000 C CNN
+F 2 "Housings_DIP:DIP-14_W7.62mm_LongPads" H 4150 3100 50  0000 C CNN
 F 3 "" H 4150 3100 50  0000 C CNN
 	1    4150 3100
@@
 $EndComp
 $Comp
-L 74HC14 U?
-U 1 1 5A159ED2
+L 74HC14 U8
+U 3 1 5A159ED2
 P 5700 2650
-F 0 "U?" H 5850 2750 50  0000 C CNN
+F 0 "U8" H 5850 2750 50  0000 C CNN
 F 1 "74HC14" H 5900 2550 50  0000 C CNN
-F 2 "" H 5700 2650 50  0000 C CNN
+F 2 "Housings_DIP:DIP-14_W7.62mm_LongPads" H 5700 2650 50  0000 C CNN
 F 3 "" H 5700 2650 50  0000 C CNN
-	1    5700 2650
-	0    -1   -1   0
-$EndComp
-$Comp
-L 74HC14 U?
-U 1 1 5A15A24E
+	3    5700 2650
+	0    -1   -1   0
+$EndComp
+$Comp
+L 74HC14 U8
+U 2 1 5A15A24E
 P 5200 6050
-F 0 "U?" H 5350 6150 50  0000 C CNN
+F 0 "U8" H 5350 6150 50  0000 C CNN
 F 1 "74HC14" H 5400 5950 50  0000 C CNN
-F 2 "" H 5200 6050 50  0000 C CNN
+F 2 "Housings_DIP:DIP-14_W7.62mm_LongPads" H 5200 6050 50  0000 C CNN
 F 3 "" H 5200 6050 50  0000 C CNN
-	1    5200 6050
-	1    0    0    -1
-$EndComp
-$Comp
-L 74HC14 U?
-U 1 1 5A15A4DE
+	2    5200 6050
+	1    0    0    -1
+$EndComp
+$Comp
+L 74HC14 U8
+U 4 1 5A15A4DE
 P 8650 5250
-F 0 "U?" H 8800 5350 50  0000 C CNN
+F 0 "U8" H 8800 5350 50  0000 C CNN
 F 1 "74HC14" H 8850 5150 50  0000 C CNN
-F 2 "" H 8650 5250 50  0000 C CNN
+F 2 "Housings_DIP:DIP-14_W7.62mm_LongPads" H 8650 5250 50  0000 C CNN
 F 3 "" H 8650 5250 50  0000 C CNN
-	1    8650 5250
+	4    8650 5250
 	0    1    1    0
 $EndComp
+Text GLabel -500 7800 0    60   Input ~ 0
+down/up/enable/load/CLR
+Wire Wire Line
+	-500 7800 -300 7800
+$Comp
+L CONN_01X01 P6
+U 1 1 5A3B1529
+P -100 7800
+F 0 "P6" H -100 7900 50  0000 C CNN
+F 1 "CONN_01X01" V 0   7800 50  0000 C CNN
+F 2 "Connect:1pin" H -100 7800 50  0000 C CNN
+F 3 "" H -100 7800 50  0000 C CNN
+	1    -100 7800
+	1    0    0    -1
+$EndComp
+$Comp
+L GND #PWR021
+U 1 1 5A3B3838
+P -650 7450
+F 0 "#PWR021" H -650 7200 50  0001 C CNN
+F 1 "GND" H -650 7300 50  0000 C CNN
+F 2 "" H -650 7450 50  0000 C CNN
+F 3 "" H -650 7450 50  0000 C CNN
+	1    -650 7450
+	0    1    1    0
+$EndComp
+Wire Wire Line
+	-650 7450 -300 7450
+$Comp
+L CONN_01X01 P5
+U 1 1 5A3B3B73
+P -100 7450
+F 0 "P5" H -100 7550 50  0000 C CNN
+F 1 "CONN_01X01" V 0   7450 50  0000 C CNN
+F 2 "Connect:1pin" H -100 7450 50  0000 C CNN
+F 3 "" H -100 7450 50  0000 C CNN
+	1    -100 7450
+	1    0    0    -1
+$EndComp
+$Comp
+L VCC #PWR022
+U 1 1 5A3B485C
+P -700 7100
+F 0 "#PWR022" H -700 6950 50  0001 C CNN
+F 1 "VCC" H -700 7250 50  0000 C CNN
+F 2 "" H -700 7100 50  0000 C CNN
+F 3 "" H -700 7100 50  0000 C CNN
+	1    -700 7100
+	0    -1   -1   0
+$EndComp
+Wire Wire Line
+	-700 7100 -300 7100
+$Comp
+L CONN_01X01 P4
+U 1 1 5A3B4A7E
+P -100 7100
+F 0 "P4" H -100 7200 50  0000 C CNN
+F 1 "CONN_01X01" V 0   7100 50  0000 C CNN
+F 2 "Connect:1pin" H -100 7100 50  0000 C CNN
+F 3 "" H -100 7100 50  0000 C CNN
+	1    -100 7100
+	1    0    0    -1
+$EndComp
 $EndSCHEMATC

Commit message: Akku to new kicad version
Parts:
- D1, D10, D11, D12, D2, D3, D4, D5, D6, D7, D8, D9: symbol LED -> bonsai:LED
- P1, P2, P3: symbol CONN_02X10 -> conn:Conn_02x10_Counter_Clockwise
- P4, P5, P6: symbol CONN_01X01 -> conn:Conn_01x01
- R1, R10, R11, R12, R13, R14, R15, R16, R17, R18, R19, R2, R20, R21, R22, R3, R4, R5, R6, R7, R8, R9: symbol R -> device:R
- SW1, SW2, SW3: symbol SWITCH_INV -> bonsai:SWITCH_INV
- U1: symbol 7400 -> 74xx:7400
- U2: symbol 74LS08 -> 74xx:74LS08
- U3: symbol 4069 -> cmos4000:4069
- U4, U6: symbol 74LS193 -> 74xx:74LS193
- U5: symbol 74LS541 -> 74xx:74LS541
- U7: symbol 74LS540 -> 74xx:74LS540
- U8: symbol 74HC14 -> 74xx:74HC14
Connections:
- wire segments 151 -> 226
Other:
- moved on the sheet: U1A, U8A, U8C

Commit message: alles neu, also alles
Parts:
- added P7, P8, P9: CONN_01X01, Connect:1pin, symbol conn:Conn_01x01
- U1, U2: footprint Housings_DIP:DIP-14_W7.62mm -> Housings_DIP:DIP-14_W7.62mm_LongPads
- U3: value 4069 -> 74HC14
Connections:
- wire segments 226 -> 229
Changed lines of the file:
@@
 P 3000 3350
 F 0 "U3" V 2954 3528 50  0000 L CNN
-F 1 "4069" V 3045 3528 50  0000 L CNN
+F 1 "74HC14" V 3045 3528 50  0000 L CNN
 F 2 "Housings_DIP:DIP-14_W7.62mm_LongPads" H 3000 3350 60  0000 C CNN
 F 3 "" H 3000 3350 60  0001 C CNN
@@
 F 0 "U2" H 1950 4400 50  0000 C CNN
 F 1 "7408" H 1950 4250 50  0000 C CNN
-F 2 "Housings_DIP:DIP-14_W7.62mm" H 1950 4350 50  0000 C CNN
+F 2 "Housings_DIP:DIP-14_W7.62mm_LongPads" H 1950 4350 50  0000 C CNN
 F 3 "" H 1950 4350 50  0000 C CNN
 	1    1950 4350
@@
 F 0 "U1" H 2650 5050 50  0000 C CNN
 F 1 "7400" H 2650 4900 50  0000 C CNN
-F 2 "Housings_DIP:DIP-14_W7.62mm" H 2650 5000 50  0000 C CNN
+F 2 "Housings_DIP:DIP-14_W7.62mm_LongPads" H 2650 5000 50  0000 C CNN
 F 3 "" H 2650 5000 50  0000 C CNN
 	2    2650 5000
@@
 F 0 "U1" H 600 4500 50  0000 C CNN
 F 1 "7400" H 600 4350 50  0000 C CNN
-F 2 "Housings_DIP:DIP-14_W7.62mm" H 600 4450 50  0000 C CNN
+F 2 "Housings_DIP:DIP-14_W7.62mm_LongPads" H 600 4450 50  0000 C CNN
 F 3 "" H 600 4450 50  0000 C CNN
 	1    600  4450
@@
 P 3150 4350
 F 0 "U3" V 3104 4528 50  0000 L CNN
-F 1 "4069" V 3195 4528 50  0000 L CNN
+F 1 "74HC14" V 3195 4528 50  0000 L CNN
 F 2 "Housings_DIP:DIP-14_W7.62mm_LongPads" H 3150 4350 60  0000 C CNN
 F 3 "" H 3150 4350 60  0001 C CNN
@@
 F 0 "U1" H 2650 6000 50  0000 C CNN
 F 1 "7400" H 2650 5850 50  0000 C CNN
-F 2 "Housings_DIP:DIP-14_W7.62mm" H 2650 5950 50  0000 C CNN
+F 2 "Housings_DIP:DIP-14_W7.62mm_LongPads" H 2650 5950 50  0000 C CNN
 F 3 "" H 2650 5950 50  0000 C CNN
 	3    2650 5950
@@
 F 0 "U1" H 2650 6800 50  0000 C CNN
 F 1 "7400" H 2650 6650 50  0000 C CNN
-F 2 "Housings_DIP:DIP-14_W7.62mm" H 2650 6750 50  0000 C CNN
+F 2 "Housings_DIP:DIP-14_W7.62mm_LongPads" H 2650 6750 50  0000 C CNN
 F 3 "" H 2650 6750 50  0000 C CNN
 	4    2650 6750
@@
 F 0 "U2" H 4000 6100 50  0000 C CNN
 F 1 "7408" H 4000 5950 50  0000 C CNN
-F 2 "Housings_DIP:DIP-14_W7.62mm" H 4000 6050 50  0000 C CNN
+F 2 "Housings_DIP:DIP-14_W7.62mm_LongPads" H 4000 6050 50  0000 C CNN
 F 3 "" H 4000 6050 50  0000 C CNN
 	4    4000 6050
@@
 	1    0    0    -1
 $EndComp
-$Comp
-L power:VCC #PWR022
-U 1 1 5A3B485C
-P -700 7100
-F 0 "#PWR022" H -700 6950 50  0001 C CNN
-F 1 "VCC" H -700 7250 50  0000 C CNN
-F 2 "" H -700 7100 50  0000 C CNN
-F 3 "" H -700 7100 50  0000 C CNN
-	1    -700 7100
-	0    -1   -1   0
-$EndComp
 Wire Wire Line
 	-700 7100 -300 7100
@@
 Wire Wire Line
 	5250 3550 5250 3400
+Text GLabel -700 7100 0    60   Input ~ 0
+down/up/enable/load/CLR
+$Comp
+L conn:Conn_01x01 P9
+U 1 1 5A616C3E
+P -100 6800
+F 0 "P9" H -100 6900 50  0000 C CNN
+F 1 "CONN_01X01" V 0   6800 50  0000 C CNN
+F 2 "Connect:1pin" H -100 6800 50  0000 C CNN
+F 3 "" H -100 6800 50  0000 C CNN
+	1    -100 6800
+	1    0    0    -1
+$EndComp
+$Comp
+L conn:Conn_01x01 P8
+U 1 1 5A616D5C
+P -100 6450
+F 0 "P8" H -100 6550 50  0000 C CNN
+F 1 "CONN_01X01" V 0   6450 50  0000 C CNN
+F 2 "Connect:1pin" H -100 6450 50  0000 C CNN
+F 3 "" H -100 6450 50  0000 C CNN
+	1    -100 6450
+	1    0    0    -1
+$EndComp
+$Comp
+L conn:Conn_01x01 P7
+U 1 1 5A616F2D
+P -100 6100
+F 0 "P7" H -100 6200 50  0000 C CNN
+F 1 "CONN_01X01" V 0   6100 50  0000 C CNN
+F 2 "Connect:1pin" H -100 6100 50  0000 C CNN
+F 3 "" H -100 6100 50  0000 C CNN
+	1    -100 6100
+	1    0    0    -1
+$EndComp
+Text GLabel -650 6800 0    60   Input ~ 0
+down/up/enable/load/CLR
+Text GLabel -600 6450 0    60   Input ~ 0
+down/up/enable/load/CLR
+Text GLabel -550 6100 0    60   Input ~ 0
+down/up/enable/load/CLR
+Wire Wire Line
+	-300 6100 -550 6100
+Wire Wire Line
+	-600 6450 -300 6450
+Wire Wire Line
+	-300 6800 -650 6800
 Wire Bus Line
 	450  1050 450  1750

Commit message: Akku Debug
Connections:
- wire segments 229 -> 227
Other:
- moved on the sheet: U1A
Changed lines of the file:
@@
 L 74xx:74LS08 U2
 U 1 1 580F517F
-P 1950 4350
-F 0 "U2" H 1950 4400 50  0000 C CNN
-F 1 "7408" H 1950 4250 50  0000 C CNN
-F 2 "Housings_DIP:DIP-14_W7.62mm_LongPads" H 1950 4350 50  0000 C CNN
-F 3 "" H 1950 4350 50  0000 C CNN
-	1    1950 4350
+P 4150 4050
+F 0 "U2" H 4150 4100 50  0000 C CNN
+F 1 "7408" H 4150 3950 50  0000 C CNN
+F 2 "Housings_DIP:DIP-14_W7.62mm_LongPads" H 4150 4050 50  0000 C CNN
+F 3 "" H 4150 4050 50  0000 C CNN
+	1    4150 4050
 	1    0    0    -1
 $EndComp
@@
 L 74xx:7400 U1
 U 1 1 580F5818
-P 600 4450
-F 0 "U1" H 600 4500 50  0000 C CNN
-F 1 "7400" H 600 4350 50  0000 C CNN
-F 2 "Housings_DIP:DIP-14_W7.62mm_LongPads" H 600 4450 50  0000 C CNN
-F 3 "" H 600 4450 50  0000 C CNN
-	1    600  4450
+P 2650 4200
+F 0 "U1" H 2650 4250 50  0000 C CNN
+F 1 "7400" H 2650 4100 50  0000 C CNN
+F 2 "Housings_DIP:DIP-14_W7.62mm_LongPads" H 2650 4200 50  0000 C CNN
+F 3 "" H 2650 4200 50  0000 C CNN
+	1    2650 4200
 	1    0    0    -1
 $EndComp
@@
 L device:R R1
 U 1 1 58100242
-P -50 4100
-F 0 "R1" V 30  4100 50  0000 C CNN
-F 1 "R" V -50 4100 50  0000 C CNN
-F 2 "Resistors_ThroughHole:Resistor_Horizontal_RM10mm" V -120 4100 50  0000 C CNN
-F 3 "" H -50 4100 50  0000 C CNN
-	1    -50  4100
-	1    0    0    -1
+P 1750 4100
+F 0 "R1" V 1830 4100 50  0000 C CNN
+F 1 "R" V 1750 4100 50  0000 C CNN
+F 2 "Resistors_ThroughHole:Resistor_Horizontal_RM10mm" V 1680 4100 50  0000 C CNN
+F 3 "" H 1750 4100 50  0000 C CNN
+	1    1750 4100
+	0    -1   -1   0
 $EndComp
 $Comp
 L power:VCC #PWR012
 U 1 1 581002AD
-P -50 3950
-F 0 "#PWR012" H -50 3800 50  0001 C CNN
-F 1 "VCC" H -50 4100 50  0000 C CNN
-F 2 "" H -50 3950 50  0000 C CNN
-F 3 "" H -50 3950 50  0000 C CNN
-	1    -50  3950
-	1    0    0    -1
+P 1600 4100
+F 0 "#PWR012" H 1600 3950 50  0001 C CNN
+F 1 "VCC" H 1600 4250 50  0000 C CNN
+F 2 "" H 1600 4100 50  0000 C CNN
+F 3 "" H 1600 4100 50  0000 C CNN
+	1    1600 4100
+	0    -1   -1   0
 $EndComp
 $Comp
@@
 L cmos4000:4069 U3
 U 3 1 581014B6
-P 3150 4350
-F 0 "U3" V 3104 4528 50  0000 L CNN
-F 1 "74HC14" V 3195 4528 50  0000 L CNN
-F 2 "Housings_DIP:DIP-14_W7.62mm_LongPads" H 3150 4350 60  0000 C CNN
-F 3 "" H 3150 4350 60  0001 C CNN
-	3    3150 4350
+P 5400 4050
+F 0 "U3" V 5354 4228 50  0000 L CNN
+F 1 "74HC14" V 5445 4228 50  0000 L CNN
+F 2 "Housings_DIP:DIP-14_W7.62mm_LongPads" H 5400 4050 60  0000 C CNN
+F 3 "" H 5400 4050 60  0001 C CNN
+	3    5400 4050
 	1    0    0    1
 $EndComp
@@
 L device:R R10
 U 1 1 581018B2
-P 3600 4200
-F 0 "R10" V 3680 4200 50  0000 C CNN
-F 1 "R" V 3600 4200 50  0000 C CNN
-F 2 "Resistors_ThroughHole:Resistor_Horizontal_RM10mm" V 3530 4200 50  0000 C CNN
-F 3 "" H 3600 4200 50  0000 C CNN
-	1    3600 4200
+P 5850 3900
+F 0 "R10" V 5930 3900 50  0000 C CNN
+F 1 "R" V 5850 3900 50  0000 C CNN
+F 2 "Resistors_ThroughHole:Resistor_Horizontal_RM10mm" V 5780 3900 50  0000 C CNN
+F 3 "" H 5850 3900 50  0000 C CNN
+	1    5850 3900
 	-1   0    0    1
 $EndComp
@@
 L bonsai:LED D1
 U 1 1 58101E2D
-P 3600 3850
-F 0 "D1" H 3600 3950 50  0000 C CNN
-F 1 "LED" H 3600 3750 50  0000 C CNN
-F 2 "LEDs:LED_D5.0mm_FlatTop" H 3600 3850 50  0000 C CNN
-F 3 "" H 3600 3850 50  0000 C CNN
-	1    3600 3850
+P 5850 3550
+F 0 "D1" H 5850 3650 50  0000 C CNN
+F 1 "LED" H 5850 3450 50  0000 C CNN
+F 2 "LEDs:LED_D5.0mm_FlatTop" H 5850 3550 50  0000 C CNN
+F 3 "" H 5850 3550 50  0000 C CNN
+	1    5850 3550
 	0    1    1    0
 $EndComp
@@
 L power:GND #PWR014
 U 1 1 58101F33
-P 3600 3650
-F 0 "#PWR014" H 3600 3400 50  0001 C CNN
-F 1 "GND" H 3600 3500 50  0000 C CNN
-F 2 "" H 3600 3650 50  0000 C CNN
-F 3 "" H 3600 3650 50  0000 C CNN
-	1    3600 3650
+P 5850 3350
+F 0 "#PWR014" H 5850 3100 50  0001 C CNN
+F 1 "GND" H 5850 3200 50  0000 C CNN
+F 2 "" H 5850 3350 50  0000 C CNN
+F 3 "" H 5850 3350 50  0000 C CNN
+	1    5850 3350
 	0    1    1    0
 $EndComp
@@
 	-550 3650 550  3650
 Wire Wire Line
-	1050 3650 1050 4250
-Wire Wire Line
-	1050 4250 1350 4250
-Wire Wire Line
 	4650 4450 6350 4450
-Wire Wire Line
-	2600 4600 2600 4350
-Wire Wire Line
-	2600 4600 4300 4600
-Connection ~ 2600 4350
 Connection ~ 4650 6050
 Wire Wire Line
@@
 Wire Wire Line
 	4600 6050 4650 6050
-Wire Wire Line
-	2550 4350 2600 4350
-Wire Wire Line
-	1350 4450 1200 4450
 Wire Wire Line
 	3250 5950 3400 5950
@@
 Wire Wire Line
 	2000 5400 2000 5450
-Connection ~ -50  4350
-Wire Wire Line
-	-50  4250 -50  4350
-Wire Wire Line
-	-150 4350 -150 4750
+Wire Wire Line
+	1900 4100 1900 4500
 Wire Wire Line
 	1900 5100 1900 4700
@@
 	1900 5100 2000 5100
 Wire Wire Line
-	-150 4350 -50  4350
-Wire Wire Line
 	8300 6200 9900 6200
 Wire Wire Line
-	2050 4500 3250 4700
-Wire Wire Line
-	3250 4500 2050 4700
-Wire Wire Line
-	1200 4450 1200 4750
-Wire Wire Line
 	3250 4700 3250 5000
 Wire Wire Line
-	2050 4700 2050 4900
-Wire Wire Line
-	0    4550 0    4750
+	2050 4300 2050 4500
 Connection ~ 1300 3000
 Wire Wire Line
@@
 	2600 7550 3400 7550
 Wire Wire Line
-	550  3650 1050 3650
-Wire Wire Line
-	2600 4350 2700 4350
-Wire Wire Line
 	4650 6050 4750 6050
 Wire Wire Line
@@
 	2000 5450 2000 5550
 Wire Wire Line
-	-50  4350 0    4350
-Wire Wire Line
 	1300 3000 1300 3350
 Wire Wire Line
 	1300 3350 1650 3350
 Wire Wire Line
-	3650 3350 5550 3350
+	3650 3350 4650 3350
 Wire Wire Line
 	7600 3100 7700 3100
@@
 Wire Wire Line
 	1100 2450 1350 2450
-Connection ~ 1200 4450
 Connection ~ 1450 850
 Wire Bus Line
 	1450 850  5350 850
-Wire Wire Line
-	5550 3350 5550 3550
-Wire Wire Line
-	5550 3550 5250 3550
-Wire Wire Line
-	5250 3550 5250 3400
 Text GLabel -700 7100 0    60   Input ~ 0
 down/up/enable/load/CLR
@@
 Wire Wire Line
 	-300 6800 -650 6800
+Wire Wire Line
+	3550 3950 2950 3950
+Wire Wire Line
+	4950 4050 4750 4050
+Wire Wire Line
+	2050 4500 2650 4500
+Wire Wire Line
+	2650 4500 2650 4700
+Wire Wire Line
+	2650 4700 3250 4700
+Wire Wire Line
+	3250 4200 3250 4650
+Wire Wire Line
+	3250 4650 2050 4650
+Wire Wire Line
+	2050 4650 2050 4900
+Wire Wire Line
+	3550 4150 3550 4200
+Wire Wire Line
+	3550 4200 3250 4200
+Connection ~ 3250 4200
+Connection ~ 1900 4100
+Wire Wire Line
+	2950 3950 2950 3650
+Wire Wire Line
+	1900 4100 2050 4100
+Wire Wire Line
+	550  3650 2950 3650
+Wire Wire Line
+	7600 3100 4650 3100
+Wire Wire Line
+	4650 3100 4650 3350
+Connection ~ 7600 3100
+Wire Wire Line
+	9500 2750 9600 2750
+Connection ~ 9600 2750
+Wire Bus Line
+	7400 600  5350 600
+Wire Bus Line
+	5350 600  5350 850
 Wire Bus Line
 	450  1050 450  1750

Commit message: bugfixing
Parts:
- added P10, P11: CONN_01X01, Connect:1pin, symbol conn:Conn_01x01
- SW1: value SWITCH_INV -> UP_Bonsai_SWITCH_INV
- SW2: value SWITCH_INV -> DOWN_Bonsai_SWITCH_INV
- SW3: value SWITCH_INV -> CLR_Bonsai_SWITCH_INV
- renumbered D3 to D1, D1 to D3, P8 to P1, P7 to P2, P9 to P3, P1 to P7, P2 to P8, P3 to P9, R5 to R1, R11 to R10, R10 to R11, R7 to R2, R8 to R3, R1 to R4, R2 to R5, R3 to R6, R4 to R7, R6 to R8, U8 to U1, U1 to U2, U2 to U4, U4 to U5, U5 to U6, U6 to U7, U7 to U8
Connections:
- net labels added: VDD, VSS
- net labels removed: down/up/enable/load/CLR
- wire segments 227 -> 236

Commit message: benennung der ICs
Other:
- note added: "e"
- note added: "f"
Changed lines of the file:
@@
 $Comp
 L cmos4000:4069 U3
-U 3 1 581014B6
+U 6 1 581014B6
 P 5400 4050
 F 0 "U3" V 5354 4228 50  0000 L CNN
@@
 F 2 "Housings_DIP:DIP-14_W7.62mm_LongPads" H 5400 4050 60  0000 C CNN
 F 3 "" H 5400 4050 60  0001 C CNN
-	3    5400 4050
+	6    5400 4050
 	1    0    0    1
 $EndComp
@@
 Wire Wire Line
 	4600 7150 4600 7100
+Connection ~ 4450 7150
+Text Notes 5150 5850 0    50   ~ 0
+f
 Wire Bus Line
 	450  1050 450  1750
@@
 Wire Bus Line
 	1450 850  1450 2350
-Connection ~ 4450 7150
+Text Notes 5400 3900 0    50   ~ 0
+e
 $EndSCHEMATC
