File: Akku.sch (KiCad schematic (older format))
At the start: 49 parts, among them J1 +/- Stecker, J2 load/up, J3 down/en/clear, P7 CONN_02X10, P8 CONN_02X10, P9 CONN_02X10, SW1 UP_Bonsai_SWITCH_INV, SW2 DOWN_Bonsai_SWITCH_INV, SW3 CLR_Bonsai_SWITCH_INV, U1 74HC14, U2 7400, U4 7408, U5 74LS193, U6 74LS541, U7 74LS193, U8 74LS540

Commit message: big cleanup .sch files, symbols libs, project files
Parts:
- C1, C2, C3: symbol Akku-rescue:C-bonsai-Akku-rescue -> allBonsaiSymbolLibs:C-bonsai
- D1, D10, D11, D12, D2, D3, D4, D5, D6, D7, D8, D9: symbol Akku-rescue:LED-bonsai-Akku-rescue -> allBonsaiSymbolLibs:LED-bonsai
- D13: symbol Akku-rescue:D-bonsai-Akku-rescue -> allBonsaiSymbolLibs:D-bonsai
- J1, J2: symbol Akku-rescue:2PinTerminalBlocktg-2PinTerminalBlocktg-Akku-rescue-Akku-rescue -> allBonsaiSymbolLibs:2PinTerminalBlocktg-2PinTerminalBlocktg
- J3: symbol Akku-rescue:3PinTerminalBlocktg-3PinTerminalBlocktg-Akku-rescue-Akku-rescue -> allBonsaiSymbolLibs:3PinTerminalBlocktg-3PinTerminalBlocktg
- P7, P8, P9: symbol Akku-rescue:Conn_02x10_Counter_Clockwise-conn-Akku-rescue-Akku-rescue -> allBonsaiSymbolLibs:Conn_02x10_Counter_Clockwise-conn
- R10, R11, R12, R13, R14, R15, R16, R17, R18, R19, R2, R20, R21, R3, R9: symbol Akku-rescue:R-device-Akku-rescue-Akku-rescue -> allBonsaiSymbolLibs:R-device
- RPA1, RPB1: symbol Akku-rescue:R_PACK4BUSSED-bonsai-Akku-rescue -> allBonsaiSymbolLibs:R_PACK4BUSSED
- SW1, SW2, SW3: symbol Akku-rescue:SWITCH_INV-bonsai-Akku-rescue -> allBonsaiSymbolLibs:SWITCH_INV-bonsai
- U1: symbol Akku-rescue:4069-cmos4000-Akku-rescue-Akku-rescue -> allBonsaiSymbolLibs:4069-cmos4000
- U1: symbol Akku-rescue:74HC14-RESCUE-Akku-Akku-rescue-Akku-rescue -> allBonsaiSymbolLibs:74HC14
- U2: symbol Akku-rescue:7400-RESCUE-Akku-Akku-rescue-Akku-rescue -> allBonsaiSymbolLibs:7400
- U4: symbol Akku-rescue:74LS08-74xx-Akku-rescue-Akku-rescue -> allBonsaiSymbolLibs:74LS08-74xx
- U5, U7: symbol Akku-rescue:74LS193-RESCUE-Akku-Akku-rescue-Akku-rescue -> allBonsaiSymbolLibs:74LS193
- U6: symbol Akku-rescue:74LS541-74xx-Akku-rescue-Akku-rescue -> allBonsaiSymbolLibs:74LS541-74xx
- U8: symbol Akku-rescue:74LS540-74xx-Akku-rescue-Akku-rescue -> allBonsaiSymbolLibs:74LS540-74xx
Changed lines of the file:
@@
 Akkumulator
 $Comp
-L Akku-rescue:74LS540-74xx-Akku-rescue-Akku-rescue U8
+L allBonsaiSymbolLibs:74LS540-74xx U8
 U 1 1 57E93AAD
 P 9100 2050
@@
 $EndComp
 $Comp
-L Akku-rescue:LED-bonsai-Akku-rescue D12
+L allBonsaiSymbolLibs:LED-bonsai D12
 U 1 1 57E93BF0
 P 9300 850
@@
 $EndComp
 $Comp
-L Akku-rescue:LED-bonsai-Akku-rescue D11
+L allBonsaiSymbolLibs:LED-bonsai D11
 U 1 1 57E93CED
 P 9200 850
@@
 $EndComp
 $Comp
-L Akku-rescue:LED-bonsai-Akku-rescue D10
+L allBonsaiSymbolLibs:LED-bonsai D10
 U 1 1 57E93ED1
 P 9100 850
@@
 $EndComp
 $Comp
-L Akku-rescue:LED-bonsai-Akku-rescue D9
+L allBonsaiSymbolLibs:LED-bonsai D9
 U 1 1 57E93F38
 P 9000 850
@@
 $EndComp
 $Comp
-L Akku-rescue:LED-bonsai-Akku-rescue D8
+L allBonsaiSymbolLibs:LED-bonsai D8
 U 1 1 57E93F7E
 P 8900 850
@@
 $EndComp
 $Comp
-L Akku-rescue:LED-bonsai-Akku-rescue D6
+L allBonsaiSymbolLibs:LED-bonsai D6
 U 1 1 57E93FA3
 P 8800 850
@@
 $EndComp
 $Comp
-L Akku-rescue:LED-bonsai-Akku-rescue D5
+L allBonsaiSymbolLibs:LED-bonsai D5
 U 1 1 57E93FCF
 P 8700 850
@@
 $EndComp
 $Comp
-L Akku-rescue:LED-bonsai-Akku-rescue D4
+L allBonsaiSymbolLibs:LED-bonsai D4
 U 1 1 57E93FFA
 P 8600 850
@@
 $EndComp
 $Comp
-L Akku-rescue:R-device-Akku-rescue-Akku-rescue R13
+L allBonsaiSymbolLibs:R-device R13
 U 1 1 57E94162
 P 8600 1200
@@
 $EndComp
 $Comp
-L Akku-rescue:R-device-Akku-rescue-Akku-rescue R15
+L allBonsaiSymbolLibs:R-device R15
 U 1 1 57E942DE
 P 8700 1200
@@
 $EndComp
 $Comp
-L Akku-rescue:R-device-Akku-rescue-Akku-rescue R16
+L allBonsaiSymbolLibs:R-device R16
 U 1 1 57E94316
 P 8800 1200
@@
 $EndComp
 $Comp
-L Akku-rescue:R-device-Akku-rescue-Akku-rescue R17
+L allBonsaiSymbolLibs:R-device R17
 U 1 1 57E94362
 P 8900 1200
@@
 $EndComp
 $Comp
-L Akku-rescue:R-device-Akku-rescue-Akku-rescue R18
+L allBonsaiSymbolLibs:R-device R18
 U 1 1 57E943BA
 P 9000 1200
@@
 $EndComp
 $Comp
-L Akku-rescue:R-device-Akku-rescue-Akku-rescue R19
+L allBonsaiSymbolLibs:R-device R19
 U 1 1 57E94424
 P 9100 1200
@@
 $EndComp
 $Comp
-L Akku-rescue:R-device-Akku-rescue-Akku-rescue R20
+L allBonsaiSymbolLibs:R-device R20
 U 1 1 57E94464
 P 9200 1200
@@
 $EndComp
 $Comp
-L Akku-rescue:R-device-Akku-rescue-Akku-rescue R21
+L allBonsaiSymbolLibs:R-device R21
 U 1 1 57E944B7
 P 9300 1200
@@
 $EndComp
 $Comp
-L Akku-rescue:74LS193-RESCUE-Akku-Akku-rescue-Akku-rescue U5
+L allBonsaiSymbolLibs:74LS193 U5
 U 1 1 57E9530E
 P 7050 4150
@@
 $EndComp
 $Comp
-L Akku-rescue:74LS193-RESCUE-Akku-Akku-rescue-Akku-rescue U7
+L allBonsaiSymbolLibs:74LS193 U7
 U 1 1 57E95727
 P 9000 4150
@@
 $EndComp
 $Comp
-L Akku-rescue:R-device-Akku-rescue-Akku-rescue R14
+L allBonsaiSymbolLibs:R-device R14
 U 1 1 57E98213
 P 8650 5850
@@
 $EndComp
 $Comp
-L Akku-rescue:R-device-Akku-rescue-Akku-rescue R9
+L allBonsaiSymbolLibs:R-device R9
 U 1 1 57F2FBEB
 P 3650 2250
@@
 $EndComp
 $Comp
-L Akku-rescue:LED-bonsai-Akku-rescue D7
+L allBonsaiSymbolLibs:LED-bonsai D7
 U 1 1 57FBC65C
 P 8850 6000
@@
 $EndComp
 $Comp
-L Akku-rescue:R-device-Akku-rescue-Akku-rescue R12
+L allBonsaiSymbolLibs:R-device R12
 U 1 1 57FC1E29
 P 8150 6200
@@
 $EndComp
 $Comp
-L Akku-rescue:SWITCH_INV-bonsai-Akku-rescue SW3
+L allBonsaiSymbolLibs:SWITCH_INV-bonsai SW3
 U 1 1 57FC34DF
 P 7500 6200
@@
 $EndComp
 $Comp
-L Akku-rescue:74LS541-74xx-Akku-rescue-Akku-rescue U6
+L allBonsaiSymbolLibs:74LS541-74xx U6
 U 1 1 57E939A0
 P 7200 2000
@@
 $EndComp
 $Comp
-L Akku-rescue:Conn_02x10_Counter_Clockwise-conn-Akku-rescue-Akku-rescue P7
+L allBonsaiSymbolLibs:Conn_02x10_Counter_Clockwise-conn P7
 U 1 1 58057A43
 P 4850 1600
@@
 $EndComp
 $Comp
-L Akku-rescue:Conn_02x10_Counter_Clockwise-conn-Akku-rescue-Akku-rescue P8
+L allBonsaiSymbolLibs:Conn_02x10_Counter_Clockwise-conn P8
 U 1 1 5805867B
 P 4100 1600
@@
 $EndComp
 $Comp
-L Akku-rescue:Conn_02x10_Counter_Clockwise-conn-Akku-rescue-Akku-rescue P9
+L allBonsaiSymbolLibs:Conn_02x10_Counter_Clockwise-conn P9
 U 1 1 58058F42
 P 5600 1600
@@
 $EndComp
 $Comp
-L Akku-rescue:LED-bonsai-Akku-rescue D1
+L allBonsaiSymbolLibs:LED-bonsai D1
 U 1 1 580EE5C2
 P 3450 2050
@@
 $EndComp
 $Comp
-L Akku-rescue:4069-cmos4000-Akku-rescue-Akku-rescue U1
+L allBonsaiSymbolLibs:4069-cmos4000 U1
 U 2 1 580F11C5
 P 3000 3350
@@
 $EndComp
 $Comp
-L Akku-rescue:R-device-Akku-rescue-Akku-rescue R2
+L allBonsaiSymbolLibs:R-device R2
 U 1 1 580F178A
 P 1700 2800
@@
 $EndComp
 $Comp
-L Akku-rescue:R-device-Akku-rescue-Akku-rescue R3
+L allBonsaiSymbolLibs:R-device R3
 U 1 1 580F350E
 P 1700 3000
@@
 (PC)
 $Comp
-L Akku-rescue:74LS08-74xx-Akku-rescue-Akku-rescue U4
+L allBonsaiSymbolLibs:74LS08-74xx U4
 U 4 1 580F517F
 P 4150 4050
@@
 $EndComp
 $Comp
-L Akku-rescue:7400-RESCUE-Akku-Akku-rescue-Akku-rescue U2
+L allBonsaiSymbolLibs:7400 U2
 U 4 1 580F5956
 P 2650 5000
@@
 $EndComp
 $Comp
-L Akku-rescue:7400-RESCUE-Akku-Akku-rescue-Akku-rescue U2
+L allBonsaiSymbolLibs:7400 U2
 U 1 1 580F5818
 P 2650 4200
@@
 $EndComp
 $Comp
-L Akku-rescue:SWITCH_INV-bonsai-Akku-rescue SW1
+L allBonsaiSymbolLibs:SWITCH_INV-bonsai SW1
 U 1 1 58100CBF
 P 1400 4600
@@
 $EndComp
 $Comp
-L Akku-rescue:4069-cmos4000-Akku-rescue-Akku-rescue U1
+L allBonsaiSymbolLibs:4069-cmos4000 U1
 U 5 1 581014B6
 P 5400 4050
@@
 $EndComp
 $Comp
-L Akku-rescue:R-device-Akku-rescue-Akku-rescue R11
+L allBonsaiSymbolLibs:R-device R11
 U 1 1 581018B2
 P 5850 3900
@@
 $EndComp
 $Comp
-L Akku-rescue:LED-bonsai-Akku-rescue D3
+L allBonsaiSymbolLibs:LED-bonsai D3
 U 1 1 58101E2D
 P 5850 3550
@@
 $EndComp
 $Comp
-L Akku-rescue:7400-RESCUE-Akku-Akku-rescue-Akku-rescue U2
+L allBonsaiSymbolLibs:7400 U2
 U 3 1 58103E9D
 P 2650 5950
@@
 $EndComp
 $Comp
-L Akku-rescue:7400-RESCUE-Akku-Akku-rescue-Akku-rescue U2
+L allBonsaiSymbolLibs:7400 U2
 U 2 1 58103EA3
 P 2650 6750
@@
 $EndComp
 $Comp
-L Akku-rescue:SWITCH_INV-bonsai-Akku-rescue SW2
+L allBonsaiSymbolLibs:SWITCH_INV-bonsai SW2
 U 1 1 58103EB5
 P 1400 6350
@@
 $EndComp
 $Comp
-L Akku-rescue:74LS08-74xx-Akku-rescue-Akku-rescue U4
+L allBonsaiSymbolLibs:74LS08-74xx U4
 U 1 1 581052DF
 P 4000 6050
@@
 	7300 2700 7300 3050
 $Comp
-L Akku-rescue:74HC14-RESCUE-Akku-Akku-rescue-Akku-rescue U1
+L allBonsaiSymbolLibs:74HC14 U1
 U 1 1 5A159C74
 P 2100 3350
@@
 $EndComp
 $Comp
-L Akku-rescue:74HC14-RESCUE-Akku-Akku-rescue-Akku-rescue U1
+L allBonsaiSymbolLibs:74HC14 U1
 U 3 1 5A159ED2
 P 3650 2900
@@
 $EndComp
 $Comp
-L Akku-rescue:74HC14-RESCUE-Akku-Akku-rescue-Akku-rescue U1
+L allBonsaiSymbolLibs:74HC14 U1
 U 6 1 5A15A24E
 P 5200 6050
@@
 $EndComp
 $Comp
-L Akku-rescue:74HC14-RESCUE-Akku-Akku-rescue-Akku-rescue U1
+L allBonsaiSymbolLibs:74HC14 U1
 U 4 1 5A15A4DE
 P 8650 5250
@@
 	850  1400 800  1400
 $Comp
-L Akku-rescue:2PinTerminalBlocktg-2PinTerminalBlocktg-Akku-rescue-Akku-rescue J1
+L allBonsaiSymbolLibs:2PinTerminalBlocktg-2PinTerminalBlocktg J1
 U 1 1 5AECBED9
 P 850 850
@@
 $EndComp
 $Comp
-L Akku-rescue:2PinTerminalBlocktg-2PinTerminalBlocktg-Akku-rescue-Akku-rescue J2
+L allBonsaiSymbolLibs:2PinTerminalBlocktg-2PinTerminalBlocktg J2
 U 1 1 5AECC155
 P 10650 5300
@@
 $EndComp
 $Comp
-L Akku-rescue:3PinTerminalBlocktg-3PinTerminalBlocktg-Akku-rescue-Akku-rescue J3
+L allBonsaiSymbolLibs:3PinTerminalBlocktg-3PinTerminalBlocktg J3
 U 1 1 5AECC360
 P 10650 5650
@@
 	1150 1150 1200 1150
 $Comp
-L Akku-rescue:R_PACK4BUSSED-bonsai-Akku-rescue RPA1
+L allBonsaiSymbolLibs:R_PACK4BUSSED RPA1
 U 1 1 5B220C3D
 P 2800 1000
@@
 $EndComp
 $Comp
-L Akku-rescue:R-device-Akku-rescue-Akku-rescue R10
+L allBonsaiSymbolLibs:R-device R10
 U 1 1 5810516E
 P 5650 6200
@@
 $EndComp
 $Comp
-L Akku-rescue:LED-bonsai-Akku-rescue D2
+L allBonsaiSymbolLibs:LED-bonsai D2
 U 1 1 58105174
 P 5650 6550
@@
 RPA3
 $Comp
-L Akku-rescue:R_PACK4BUSSED-bonsai-Akku-rescue RPB1
+L allBonsaiSymbolLibs:R_PACK4BUSSED RPB1
 U 1 1 5B22DE13
 P 2800 1700
@@
 Connection ~ 6000 600
 $Comp
-L Akku-rescue:C-bonsai-Akku-rescue C1
+L allBonsaiSymbolLibs:C-bonsai C1
 U 1 1 5CBF3D2E
 P 1000 1400
@@
 $EndComp
 $Comp
-L Akku-rescue:C-bonsai-Akku-rescue C2
+L allBonsaiSymbolLibs:C-bonsai C2
 U 1 1 5CBF52E5
 P 1000 1600
@@
 $EndComp
 $Comp
-L Akku-rescue:D-bonsai-Akku-rescue D13
+L allBonsaiSymbolLibs:D-bonsai D13
 U 1 1 5CC05CEA
 P 1000 1250
@@
 Connection ~ 850  1550
 $Comp
-L Akku-rescue:C-bonsai-Akku-rescue C3
+L allBonsaiSymbolLibs:C-bonsai C3
 U 1 1 5CC7F388
 P 1000 1800

Commit message: BIB Cleanup finished
Parts:
- C1, C2, C3: footprint tg_foodprint:C_Disc_D10.0mm_W2.5mm_P5.00mm -> allBonsaiFootprintsLibs:C_Disc_D10.0mm_W2.5mm_P5.00mm
- P7, P8, P9: footprint tg_foodprint:Pin_Header_Straight_2x10_Pitch2.00mmBonsai.pretty -> allBonsaiFootprintsLibs:Pin_Header_Straight_2x10_Pitch2.00mmBonsai.pretty
- SW1, SW2, SW3: footprint tg_foodprint:SW_PUSH_LCD_E3_SAxxxx_tg_V2 -> allBonsaiFootprintsLibs:SW_PUSH_LCD_E3_SAxxxx_tg_V2
Changed lines of the file:
@@
 F 0 "SW3" H 7300 6350 50  0000 C CNN
 F 1 "CLR_Bonsai_SWITCH_INV" H 7350 6050 50  0000 C CNN
-F 2 "tg_foodprint:SW_PUSH_LCD_E3_SAxxxx_tg_V2" H 7500 6200 50  0001 C CNN
+F 2 "allBonsaiFootprintsLibs:SW_PUSH_LCD_E3_SAxxxx_tg_V2" H 7500 6200 50  0001 C CNN
 F 3 "" H 7500 6200 50  0000 C CNN
 	1    7500 6200
@@
 F 0 "P7" H 4850 2150 50  0000 C CNN
 F 1 "CONN_02X10" V 4850 1600 50  0000 C CNN
-F 2 "tg_foodprint:Pin_Header_Straight_2x10_Pitch2.00mmBonsai.pretty" H 4850 1600 50  0001 C CNN
+F 2 "allBonsaiFootprintsLibs:Pin_Header_Straight_2x10_Pitch2.00mmBonsai.pretty" H 4850 1600 50  0001 C CNN
 F 3 "" H 4850 400 50  0000 C CNN
 	1    4850 1600
@@
 F 0 "P8" H 4100 2150 50  0000 C CNN
 F 1 "CONN_02X10" V 4100 1600 50  0000 C CNN
-F 2 "tg_foodprint:Pin_Header_Straight_2x10_Pitch2.00mmBonsai.pretty" H 4100 1650 50  0001 C CNN
+F 2 "allBonsaiFootprintsLibs:Pin_Header_Straight_2x10_Pitch2.00mmBonsai.pretty" H 4100 1650 50  0001 C CNN
 F 3 "" H 4100 400 50  0000 C CNN
 	1    4100 1600
@@
 F 0 "P9" H 5600 2150 50  0000 C CNN
 F 1 "CONN_02X10" V 5600 1600 50  0000 C CNN
-F 2 "tg_foodprint:Pin_Header_Straight_2x10_Pitch2.00mmBonsai.pretty" H 5600 1600 50  0001 C CNN
+F 2 "allBonsaiFootprintsLibs:Pin_Header_Straight_2x10_Pitch2.00mmBonsai.pretty" H 5600 1600 50  0001 C CNN
 F 3 "" H 5600 400 50  0000 C CNN
 	1    5600 1600
@@
 F 0 "SW1" H 1200 4750 50  0000 C CNN
 F 1 "UP_Bonsai_SWITCH_INV" H 1250 4450 50  0000 C CNN
-F 2 "tg_foodprint:SW_PUSH_LCD_E3_SAxxxx_tg_V2" H 1400 4600 50  0001 C CNN
+F 2 "allBonsaiFootprintsLibs:SW_PUSH_LCD_E3_SAxxxx_tg_V2" H 1400 4600 50  0001 C CNN
 F 3 "" H 1400 4600 50  0000 C CNN
 	1    1400 4600
@@
 F 0 "SW2" H 1200 6500 50  0000 C CNN
 F 1 "DOWN_Bonsai_SWITCH_INV" H 1250 6200 50  0000 C CNN
-F 2 "tg_foodprint:SW_PUSH_LCD_E3_SAxxxx_tg_V2" H 1400 6350 50  0001 C CNN
+F 2 "allBonsaiFootprintsLibs:SW_PUSH_LCD_E3_SAxxxx_tg_V2" H 1400 6350 50  0001 C CNN
 F 3 "" H 1400 6350 50  0000 C CNN
 	1    1400 6350
@@
 F 0 "C1" V 688 1400 50  0000 C CNN
 F 1 "C" V 779 1400 50  0000 C CNN
-F 2 "tg_foodprint:C_Disc_D10.0mm_W2.5mm_P5.00mm" V 855 1400 30  0001 C CNN
+F 2 "allBonsaiFootprintsLibs:C_Disc_D10.0mm_W2.5mm_P5.00mm" V 855 1400 30  0001 C CNN
 F 3 "" H 1000 1400 60  0000 C CNN
 	1    1000 1400
@@
 F 0 "C2" V 688 1600 50  0000 C CNN
 F 1 "C" V 779 1600 50  0000 C CNN
-F 2 "tg_foodprint:C_Disc_D10.0mm_W2.5mm_P5.00mm" V 855 1600 30  0001 C CNN
+F 2 "allBonsaiFootprintsLibs:C_Disc_D10.0mm_W2.5mm_P5.00mm" V 855 1600 30  0001 C CNN
 F 3 "" H 1000 1600 60  0000 C CNN
 	1    1000 1600
@@
 F 0 "C3" V 688 1800 50  0000 C CNN
 F 1 "C" V 779 1800 50  0000 C CNN
-F 2 "tg_foodprint:C_Disc_D10.0mm_W2.5mm_P5.00mm" V 855 1800 30  0001 C CNN
+F 2 "allBonsaiFootprintsLibs:C_Disc_D10.0mm_W2.5mm_P5.00mm" V 855 1800 30  0001 C CNN
 F 3 "" H 1000 1800 60  0000 C CNN
 	1    1000 1800
