File: EinTaktReset.kicad_pcb (KiCad board)
At the start: 2 copper layers, 65 parts, among them IC1 74LS624, P1 CONN_02X10, P10 CONN_01X01, P11 CONN_01X01, P12 CONN_01X01, P13 CONN_01X01, P14 CONN_01X01, P15 CONN_01X01, P2 CONN_01X01, P3 CONN_01X01, P4 CONN_02X10, P5 CONN_01X01, P6 CONN_01X01, P7 CONN_01X01, P8 CONN_01X01, P9 CONN_01X01, SW1 SPST, SW10 SPST, SW11 SPST, SW12 SPST, SW13 SPST, SW2 SWITCH_INV, SW3 SPST, SW4 SPST, SW5 SPST, SW6 SWITCH_INV, SW7 SPST, SW8 SPST, SW9 SPST, U1 74LS132, U10 74LS00, U2 74540En, U3 74HCT541_PWR, U4 74LS32, U5 74LS00, U6 74LS132, U8 74LS32, U9 74LS32

Commit message: TerminalBlochTested
Parts:
- removed P10, P11, P12, P13, P14, P15, P5, P6, P7: CONN_01X01, Connect:1pin
- removed U10: 74LS00, Housings_DIP:DIP-14_W7.62mm_Socket_LongPads
- removed U8, U9: 74LS32, Housings_DIP:DIP-14_W7.62mm_Socket_LongPads
- added J1: 3PinTerminalBlocktg, 3PinTerminalBlocktg, F.Cu at (195.3, 109.5)
- added J2: 3PinTerminalBlocktg, 3PinTerminalBlocktg, F.Cu at (211.9, 109.5)
Connections:
- IC1 pad 5: Net-(4,7k3-Pad2) -> Net-(IC1-Pad5)
- P1 pad 1: GND -> Net-(P1-Pad1)
- P1 pad 10: GND -> Net-(P1-Pad10)
- P1 pad 2: GND -> Net-(P1-Pad2)
- P1 pad 3: GND -> Net-(P1-Pad3)
- P1 pad 4: GND -> Net-(P1-Pad4)
- P1 pad 5: GND -> Net-(P1-Pad5)
- P1 pad 6: GND -> Net-(P1-Pad6)
- P1 pad 7: GND -> Net-(P1-Pad7)
- P1 pad 8: GND -> Net-(P1-Pad8)
- P1 pad 9: GND -> Net-(P1-Pad9)
- P4 pad 11: GND -> Net-(P4-Pad11)
- P4 pad 12: GND -> Net-(P4-Pad12)
- P4 pad 13: GND -> Net-(P4-Pad13)
- P4 pad 14: GND -> Net-(P4-Pad14)
- P4 pad 15: GND -> Net-(P4-Pad15)
- P4 pad 16: GND -> Net-(P4-Pad16)
- P4 pad 17: GND -> Net-(P4-Pad17)
- P4 pad 18: GND -> Net-(P4-Pad18)
- P4 pad 19: GND -> Net-(P4-Pad19)
- P4 pad 20: GND -> Net-(P4-Pad20)
- SW2 pad 1: Net-(4,7k1-Pad2) -> Net-(SW2-Pad1)
- SW2 pad 3: Net-(4,7k2-Pad1) -> Net-(SW2-Pad3)
- SW3 pad 2: Net-(4,7k3-Pad2) -> Net-(IC1-Pad5)
- U1 pad 13: Net-(4,7k2-Pad1) -> Net-(SW2-Pad3)
- U1 pad 9: Net-(4,7k1-Pad2) -> Net-(SW2-Pad1)
- U2 pad 18: Net-(4,7k2-Pad1) -> Net-(SW2-Pad3)
- U3 pad 19: Net-(U3-Pad1) -> Net-(U3-Pad19)
- U4 pad 5: Net-(U3-Pad1) -> Net-(U4-Pad5)
- U4 pad 8: CLK -> Net-(U4-Pad8)
- U5 pad 11: Net-(U5-Pad10) -> Net-(U5-Pad11)
- U5 pad 5: Net-(U5-Pad3) -> Net-(U5-Pad5)

Commit message: Pin Header reorganized localy and adapted
Parts:
- P1, P4: footprint Pin_Headers:Pin_Header_Straight_2x10_Pitch2.00mm -> tg_foodprint:Pin_Header_Straight_2x10_Pitch2.00mmBonsai.pretty
- moved SW5 317.2 mm to (18.7, 133.1), turned to 90 degrees
- moved SW8 314.1 mm to (30.5, 133.3), turned to 90 degrees
- moved SW11 309.6 mm to (44.1, 134.5), turned to 90 degrees
- moved SW7 308.9 mm to (25.0, 133.1), turned to 90 degrees
- moved SW10 302.7 mm to (40.3, 133.8), turned to 90 degrees
- moved SW13 301.2 mm to (50.4, 134.5), turned to 90 degrees
- moved SW9 295.7 mm to (36.8, 133.3), turned to 90 degrees
- moved SW12 294.4 mm to (46.6, 133.8), turned to 90 degrees
- moved P1 202.5 mm to (20.3, 61.0)
- moved U5 179.9 mm to (135.8, 115.0)
- moved U6 179.9 mm to (147.0, 115.0)
- moved RP1 134.7 mm to (39.4, 115.6)
- moved U3 103.0 mm to (30.5, 96.5), turned to 90 degrees
- moved P4 23.4 mm to (61.0, 59.7)
Connections:
- P1 pad 1: Net-(P1-Pad1) -> GND
- P1 pad 10: Net-(P1-Pad10) -> GND
- P1 pad 12: /a7 -> GND
- P1 pad 13: /a6 -> GND
- P1 pad 14: /a5 -> GND
- P1 pad 15: /a4 -> GND
- P1 pad 16: /a3 -> GND
- P1 pad 17: /a2 -> GND
- P1 pad 18: /a1 -> GND
- P1 pad 19: /a0 -> GND
- P1 pad 2: Net-(P1-Pad2) -> /a0
- P1 pad 3: Net-(P1-Pad3) -> /a1
- P1 pad 4: Net-(P1-Pad4) -> /a2
- P1 pad 5: Net-(P1-Pad5) -> /a3
- P1 pad 6: Net-(P1-Pad6) -> /a4
- P1 pad 7: Net-(P1-Pad7) -> /a5
- P1 pad 8: Net-(P1-Pad8) -> /a6
- P1 pad 9: Net-(P1-Pad9) -> /a7
- P4 pad 11: Net-(P4-Pad11) -> GND
- P4 pad 12: Net-(P4-Pad12) -> GND
- P4 pad 13: Net-(P4-Pad13) -> GND
- P4 pad 14: Net-(P4-Pad14) -> GND
- P4 pad 15: Net-(P4-Pad15) -> GND
- P4 pad 16: Net-(P4-Pad16) -> GND
- P4 pad 17: Net-(P4-Pad17) -> GND
- P4 pad 18: Net-(P4-Pad18) -> GND
- P4 pad 19: Net-(P4-Pad19) -> GND
- P4 pad 20: Net-(P4-Pad20) -> GND
- SW2 pad 1: Net-(SW2-Pad1) -> Net-(4,7k1-Pad2)
- SW2 pad 3: Net-(SW2-Pad3) -> Net-(4,7k2-Pad1)
- U1 pad 13: Net-(SW2-Pad3) -> Net-(4,7k2-Pad1)
- U1 pad 9: Net-(SW2-Pad1) -> Net-(4,7k1-Pad2)
- U2 pad 18: Net-(SW2-Pad3) -> Net-(4,7k2-Pad1)
- U3 pad 19: Net-(U3-Pad19) -> Net-(U3-Pad1)
- U4 pad 5: Net-(U4-Pad5) -> Net-(U3-Pad1)
- U4 pad 8: Net-(U4-Pad8) -> CLK
- U5 pad 11: Net-(U5-Pad11) -> Net-(U5-Pad10)
- U5 pad 5: Net-(U5-Pad5) -> Net-(U5-Pad3)

Commit message: pcb gelayoutet, Libraries benannt, todo.txt geändert!
Parts:
- removed 10k1, 4,7k1, 4,7k2, 4,7k3: ., Resistors_ThroughHole:R_Axial_DIN0207_L6.3mm_D2.5mm_P10.16mm_Horizontal
- removed P2, P3, P8, P9: CONN_01X01, Connect:1pin
- added J3: 2PinTerminalBlocktg, 2PinTerminalBlocktg, F.Cu at (415.3, 20.7)
- added J4: 3PinTerminalBlocktg, 3PinTerminalBlocktg, F.Cu at (415.7, 6.61)
- added J5: 2PinTerminalBlocktg, 2PinTerminalBlocktg, F.Cu at (431.9, 7.65)
- R4: value R -> 150
- moved D1 397.1 mm to (27.9, 170.2)
- moved C1 386.5 mm to (20.3, 180.3), turned to 180 degrees
- moved SW1 371.5 mm to (17.8, 149.9), turned to 90 degrees
- moved SW2 355.8 mm to (27.9, 144.8)
- moved SW6 263.0 mm to (27.9, 179.1)
- moved U1 248.2 mm to (48.3, 180.3), turned to 90 degrees
- moved U2 191.1 mm to (83.8, 180.3), turned to 90 degrees
- moved SW13 49.1 mm to (68.6, 88.9)
- moved SW12 47.6 mm to (62.2, 88.9)
- moved SW11 47.1 mm to (55.9, 88.9)
- moved SW10 45.9 mm to (49.5, 88.9)
- moved SW8 44.9 mm to (36.8, 88.9)
- moved SW9 44.9 mm to (43.2, 88.9)
- moved SW7 44.5 mm to (30.5, 88.9)
- moved SW5 44.5 mm to (24.1, 88.9)
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Connections:
- J1 pad 1: clrMPC -> en-ln1
- J1 pad 2: enAkku -> en-ln2
- J1 pad 3: loadIR -> auto
- J2 pad 1: auto -> CLK
- J2 pad 2: enSTW -> enDEC
- J2 pad 3: enDEC -> enSTW
Routing:
- net Net-(RP1-Pad9): track 0.00 -> 31.3 mm
- net Net-(RP1-Pad2): track 0.00 -> 28.6 mm
- net Net-(RP1-Pad8): track 0.00 -> 28.2 mm
- net Net-(RP1-Pad3): track 0.00 -> 26.2 mm
- net Net-(RP1-Pad7): track 0.00 -> 25.2 mm
- net Net-(RP1-Pad4): track 0.00 -> 22.4 mm
- net Net-(RP1-Pad6): track 0.00 -> 21.4 mm
- net Net-(RP1-Pad5): track 0.00 -> 20.8 mm
Other:
- net class Default: trace_width 0.25 -> 1
