File: Steuerwerk.kicad_pcb (KiCad board)
At the start: 2 copper layers, 114 parts, among them J1 2PinTerminalBlocktg, J10 2PinTerminalBlocktg, J11 2PinTerminalBlocktg, J12 2PinTerminalBlocktg, J2 2PinTerminalBlocktg, J3 3PinTerminalBlocktg, J4 3PinTerminalBlocktg, J5 2PinTerminalBlocktg, J6 2PinTerminalBlocktg, J7 2PinTerminalBlocktg, J8 2PinTerminalBlocktg, J9 2PinTerminalBlocktg, Q1 Q_PNP_BCE, U1 74ls240, U2 74541, U3 74LS161, U4 74LS138, U5 74LS138, U6 74541, U7 74LS374, U8 74LS374

Commit message: Steuerwerk: a lot of things ...
Parts:
- added D63: Led_Small, tg_foodprint:LED_D1.8mm_W3.3mm_H2.4mmBonsai, F.Cu at (118.1, 90.1)
- U8: footprint Housings_DIP:DIP-20_W7.62mm_Socket_LongPads -> tg_foodprint:DIP-20_W7.62mm_Socket_LongPadstg
- moved R16 130.8 mm to (71.2, 52.7), turned to 90 degrees
- moved D61 106.1 mm to (120.6, 102.8)
- moved D40 106.0 mm to (91.5, 92.7)
- moved D60 105.4 mm to (118.1, 97.8)
- moved D38 104.8 mm to (88.9, 87.6)
- moved D52 103.6 mm to (115.6, 87.6)
- moved D53 103.6 mm to (115.6, 90.2)
- moved D56 103.6 mm to (115.6, 97.7)
- moved D54 103.6 mm to (115.5, 92.6)
- moved D55 103.6 mm to (115.5, 95.2)
- moved D57 103.6 mm to (115.5, 100.3)
- moved D58 103.6 mm to (115.6, 102.8)
- moved D35 103.5 mm to (86.4, 90.1)
- moved D31 101.0 mm to (81.3, 92.7)
- moved D28 99.8 mm to (78.8, 102.8)
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Connections:
- D1 pad 1: GND -> Net-(D1-Pad1)
- D1 pad 2: Net-(D1-Pad2) -> GND
- D10 pad 1: Net-(D10-Pad1) -> (no net)
- D10 pad 2: Net-(D10-Pad2) -> (no net)
- D11 pad 1: Net-(D11-Pad1) -> VCC
- D11 pad 2: VCC -> Net-(D11-Pad2)
- D12 pad 1: Net-(D12-Pad1) -> VCC
- D12 pad 2: VCC -> Net-(D12-Pad2)
- D14 pad 1: Net-(D14-Pad1) -> VCC
- D14 pad 2: VCC -> Net-(D14-Pad2)
- D15 pad 1: Net-(D15-Pad1) -> VCC
- D15 pad 2: VCC -> Net-(D15-Pad2)
- D16 pad 1: Net-(D16-Pad1) -> VCC
- D16 pad 2: VCC -> Net-(D16-Pad2)
- D17 pad 1: Net-(D17-Pad1) -> /a1
- D18 pad 1: Net-(D18-Pad1) -> /a1
- D18 pad 2: Net-(D17-Pad2) -> Net-(D18-Pad2)
- D19 pad 1: Net-(D19-Pad1) -> /a1
- D19 pad 2: Net-(D17-Pad2) -> Net-(D19-Pad2)
- D2 pad 1: Net-(D2-Pad1) -> VCC
- D2 pad 2: VCC -> Net-(D2-Pad2)
- D20 pad 1: Net-(D20-Pad1) -> /a1
- D20 pad 2: Net-(D17-Pad2) -> Net-(D20-Pad2)
- D21 pad 1: Net-(D21-Pad1) -> /a2
- D22 pad 1: Net-(D22-Pad1) -> VCC
- D22 pad 2: VCC -> Net-(D22-Pad2)
- D23 pad 1: Net-(D23-Pad1) -> /a3
- D24 pad 1: Net-(D21-Pad1) -> /a3
- D24 pad 2: Net-(D23-Pad2) -> Net-(D21-Pad2)
- D25 pad 1: Net-(D25-Pad1) -> /a3
- D25 pad 2: Net-(D23-Pad2) -> Net-(D25-Pad2)
- D26 pad 1: Net-(D26-Pad1) -> /a3
- D26 pad 2: Net-(D23-Pad2) -> Net-(D26-Pad2)
- D27 pad 1: Net-(D27-Pad1) -> /a3
- D27 pad 2: Net-(D23-Pad2) -> Net-(D27-Pad2)
- D28 pad 1: Net-(D20-Pad1) -> /a3
- D28 pad 2: Net-(D23-Pad2) -> Net-(D20-Pad2)
- D29 pad 1: Net-(D29-Pad1) -> VCC
- D29 pad 2: VCC -> Net-(D29-Pad2)
- D3 pad 1: Net-(D3-Pad1) -> VCC
- D3 pad 2: VCC -> Net-(D3-Pad2)
- D30 pad 1: Net-(D17-Pad1) -> /a4
- D30 pad 2: Net-(D30-Pad2) -> Net-(D17-Pad2)
- D31 pad 1: Net-(D18-Pad1) -> /a4
- D31 pad 2: Net-(D30-Pad2) -> Net-(D18-Pad2)
- D32 pad 1: Net-(D32-Pad1) -> VCC
- D32 pad 2: VCC -> Net-(D32-Pad2)
- D33 pad 1: Net-(D33-Pad1) -> /a5
- D34 pad 1: Net-(D34-Pad1) -> VCC
- D34 pad 2: VCC -> Net-(D34-Pad2)
- D35 pad 1: Net-(D35-Pad1) -> /a6
- D36 pad 1: Net-(D36-Pad1) -> VCC
- D36 pad 2: VCC -> Net-(D36-Pad2)
- D37 pad 1: Net-(D25-Pad1) -> /a7
- D37 pad 2: Net-(D37-Pad2) -> Net-(D25-Pad2)
- D38 pad 1: Net-(D26-Pad1) -> /a7
- D38 pad 2: Net-(D37-Pad2) -> Net-(D26-Pad2)
- D39 pad 1: Net-(D17-Pad1) -> /a8
- D39 pad 2: Net-(D39-Pad2) -> Net-(D17-Pad2)
- D4 pad 1: Net-(D4-Pad1) -> (no net)
- D4 pad 2: Net-(D4-Pad2) -> (no net)
- D40 pad 1: Net-(D18-Pad1) -> /a8
- D40 pad 2: Net-(D39-Pad2) -> Net-(D18-Pad2)
- D41 pad 1: Net-(D41-Pad1) -> VCC
- D41 pad 2: VCC -> Net-(D41-Pad2)
- D42 pad 1: Net-(D19-Pad1) -> /b1
- D42 pad 2: Net-(D42-Pad2) -> Net-(D19-Pad2)
- D43 pad 1: Net-(D43-Pad1) -> /b2
- D44 pad 1: Net-(D23-Pad1) -> /b2
- D44 pad 2: Net-(D43-Pad2) -> Net-(D23-Pad2)
- D45 pad 1: Net-(D21-Pad1) -> /b2
- D45 pad 2: Net-(D43-Pad2) -> Net-(D21-Pad2)
- D46 pad 1: Net-(D23-Pad1) -> /b3
- D46 pad 2: Net-(D46-Pad2) -> Net-(D23-Pad2)
- D47 pad 1: Net-(D47-Pad1) -> /b4
- D48 pad 1: Net-(D25-Pad1) -> /b4
- D48 pad 2: Net-(D47-Pad2) -> Net-(D25-Pad2)
- D49 pad 1: Net-(D33-Pad1) -> /b4
- D49 pad 2: Net-(D47-Pad2) -> Net-(D33-Pad2)
- D5 pad 1: Net-(D5-Pad1) -> VCC
- D5 pad 2: VCC -> Net-(D5-Pad2)
- D50 pad 1: Net-(D17-Pad1) -> /b4
- D50 pad 2: Net-(D47-Pad2) -> Net-(D17-Pad2)
- D51 pad 1: Net-(D51-Pad1) -> /b4
- D51 pad 2: Net-(D47-Pad2) -> Net-(D51-Pad2)
- D52 pad 1: Net-(D26-Pad1) -> /b4
- D52 pad 2: Net-(D47-Pad2) -> Net-(D26-Pad2)
- D53 pad 1: Net-(D35-Pad1) -> /b4
- D53 pad 2: Net-(D47-Pad2) -> Net-(D35-Pad2)
- D54 pad 1: Net-(D18-Pad1) -> /b4
- D54 pad 2: Net-(D47-Pad2) -> Net-(D18-Pad2)
- D55 pad 1: Net-(D19-Pad1) -> /b4
- D55 pad 2: Net-(D47-Pad2) -> Net-(D19-Pad2)
- D56 pad 1: Net-(D56-Pad1) -> /b4
- D56 pad 2: Net-(D47-Pad2) -> Net-(D56-Pad2)
- D57 pad 1: Net-(D27-Pad1) -> /b4
- D57 pad 2: Net-(D47-Pad2) -> Net-(D27-Pad2)
- D58 pad 1: Net-(D20-Pad1) -> /b4
- D58 pad 2: Net-(D47-Pad2) -> Net-(D20-Pad2)
- D59 pad 1: Net-(D33-Pad1) -> /b5
- D59 pad 2: Net-(D59-Pad2) -> Net-(D33-Pad2)
- D6 pad 1: Net-(D6-Pad1) -> (no net)
- D6 pad 2: Net-(D6-Pad2) -> (no net)
- D60 pad 1: Net-(D20-Pad1) -> /b5
- D60 pad 2: Net-(D59-Pad2) -> Net-(D56-Pad2)
- D61 pad 1: Net-(D27-Pad1) -> /b6
- D61 pad 2: Net-(D61-Pad2) -> Net-(D20-Pad2)
- D7 pad 1: Net-(D7-Pad1) -> VCC
- D7 pad 2: VCC -> Net-(D7-Pad2)
- D8 pad 1: Net-(D8-Pad1) -> (no net)
- D8 pad 2: Net-(D8-Pad2) -> (no net)
- D9 pad 1: Net-(D9-Pad1) -> VCC
- D9 pad 2: VCC -> Net-(D9-Pad2)
- J1 pad 1: /vom_Befehle-decoder -> Net-(J1-Pad1)
- J1 pad 2: /vom_Befehle-decoder -> Net-(J1-Pad2)
- J2 pad 1: /vom_Befehle-decoder -> Net-(J2-Pad1)
- J2 pad 2: /vom_Befehle-decoder -> Net-(J2-Pad2)
- J3 pad 1: /Takt -> /enSTW
- R1 pad 2: Net-(D1-Pad2) -> Net-(D1-Pad1)
- R10 pad 2: Net-(R10-Pad2) -> (no net)
- R11 pad 2: Net-(D11-Pad1) -> Net-(D11-Pad2)
- R13 pad 2: Net-(D12-Pad1) -> Net-(D12-Pad2)
- R14 pad 2: Net-(D14-Pad1) -> Net-(D14-Pad2)
- R15 pad 2: Net-(D15-Pad1) -> Net-(D15-Pad2)
- R16 pad 1: Net-(R16-Pad1) -> /a2
- R17 pad 2: Net-(D16-Pad1) -> Net-(D16-Pad2)
- R19 pad 2: Net-(D22-Pad1) -> Net-(D22-Pad2)
- R2 pad 2: Net-(D2-Pad1) -> Net-(D2-Pad2)
- R21 pad 2: Net-(D29-Pad1) -> Net-(D29-Pad2)
- R24 pad 2: Net-(D32-Pad1) -> Net-(D32-Pad2)
- R26 pad 2: Net-(D34-Pad1) -> Net-(D34-Pad2)
- R28 pad 2: Net-(D36-Pad1) -> Net-(D36-Pad2)
- R3 pad 2: Net-(D3-Pad1) -> Net-(D3-Pad2)
- R30 pad 2: Net-(D41-Pad1) -> Net-(D41-Pad2)
- R4 pad 2: Net-(R4-Pad2) -> (no net)
- R5 pad 2: Net-(D5-Pad1) -> Net-(D5-Pad2)
- R6 pad 2: Net-(R6-Pad2) -> (no net)
- R7 pad 2: Net-(D7-Pad1) -> Net-(D7-Pad2)
- R8 pad 2: Net-(R8-Pad2) -> (no net)
- R9 pad 2: Net-(D9-Pad1) -> Net-(D9-Pad2)
- RP1 pad 1: Net-(RP1-Pad1) -> VCC
- RP1 pad 2: Net-(RP1-Pad2) -> /b1
- RP1 pad 3: Net-(RP1-Pad3) -> /b2
- RP1 pad 4: Net-(RP1-Pad4) -> /b3
- RP1 pad 5: Net-(RP1-Pad5) -> /b4
- RP1 pad 6: Net-(RP1-Pad6) -> /b5
- RP1 pad 7: Net-(RP1-Pad7) -> /b6
- RP1 pad 8: Net-(RP1-Pad8) -> /b7
- RP1 pad 9: Net-(RP1-Pad9) -> /b8
- RP2 pad 1: Net-(RP2-Pad1) -> VCC
- RP2 pad 2: Net-(RP2-Pad2) -> /a1
- RP2 pad 3: Net-(RP2-Pad3) -> /a2
- RP2 pad 4: Net-(RP2-Pad4) -> /a3
- RP2 pad 5: Net-(RP2-Pad5) -> /a4
- RP2 pad 6: Net-(RP2-Pad6) -> /a5
- RP2 pad 7: Net-(RP2-Pad7) -> /a6
- RP2 pad 8: Net-(RP2-Pad8) -> /a7
- RP2 pad 9: Net-(RP2-Pad9) -> /a8
- U1 pad 1: Net-(U1-Pad1) -> (no net)
- U1 pad 19: Net-(U1-Pad19) -> (no net)
- U2 pad 1: Net-(U2-Pad1) -> (no net)
- U2 pad 19: Net-(U2-Pad19) -> (no net)
- U2 pad 20: (no net) -> VCC
- U3 pad 15: Net-(U3-Pad15) -> (no net)
- U3 pad 3: /vom_Befehle-decoder -> Net-(J2-Pad1)
- U3 pad 4: /vom_Befehle-decoder -> Net-(J2-Pad2)
- U3 pad 5: /vom_Befehle-decoder -> Net-(J1-Pad1)
- U3 pad 6: /vom_Befehle-decoder -> Net-(J1-Pad2)
- U3 pad 9: Net-(D21-Pad2) -> /a2
- U4 pad 10: Net-(D33-Pad1) -> Net-(D33-Pad2)
- U4 pad 11: Net-(D25-Pad1) -> Net-(D25-Pad2)
- U4 pad 12: Net-(D47-Pad1) -> Net-(D47-Pad2)
- U4 pad 13: Net-(D21-Pad1) -> Net-(D21-Pad2)
- U4 pad 14: Net-(D23-Pad1) -> Net-(D23-Pad2)
- U4 pad 15: Net-(D43-Pad1) -> Net-(D43-Pad2)
- U4 pad 7: Net-(D51-Pad1) -> Net-(D51-Pad2)
- U4 pad 9: Net-(D17-Pad1) -> Net-(D17-Pad2)
- U5 pad 10: Net-(D27-Pad1) -> Net-(D27-Pad2)
- U5 pad 11: Net-(D56-Pad1) -> Net-(D56-Pad2)
- U5 pad 12: Net-(D19-Pad1) -> Net-(D19-Pad2)
- U5 pad 13: Net-(D18-Pad1) -> Net-(D18-Pad2)
- U5 pad 14: Net-(D35-Pad1) -> Net-(D35-Pad2)
- U5 pad 15: Net-(D26-Pad1) -> Net-(D26-Pad2)
- U5 pad 7: Net-(U5-Pad7) -> (no net)
- U5 pad 9: Net-(D20-Pad1) -> Net-(D20-Pad2)
- U6 pad 1: Net-(U6-Pad1) -> /enSTW
- U6 pad 19: Net-(U6-Pad19) -> /enSTW
- U6 pad 20: (no net) -> VCC
- U7 pad 1: /Takt -> /enSTW
- U7 pad 13: Net-(D37-Pad2) -> /a7
- U7 pad 14: Net-(D33-Pad2) -> /a5
- U7 pad 17: Net-(D23-Pad2) -> /a3
- U7 pad 18: Net-(D17-Pad2) -> /a1
- U7 pad 3: Net-(D21-Pad2) -> /a2
- U7 pad 4: Net-(D30-Pad2) -> /a4
- U7 pad 7: Net-(U7-Pad7) -> /a6
- U7 pad 8: Net-(D39-Pad2) -> /a8
- U8 pad 1: /Takt -> /enSTW
- U8 pad 13: Net-(U8-Pad13) -> /b7
- U8 pad 14: Net-(D59-Pad2) -> /b5
- U8 pad 17: Net-(D46-Pad2) -> /b3
- U8 pad 18: Net-(D42-Pad2) -> /b1
- U8 pad 3: Net-(D43-Pad2) -> /b2
- U8 pad 4: Net-(D47-Pad2) -> /b4
- U8 pad 7: Net-(D61-Pad2) -> /b6
- U8 pad 8: Net-(U8-Pad8) -> /b8
Routing:
- net VCC: track 748.4 -> 634.7 mm
- net (no net): track 0.00 -> 77.7 mm
- net Net-(D51-Pad2): track 0.00 -> 77.7 mm
- net Net-(D35-Pad2): track 0.00 -> 67.9 mm
- net Net-(D20-Pad2): track 0.00 -> 67.9 mm
- net Net-(D19-Pad2): track 0.00 -> 67.9 mm
- net Net-(D18-Pad2): track 0.00 -> 67.9 mm
- net Net-(D56-Pad2): track 0.00 -> 67.9 mm
- net Net-(D27-Pad2): track 0.00 -> 67.9 mm
- net Net-(D26-Pad2): track 0.00 -> 67.9 mm
- net Net-(D17-Pad2): track 0.00 -> 67.9 mm
- net Net-(D47-Pad2): track 0.00 -> 67.8 mm
- net Net-(D43-Pad2): track 0.00 -> 67.8 mm
- net Net-(D33-Pad2): track 0.00 -> 67.8 mm
- net Net-(D25-Pad2): track 0.00 -> 67.8 mm
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
Commit message: steuerwerk improvements
Parts:
- removed U1: 74ls240, Housings_DIP:DIP-20_W7.62mm_Socket_LongPads
- added REF**: EuroBoard160mmX100mm_holes, tg_foodprint:EuroBoard160mmX100mm_holes, F.Cu at (141.6, 193.6)
- added U9: 74ls240, Package_DIP:DIP-20_W7.62mm_Socket_LongPads, F.Cu at (45.8, 121.2)
- moved R12 28.7 mm to (96.0, 43.0), turned to 270 degrees
- moved U3 20.4 mm to (63.5, 49.4), turned to 270 degrees
- moved J1 12.1 mm to (116.9, 40.7), turned to 180 degrees
- moved C3 9.96 mm to (66.3, 109.6), turned to 180 degrees
- moved R16 9.91 mm to (81.1, 52.7)
- moved J2 8.29 mm to (127.0, 40.7), turned to 180 degrees
- moved C4 5.16 mm to (100.1, 114.9), turned to 270 degrees
- moved Q1 4.02 mm to (87.7, 39.3)
- moved D13 4.02 mm to (95.9, 37.4)
- moved J3 3.56 mm to (46.0, 95.3)
- moved R10 2.54 mm to (63.9, 126.9)
- moved R4 2.54 mm to (48.6, 126.9)
- moved R6 2.54 mm to (53.7, 126.9)
- moved R8 2.54 mm to (58.8, 126.9)
- moved C2 2.18 mm to (67.1, 55.7)
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Connections:
- D10 pad 1: (no net) -> Net-(D10-Pad1)
- D10 pad 2: (no net) -> VCC
- D4 pad 1: (no net) -> Net-(D4-Pad1)
- D4 pad 2: (no net) -> VCC
- D6 pad 1: (no net) -> Net-(D6-Pad1)
- D6 pad 2: (no net) -> VCC
- D8 pad 1: (no net) -> Net-(D8-Pad1)
- D8 pad 2: (no net) -> VCC
- R10 pad 2: (no net) -> Net-(D10-Pad1)
- R4 pad 2: (no net) -> Net-(D4-Pad1)
- R6 pad 2: (no net) -> Net-(D6-Pad1)
- R8 pad 2: (no net) -> Net-(D8-Pad1)
- U2 pad 1: (no net) -> /enSTW
- U2 pad 19: (no net) -> /enSTW
Routing:
- net GND: track 0.00 -> 197.6 mm, vias 0 -> 3
- net VCC: track 634.7 -> 816.0 mm, vias 0 -> 2
- net /enSTW: track 0.00 -> 104.4 mm, vias 0 -> 4
- net Net-(J2-Pad1): track 0.00 -> 77.7 mm
- net Net-(J2-Pad2): track 0.00 -> 74.9 mm
- net Net-(J1-Pad1): track 0.00 -> 72.2 mm
- net Net-(J1-Pad2): track 0.00 -> 69.4 mm
- net Net-(U3-Pad12): track 0.00 -> 60.9 mm
- net /11: track 82.7 -> 143.1 mm, vias 0 -> 2
- net /a2: track 63.8 -> 123.8 mm
- net Net-(U3-Pad11): track 0.00 -> 59.6 mm
- net /enAkku: track 70.9 -> 116.4 mm, vias 0 -> 2
- net /clrMPC: track 25.3 -> 62.2 mm
- net Net-(Q1-Pad1): track 0.00 -> 7.92 mm
- net Net-(D13-Pad1): track 0.00 -> 6.50 mm
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Other:
- board outline added: 100 x 160 mm
