File: Steuerwerk.kicad_pcb (KiCad board)
At the start: 2 copper layers, 100 x 160 mm, 116 parts, among them J1 2PinTerminalBlocktg, J10 2PinTerminalBlocktg, J11 2PinTerminalBlocktg, J12 2PinTerminalBlocktg, J2 2PinTerminalBlocktg, J3 3PinTerminalBlocktg, J4 3PinTerminalBlocktg, J5 2PinTerminalBlocktg, J6 2PinTerminalBlocktg, J7 2PinTerminalBlocktg, J8 2PinTerminalBlocktg, J9 2PinTerminalBlocktg, Q1 Q_PNP_BCE, U2 74541, U3 74LS161, U4 74LS138, U5 74LS138, U6 74541, U7 74LS374, U8 74LS374, U9 74ls240

Commit message: tracs tracs tracs
Parts:
- moved C3 4.21 mm to (70.5, 109.2)
Connections:
- U3 pad 14: Net-(U3-Pad11) -> Net-(U3-Pad14)
- U4 pad 1: Net-(U3-Pad11) -> Net-(U3-Pad14)
- U5 pad 1: Net-(U3-Pad11) -> Net-(U3-Pad14)
- U9 pad 11: Net-(U3-Pad11) -> Net-(U3-Pad14)
Routing:
- net Net-(U3-Pad13): track 0.00 -> 75.1 mm, vias 0 -> 4
- net Net-(U3-Pad14): track 0.00 -> 74.6 mm
- net Net-(U3-Pad11): track 59.6 -> 79.4 mm, vias 0 -> 4
- net VCC: track 816.0 -> 833.2 mm
- net Net-(U3-Pad12): track 60.9 -> 76.2 mm, vias 0 -> 4
- net /enDEC: track 0.00 -> 13.0 mm, vias 0 -> 1
- net Net-(R8-Pad1): track 0.00 -> 6.52 mm
- net Net-(R6-Pad1): track 0.00 -> 6.52 mm
- net Net-(R4-Pad1): track 0.00 -> 6.52 mm
- net Net-(R10-Pad1): track 0.00 -> 6.52 mm
- net GND: track 197.6 -> 202.6 mm

Commit message: tracs tracs tracs
Routing:
- net VCC: track 833.2 -> 998.1 mm, vias 2 -> 7
Changed lines of the file:
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@@
     (thickness 1.6)
     (drawings 0)
-    (tracks 848)
+    (tracks 882)
     (zones 0)
     (modules 116)
@@
   )
   (setup
-    (last_trace_width 0.8)
+    (last_trace_width 1.25)
     (user_trace_width 0.2)
     (user_trace_width 0.4)
@@
   (segment (start 44.156 113.625998) (end 43.17 113.625998) (width 0.8) (layer B.Cu) (net 23))
   (segment (start 45.756 113.625998) (end 44.156 113.625998) (width 0.8) (layer B.Cu) (net 23) (status 10))
-  (segment (start 43.17 182.849998) (end 43.17 113.625998) (width 1.25) (layer B.Cu) (net 23))
   (segment (start 43.17 113.625998) (end 43.17 109.353998) (width 1.25) (layer B.Cu) (net 23))
   (segment (start 64.055998 142.083) (end 64.11 142.028998) (width 1.25) (layer B.Cu) (net 23) (status 30))
@@
   (segment (start 49.674 55.205998) (end 48.296 56.583998) (width 0.4) (layer B.Cu) (net 23))
   (segment (start 62.158 55.205998) (end 49.674 55.205998) (width 0.4) (layer B.Cu) (net 23))
+  (segment (start 105.446 113.225998) (end 105.446 113.625998) (width 1.25) (layer B.Cu) (net 23))
+  (segment (start 101.89 109.669998) (end 105.446 113.225998) (width 1.25) (layer B.Cu) (net 23))
+  (segment (start 103.396 59.015998) (end 101.89 60.521998) (width 1.25) (layer B.Cu) (net 23))
+  (segment (start 105.446 59.015998) (end 103.396 59.015998) (width 1.25) (layer B.Cu) (net 23))
+  (segment (start 101.382 113.625998) (end 100.112 114.895998) (width 1.25) (layer B.Cu) (net 23))
+  (segment (start 105.446 113.625998) (end 101.382 113.625998) (width 1.25) (layer B.Cu) (net 23))
+  (via (at 99.858 85.431998) (size 0.6) (drill 0.4) (layers F.Cu B.Cu) (net 23))
+  (segment (start 101.89 85.431998) (end 99.858 85.431998) (width 1.25) (layer B.Cu) (net 23))
+  (segment (start 101.89 85.431998) (end 101.89 109.669998) (width 1.25) (layer B.Cu) (net 23))
+  (via (at 70.394 85.431998) (size 0.6) (drill 0.4) (layers F.Cu B.Cu) (net 23))
+  (segment (start 99.858 85.431998) (end 70.394 85.431998) (width 1.25) (layer F.Cu) (net 23))
+  (segment (start 66.968002 85.431998) (end 66.04 86.36) (width 1.25) (layer B.Cu) (net 23))
+  (segment (start 70.394 85.431998) (end 66.968002 85.431998) (width 1.25) (layer B.Cu) (net 23))
+  (segment (start 65.480002 86.36) (end 62.266 83.145998) (width 1.25) (layer B.Cu) (net 23))
+  (segment (start 66.04 86.36) (end 65.480002 86.36) (width 1.25) (layer B.Cu) (net 23))
+  (via (at 99.604 109.561998) (size 0.6) (drill 0.4) (layers F.Cu B.Cu) (net 23))
+  (segment (start 101.89 109.669998) (end 99.712 109.669998) (width 1.25) (layer B.Cu) (net 23))
+  (segment (start 99.712 109.669998) (end 99.604 109.561998) (width 1.25) (layer B.Cu) (net 23))
+  (via (at 72.172 111.085998) (size 0.6) (drill 0.4) (layers F.Cu B.Cu) (net 23))
+  (segment (start 99.604 109.561998) (end 73.696 109.561998) (width 1.25) (layer F.Cu) (net 23))
+  (segment (start 73.696 109.561998) (end 72.172 111.085998) (width 1.25) (layer F.Cu) (net 23))
+  (via (at 70.521 109.180998) (size 0.6) (drill 0.4) (layers F.Cu B.Cu) (net 23))
+  (segment (start 72.172 111.085998) (end 72.172 110.831998) (width 1.25) (layer B.Cu) (net 23))
+  (segment (start 72.172 110.831998) (end 70.521 109.180998) (width 1.25) (layer B.Cu) (net 23))
+  (segment (start 72.135 110.831998) (end 72.172 110.831998) (width 1.25) (layer B.Cu) (net 23))
+  (segment (start 71.791 111.175998) (end 72.135 110.831998) (width 1.25) (layer B.Cu) (net 23))
+  (segment (start 71.791 113.625998) (end 71.791 111.175998) (width 1.25) (layer B.Cu) (net 23))
+  (segment (start 53.629 142.083) (end 53.629 151.978998) (width 1.25) (layer B.Cu) (net 23))
+  (segment (start 51.596 154.011998) (end 43.17 154.011998) (width 1.25) (layer B.Cu) (net 23))
+  (segment (start 53.629 151.978998) (end 51.596 154.011998) (width 1.25) (layer B.Cu) (net 23))
+  (segment (start 43.17 182.849998) (end 43.17 154.011998) (width 1.25) (layer B.Cu) (net 23))
+  (segment (start 43.17 154.011998) (end 43.17 113.625998) (width 1.25) (layer B.Cu) (net 23))
+  (segment (start 101.89 62.063998) (end 100.112 62.063998) (width 1.25) (layer B.Cu) (net 23))
+  (segment (start 101.89 62.063998) (end 101.89 85.431998) (width 1.25) (layer B.Cu) (net 23))
+  (segment (start 101.89 60.521998) (end 101.89 62.063998) (width 1.25) (layer B.Cu) (net 23))
   (segment (start 73.41 138.29) (end 73.41 129.849998) (width 0.8) (layer B.Cu) (net 24) (status 10))
   (segment (start 73.191001 129.630999) (end 73.191001 123.915999) (width 0.8) (layer B.Cu) (net 24))

Commit message: Steuerwerk wires finished
Parts:
- moved D13 7.27 mm to (102.8, 39.8)
- moved Q1 2.07 mm to (87.3, 41.4)
- moved R16 1.66 mm to (80.9, 54.3)
Routing:
- net GND: track 202.6 -> 542.3 mm, vias 3 -> 9
- net /Takt: track 0.00 -> 184.2 mm, vias 0 -> 2
- net /clrMPC: track 62.2 -> 182.9 mm, vias 0 -> 1
- net /enSTW: track 104.4 -> 166.2 mm, vias 4 -> 6
- net Net-(R1-Pad1): track 0.00 -> 39.9 mm
- net /enDEC: track 13.0 -> 44.7 mm
- net VCC: track 998.1 -> 1007.9 mm, vias 7 -> 9
- net Net-(D13-Pad1): track 6.50 -> 13.6 mm
- net Net-(D13-Pad2): track 3.10 -> 6.99 mm
- net /a2: track 123.8 -> 124.7 mm
- net Net-(J2-Pad1): track 77.7 -> 76.9 mm
- net Net-(J1-Pad2): track 69.4 -> 70.2 mm
- net Net-(Q1-Pad1): track 7.92 -> 7.22 mm

Commit message: BIB Cleanup finished
Connections:
- U2 pad 8: Net-(U2-Pad8) -> (no net)
- U7 pad 2: Net-(U2-Pad8) -> (no net)
Routing:
- net Net-(U2-Pad8): track 19.4 -> 0.00 mm
- net (no net): track 77.7 -> 97.1 mm

Commit message: labeling
Routing:
- net VCC: track 1007.9 -> 1013.5 mm
Other:
- board text added: "+"
- board text added: "-"
- board text added: "CLK"
- board text added: "Steuerwerk"
- board text added: "~clrMPC"
- board text added: "~enAkku"
- board text added: "~enCU"
- board text added: "~enDEC"
- board text added: "~loadIR"

Commit message: branding
Parts:
- added G***: LOGO, allBonsaiFootprintsLibs:agi5, F.Cu at (101.6, 87.0)
