File: _saved_Akku.sch (KiCad schematic (older format))
At the start: 50 parts, among them J1 +/- Stecker, J2 load/up, J3 down/en/clear, P7 CONN_02X10, P8 CONN_02X10, P9 CONN_02X10, SW1 UP_Bonsai_SWITCH_INV, SW2 DOWN_Bonsai_SWITCH_INV, SW3 CLR_Bonsai_SWITCH_INV, U1 74HC14, U2 7400, U4 7408, U5 74LS193, U6 74LS541, U7 74LS193, U8 74LS540

Commit message: diverse Vorbereitungen für akku, switch update
Parts:
- gave numbers to parts that had none: 1
- renumbered RPA to RPA1
Changed lines of the file:
@@
 	10900 1750 10900 1800
 $Comp
-L bonsai:R_PACK4BUSSED RPA
+L bonsai:R_PACK4BUSSED RPA1
 U 1 1 5B220C3D
 P 13200 450
-F 0 "RPA" H 13327 549 50  0000 L CNN
+F 0 "RPA1" H 13327 549 50  0000 L CNN
 F 1 "R_PACK4BUSSED" H 13327 458 50  0000 L CNN
 F 2 "Resistors_ThroughHole:R_Array_SIP5" H 13327 359 60  0000 L CNN
@@
 	13000 100  13200 100
 $Comp
-L power:VCC #PWR?
+L power:VCC #PWR0101
 U 1 1 5B22DB58
 P 13200 100
-F 0 "#PWR?" H 13200 -50 50  0001 C CNN
+F 0 "#PWR0101" H 13200 -50 50  0001 C CNN
 F 1 "VCC" V 13217 228 50  0000 L CNN
 F 2 "" H 13200 100 50  0000 C CNN
@@
 $EndComp
 $Comp
-L bonsai:R_PACK4BUSSED RPB?
+L bonsai:R_PACK4BUSSED RPB1
 U 1 1 5B22DE13
 P 13200 1650
-F 0 "RPB?" H 13327 1749 50  0000 L CNN
+F 0 "RPB1" H 13327 1749 50  0000 L CNN
 F 1 "R_PACK4BUSSED" H 13327 1658 50  0000 L CNN
 F 2 "Resistors_ThroughHole:R_Array_SIP5" H 13327 1559 60  0000 L CNN
