File: Akku.kicad_pcb (KiCad board)
At the start: 2 copper layers, 100 x 160 mm, 50 parts, among them J1 +/- Stecker, J2 load/up, J3 down/en/clear, P7 CONN_02X10, P8 CONN_02X10, P9 CONN_02X10, SW1 UP_Bonsai_SWITCH_INV, SW2 DOWN_Bonsai_SWITCH_INV, SW3 CLR_Bonsai_SWITCH_INV, U1 74HC14, U2 7400, U4 7408, U5 74LS193, U6 74LS541, U7 74LS193, U8 74LS540

Commit message: labeling
Other:
- board text added: "+"
- board text added: "-"
- board text added: "AKKU/PC"
- board text added: "CLEAR"
- board text added: "DOWN"
- board text added: "UP"
- board text added: "clear"
- board text added: "read"
- board text added: "write"
- board text added: "~down"
- board text added: "~en"
- board text added: "~load"
- board text added: "~up"
Changed lines of the file:
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@@
   (general
     (thickness 1.6)
-    (drawings 3)
+    (drawings 14)
     (tracks 857)
     (zones 0)
@@
     (descr "LED, Round, FlatTop, diameter 5.0mm, 2 pins, http://www.kingbright.com/attachments/file/psearch/000/00/00/L-483GDT(Ver.15B).pdf")
     (tags "LED Round FlatTop diameter 5.0mm 2 pins")
-    (fp_text reference D1 (at 1.27 -4.01 180) (layer F.SilkS)
-      (effects (font (size 1 1) (thickness 0.15)))
-    )
-    (fp_text value LED (at 1.27 4.01 180) (layer F.Fab)
+    (fp_text reference D1 (at -1.27 -3.81 180) (layer F.SilkS)
+      (effects (font (size 1 1) (thickness 0.15)))
+    )
+    (fp_text value LED (at 1.27 -3.81 180) (layer F.Fab)
       (effects (font (size 1 1) (thickness 0.15)))
     )
@@
     (descr "LED, Round, FlatTop, diameter 5.0mm, 2 pins, http://www.kingbright.com/attachments/file/psearch/000/00/00/L-483GDT(Ver.15B).pdf")
     (tags "LED Round FlatTop diameter 5.0mm 2 pins")
-    (fp_text reference D7 (at 1.27 -4.01) (layer F.SilkS)
+    (fp_text reference D7 (at 3.81 3.81) (layer F.SilkS)
       (effects (font (size 1 1) (thickness 0.15)))
     )
@@
     (at 134.112 221.742 270)
     (descr "<b>WR-TBL Serie 213 - 5.0mm 45° Entry Modular with Rising Cage Clamp -  1.5mm2 Wires, 3 Pins")
-    (fp_text reference J3 (at -0.352815 -5.67487 270) (layer F.SilkS)
+    (fp_text reference J3 (at -0.127 2.667 270) (layer F.SilkS)
       (effects (font (size 1.00229 1.00229) (thickness 0.05)))
     )
@@
     (at 134.112 208.534 270)
     (descr "<b>WR-TBL Serie 2165 - 5.08mm Horizontal Entry Modular with Rising Cage Clamp - 3.5mm2 Wires, 2 Pins")
-    (fp_text reference J2 (at -0.196539 -6.71131 270) (layer F.SilkS)
+    (fp_text reference J2 (at -0.196539 2.667 270) (layer F.SilkS)
       (effects (font (size 1.00265 1.00265) (thickness 0.05)))
     )
@@
     )
   )
-  (dimension 12.7 (width 0.15) (layer F.SilkS)
-    (gr_text "12,700 mm" (at 133.35 72.36) (layer F.SilkS)
-      (effects (font (size 1 1) (thickness 0.15)))
-    )
-    (feature1 (pts (xy 127 80.01) (xy 127 73.073579)))
-    (feature2 (pts (xy 139.7 80.01) (xy 139.7 73.073579)))
-    (crossbar (pts (xy 139.7 73.66) (xy 127 73.66)))
-    (arrow1a (pts (xy 127 73.66) (xy 128.126504 73.073579)))
-    (arrow1b (pts (xy 127 73.66) (xy 128.126504 74.246421)))
-    (arrow2a (pts (xy 139.7 73.66) (xy 138.573496 73.073579)))
-    (arrow2b (pts (xy 139.7 73.66) (xy 138.573496 74.246421)))
-  )
-  (dimension 12.7 (width 0.15) (layer F.SilkS)
-    (gr_text "12,700 mm" (at 34.768 83.82 270) (layer F.SilkS)
-      (effects (font (size 1 1) (thickness 0.15)))
-    )
-    (feature1 (pts (xy 45.72 90.17) (xy 35.481579 90.17)))
-    (feature2 (pts (xy 45.72 77.47) (xy 35.481579 77.47)))
-    (crossbar (pts (xy 36.068 77.47) (xy 36.068 90.17)))
-    (arrow1a (pts (xy 36.068 90.17) (xy 35.481579 89.043496)))
-    (arrow1b (pts (xy 36.068 90.17) (xy 36.654421 89.043496)))
-    (arrow2a (pts (xy 36.068 77.47) (xy 35.481579 78.596504)))
-    (arrow2b (pts (xy 36.068 77.47) (xy 36.654421 78.596504)))
-  )
-  (dimension 12.7 (width 0.15) (layer F.SilkS)
-    (gr_text "12,700 mm" (at 144.302 83.82 270) (layer F.SilkS)
-      (effects (font (size 1 1) (thickness 0.15)))
-    )
-    (feature1 (pts (xy 136.398 90.17) (xy 143.588421 90.17)))
-    (feature2 (pts (xy 136.398 77.47) (xy 143.588421 77.47)))
-    (crossbar (pts (xy 143.002 77.47) (xy 143.002 90.17)))
-    (arrow1a (pts (xy 143.002 90.17) (xy 142.415579 89.043496)))
-    (arrow1b (pts (xy 143.002 90.17) (xy 143.588421 89.043496)))
-    (arrow2a (pts (xy 143.002 77.47) (xy 142.415579 78.596504)))
-    (arrow2b (pts (xy 143.002 77.47) (xy 143.588421 78.596504)))
+  (gr_text AKKU/PC (at 89.535 88.265) (layer B.Cu)
+    (effects (font (size 3 3) (thickness 0.6)) (justify mirror))
+  )
+  (gr_text AKKU/PC (at 89.535 88.265) (layer F.SilkS)
+    (effects (font (size 3 3) (thickness 0.6)))
+  )
+  (gr_text - (at 61.595 82.55) (layer F.SilkS)
+    (effects (font (size 1.5 1.5) (thickness 0.3)))
+  )
+  (gr_text + (at 49.53 82.55) (layer F.SilkS)
+    (effects (font (size 1.5 1.5) (thickness 0.3)))
+  )
+  (gr_text read (at 55.88 114.935) (layer F.SilkS)
+    (effects (font (size 1.5 1.5) (thickness 0.3)))
+  )
+  (gr_text write (at 62.23 114.935) (layer F.SilkS)
+    (effects (font (size 1.5 1.5) (thickness 0.3)))
+  )
+  (gr_text clear (at 125.095 226.695) (layer F.SilkS)
+    (effects (font (size 1.5 1.5) (thickness 0.3)))
+  )
+  (gr_text ~en (at 125.73 221.615) (layer F.SilkS)
+    (effects (font (size 1.5 1.5) (thickness 0.3)))
+  )
+  (gr_text ~down (at 125.73 216.535) (layer F.SilkS)
+    (effects (font (size 1.5 1.5) (thickness 0.3)))
+  )
+  (gr_text ~up (at 125.73 210.82) (layer F.SilkS)
+    (effects (font (size 1.5 1.5) (thickness 0.3)))
+  )
+  (gr_text ~load (at 125.73 205.74) (layer F.SilkS)
+    (effects (font (size 1.5 1.5) (thickness 0.3)))
+  )
+  (gr_text CLEAR (at 82.55 218.44) (layer F.SilkS)
+    (effects (font (size 1.5 1.5) (thickness 0.3)))
+  )
+  (gr_text DOWN (at 68.58 218.44) (layer F.SilkS)
+    (effects (font (size 1.5 1.5) (thickness 0.3)))
+  )
+  (gr_text UP (at 54.61 218.44) (layer F.SilkS)
+    (effects (font (size 1.5 1.5) (thickness 0.3)))
   )
   (segment (start 93.98 121.92) (end 93.98 124.46) (width 0.6) (layer B.Cu) (net 1) (status 30))
